Commit message: El bote se logra mover con inputs de thrust a los motores. Alto empuje hace que se mueva un poco chueco. Verificar

File: src/vtec_s3_description/robots/vtecs3_default.xacro (robot description, xacro)
@@ -15,5 +15,5 @@
     <gazebo>
       <plugin name="uuv_plugin" filename="libuuv_underwater_object_ros_plugin.so">
-        <fluid_density>1028.0</fluid_density>
+        <fluid_density>1000.0</fluid_density>
         <flow_velocity_topic>hydrodynamics/current_velocity</flow_velocity_topic>
         <debug>$(arg debug)</debug>

File: src/vtec_s3_description/urdf/actuators.xacro (robot description, xacro)
@@ -10,10 +10,10 @@
     <!-- Improve origin -->
     <xacro:thruster_macro robot_namespace="${namespace}" thruster_id="0">
-        <origin xyz="-0.2 -0.205 -0.25" rpy="0 0 0"/>
+        <origin xyz="-0.305 -0.19905 -0.1473" rpy="0 0 3.14159"/>
         <!-- yaw anterior : "${pi}" -->
     </xacro:thruster_macro>
     <!-- Improve origin -->
     <xacro:thruster_macro robot_namespace="${namespace}" thruster_id="1">
-        <origin xyz="-0.2 0.205 -0.25" rpy="0 0 0" />
+        <origin xyz="-0.305 0.19905 -0.1473" rpy="0 0 3.14159" />
         <!-- yaw anterior : "${pi}" -->
     </xacro:thruster_macro>

File: src/vtec_s3_description/urdf/base.xacro (robot description, xacro)
@@ -14,5 +14,5 @@
   <xacro:property name="mass" value="30"/>
   <!-- Center of gravity -->
-  <xacro:property name="cog" value="0 0 0.19"/> <!-- Superficie del barco esta a 0.16 m de COM en Z-->
+  <xacro:property name="cog" value="0 0 0.19"/> <!-- Superficie del barco esta a 0.19 m de COM en Z-->
   <!-- Fluid density -->
   <xacro:property name="rho" value="1000"/>
@@ -70,5 +70,5 @@
     <xacro:insert_block name="gazebo"/>
     <!-- Include the thruster modules -->
-    <!-- <xacro:include filename="$(find vtec_s3_description)/urdf/actuators.xacro"/> -->
+    <xacro:include filename="$(find vtec_s3_description)/urdf/actuators.xacro"/>
     <!-- Include the sensor modules -->
     <!-- <xacro:include filename="$(find vtec_s3_description)/urdf/sensors.xacro"/> -->

File: src/vtec_s3_description/urdf/snippets.xacro (robot description, xacro)
@@ -51,7 +51,7 @@
         <gain>1</gain>
         <!-- Maximum allowed input value for the input signal for thruster unit -->
-        <!-- <clampMax>0</clampMax> -->
+        <!-- <clampMax>-3000</clampMax> -->
         <!-- Minimum allowed value for the input signal for thruster unit -->
-        <!-- <clampMin>0</clampMin> -->
+        <!-- <clampMin>3000</clampMin> -->
         <!-- Minimum and maximum thrust force output allowed -->
         <thrustMin>-30</thrustMin>
@@ -81,5 +81,5 @@
         <dynamics>
           <type>FirstOrder</type>
-          <timeConstant>0.2</timeConstant>
+          <timeConstant>0.002</timeConstant>
         </dynamics>
         <!-- 3) Yoerger's nonlinear dynamic model
@@ -121,5 +121,5 @@
         <conversion>
           <type>Basic</type>
-          <rotorConstant>0.00001</rotorConstant>
+          <rotorConstant>0.002</rotorConstant>
         </conversion>
         <!-- 2) Dead-zone nonlinearity described in Bessa, 2006
