Commit message: Checked for stability in the whole submarine: Damping coefficients turned out to be enough for the simulation COG is now at the geometric origin of the uuv Thrusters' position modified according to the change of the COG ISSUE: real COB turned out to be around 2 cm above COG. This affected pitch stability in the simulation and could potentially affect the real uuv. To achieve stability, COB was set 22 cm above COG. Surge speed is completely rectilinear Sway presents some inestability at large speed At most, heave can achieve a speed of cero for now TO DO: change gains of thrusters to achieve heave

File: vtec_u3_description/robots/default.xacro (robot description, xacro)
@@ -3,5 +3,5 @@
   <xacro:arg name="debug" default="0"/>
   <xacro:arg name="namespace" default="vtec_u3"/>
-  <!-- Include the ROV macro file -->
+  <!-- Include the UUV macro file -->
   <xacro:include filename="$(find vtec_u3_description)/urdf/base.xacro"/>
   <xacro:include filename="$(find vtec_u3_description)/urdf/gazebo.xacro"/>

File: vtec_u3_description/urdf/actuators.xacro (robot description, xacro)
@@ -10,20 +10,20 @@
     <!-- Note: measurements are as exact as were possible from SolidWorks. Just check the result -->
     <xacro:thruster_macro robot_namespace="${namespace}" thruster_id="0">
-        <origin xyz="0.19511 0.30924 0.01005" rpy="0 0 ${0.75*pi}" />
+        <origin xyz="0.18829 0.30023 0" rpy="0 0 ${0.75*pi}" />
     </xacro:thruster_macro>
     <xacro:thruster_macro robot_namespace="${namespace}" thruster_id="1">
-        <origin xyz="0.19519 -0.29114 0.01005" rpy="0 0 -${0.75*pi}" />
+        <origin xyz="0.18829 -0.30023 0" rpy="0 0 -${0.75*pi}" />
     </xacro:thruster_macro>
     <xacro:thruster_macro robot_namespace="${namespace}" thruster_id="2">
-    <origin xyz="0.04519 -0.26079 -0.03151" rpy="0 ${0.5*pi} 0" />
+        <origin xyz="-0.03828 0.26988 -0.04156" rpy="0 ${0.5*pi} 0" />
     </xacro:thruster_macro>
     <xacro:thruster_macro robot_namespace="${namespace}" thruster_id="3">
-        <origin xyz="-0.03138 0.27898 -0.03151" rpy="0 ${0.5*pi} 0" />
+        <origin xyz="0.03828 -0.26988 -0.04156" rpy="0 ${0.5*pi} 0" />
     </xacro:thruster_macro>
     <xacro:thruster_macro robot_namespace="${namespace}" thruster_id="4">
-        <origin xyz="-0.18139 -0.29113 0.01005" rpy="0 0 -${0.25*pi}" />
+        <origin xyz="-0.18829 0.30023 0" rpy="0 0 ${0.25*pi}" />
     </xacro:thruster_macro>
     <xacro:thruster_macro robot_namespace="${namespace}" thruster_id="5">
-    <origin xyz="-0.18139 0.30932 0.01005" rpy="0 0 ${0.25*pi}" />
+        <origin xyz="-0.18829 -0.30023 0" rpy="0 0 -${0.25*pi}" />
     </xacro:thruster_macro>
 </robot>

File: vtec_u3_description/urdf/base.xacro (robot description, xacro)
@@ -13,6 +13,9 @@
   -->
   <xacro:property name="mass" value="18.74"/>
+  <!-- The origin of the model is at 0,0,0 in ENU, which is coincident with the COG of the CAD model, but to increase stability, the COG is assumed
+       to be in the same position as the geometric center of the UUV, hence the little offset presented when the COG is described below -->
   <!-- Center of gravity -->
-  <xacro:property name="cog" value="0 0 0"/>
+  <xacro:property name="cog" value="0 0 0"/> <!-- At the quasi geometric center -> we'll take it as the COG-->
+  <xacro:property name="geocenter" value="-0.0069 -0.00909 -0.01005"/>
   <!-- Fluid density -->
   <xacro:property name="rho" value="1000"/>
@@ -38,11 +41,20 @@
         <inertial>
           <mass value="${mass}" />
-          <origin xyz="${cog}" rpy="0 0 0"/>
-          <inertia ixx="0.49770495" ixy="0.00275177" ixz="-0.0574426"
+          <origin xyz="0 0 0" rpy="0 0 0"/>
+          <!-- From Pedro's report -->
+          <!-- <inertia ixx="0.49770495" ixy="0.00275177" ixz="-0.0574426"
                    iyy="0.37089716" iyz="-0.0036791"
-                   izz="0.64879823" />
+                   izz="0.64879823" /> -->
+          <!-- From Solidworks -->
+          <!-- <inertia ixx="0.66676616706" ixy="0.00116837789" ixz="0.05627875991"
+                   iyy="0.41083355789" iyz="-0.01350290989"
+                   izz="0.81311081679" /> -->
+          <!-- For COM nearly in geometric center -->
+            <inertia ixx="0.83639798529" ixy="-0.00503680373" ixz="0.0560001532"
+                      iyy="0.46118483068" iyz="-0.01377965358"
+                      izz="1.02986207702" />
         </inertial>
         <visual>
-          <origin xyz="0 0 0" rpy="0 0 0"/>
+          <origin xyz="${geocenter}" rpy="0 0 0"/>
           <geometry>
             <mesh filename="${visual_mesh_file}" scale="0.001 0.001 0.001" />

File: vtec_u3_description/urdf/gazebo.xacro (robot description, xacro)
@@ -1,11 +1,14 @@
 <?xml version="1.0"?>
 <robot xmlns:xacro="http://www.ros.org/wiki/xacro">
-    <!-- Center of buoyancy -->
-    <xacro:property name="vtec_u3_cob" value="0 0 0"/>
+    <!-- Center of buoyancy (must be set with respect to COG)-->
+    <xacro:property name="vtec_u3_cob" value="0 0 0.22"/> <!-- For stability, it should remain as far as possible from COM in z -->
+    <!-- In solidworks, the COB proved to be in 0.00777 0.00725 0.0146 with respect to the origin of the CAD (the real COG), which means
+         unstability will be presented. COB should be in the same place as COG in the XY plane and as possible from it in z -->
+    <!-- Having a COB so close to COG means problems in pitch-->
     <!-- Vehicle's actual volume (Gazebo cannot compute the volume out of the mesh) -->
     <xacro:property name="vtec_u3_volume" value="0.01209"/>
     <!-- Describing the dimensions of the vehicle's bounding box -->
-    <xacro:property name="vtec_u3_length" value="0.45"/>
-    <xacro:property name="vtec_u3_width"  value="0.7"/>
+    <xacro:property name="vtec_u3_length" value="0.7"/>
+    <xacro:property name="vtec_u3_width"  value="0.45"/>
     <xacro:property name="vtec_u3_height" value="0.34"/>
     <xacro:macro name="vtec_u3_hydro_model" params="namespace">
@@ -65,5 +68,5 @@
           -->
           <quadratic_damping>
-            -45.808 -41.282 -42.243 -0.3185 -0.4752 -0.607
+            -45.808 -41.282 -42.243 0.3185 -0.4752 -0.607
           </quadratic_damping>
           <!--

File: vtec_u3_description/urdf/sensors.xacro (robot description, xacro)
@@ -7,4 +7,5 @@
     more examples or add you own custom sensor units.
   -->
+  <!-- Must be set with respect to COG -->
   <!-- Mount a GPS. -->
   <xacro:default_gps namespace="${namespace}" parent_link="${namespace}/base_link" />

File: vtec_u3_description/urdf/snippets.xacro (robot description, xacro)
@@ -122,5 +122,5 @@
         <conversion>
           <type>Basic</type>
-          <rotorConstant>0.002</rotorConstant>
+          <rotorConstant>0.02</rotorConstant>
         </conversion>
         <!-- 2) Dead-zone nonlinearity described in Bessa, 2006
