Commit message: Changes

File: vtec_u3_description/urdf/actuators.xacro (robot description, xacro)
@@ -18,5 +18,5 @@
     </xacro:thruster_macro>
     <!-- Instantiate fins, if necessary -->
-    <xacro:fin_macro namespace="${namespace}" fin_id="0">
+    <!-- <xacro:fin_macro namespace="${namespace}" fin_id="0">
       <origin xyz="0 0 0" rpy="0 0 0" />
     </xacro:fin_macro>
@@ -29,4 +29,4 @@
     <xacro:fin_macro namespace="${namespace}" fin_id="3">
       <origin xyz="0 0 0" rpy="0 0 0" />
-    </xacro:fin_macro>
+    </xacro:fin_macro> -->
 </robot>

File: vtec_u3_description/urdf/base.xacro (robot description, xacro)
@@ -62,5 +62,5 @@
     <xacro:insert_block name="gazebo"/>
     <!-- Include the thruster modules -->
-    <!-- <xacro:include filename="$(find vtec_u3_description)/urdf/actuators.xacro"/> -->
+    <xacro:include filename="$(find vtec_u3_description)/urdf/actuators.xacro"/>
     <!-- Include the sensor modules -->
     <!-- <xacro:include filename="$(find vtec_u3_description)/urdf/sensors.xacro"/> -->

File: vtec_u3_description/urdf/snippets.xacro (robot description, xacro)
@@ -7,5 +7,5 @@
   over propeller's frame X-axis in DAE (Collada) or STL format.
   -->
-  <xacro:property name="prop_mesh_file" value="file://$(find vtec_s3_description)/meshes/bluerob_propcw.dae"/>
+  <xacro:property name="prop_mesh_file" value="file://$(find vtec_u3_description)/meshes/bluerob_propcw.dae"/>
   <!--
     Thruster macro with integration of joint and link. The thrusters should

Commit message: Added actuators' poses for the model. I consider they are very accurate

File: vtec_u3_description/urdf/actuators.xacro (robot description, xacro)
@@ -8,25 +8,22 @@
           aware that Gazebo does not use the SNAME convention per default.
     -->
+    <!-- Note: measurements are as exact as were possible from SolidWorks. Just check the result -->
     <xacro:thruster_macro robot_namespace="${namespace}" thruster_id="0">
-        <origin xyz="0 0 0" rpy="0 0 ${pi}" />
+        <origin xyz="0.19511 0.30924 0.01005" rpy="0 0 ${0.75*pi}" />
     </xacro:thruster_macro>
     <xacro:thruster_macro robot_namespace="${namespace}" thruster_id="1">
-        <origin xyz="0 0 0" rpy="0 0 ${pi}" />
+        <origin xyz="0.19519 -0.29114 0.01005" rpy="0 0 -${0.75*pi}" />
     </xacro:thruster_macro>
     <xacro:thruster_macro robot_namespace="${namespace}" thruster_id="2">
-    <origin xyz="0 0 0" rpy="0 -${0.5*pi} 0" />
+    <origin xyz="0.04519 -0.26079 -0.03151" rpy="0 ${0.5*pi} 0" />
     </xacro:thruster_macro>
-    <!-- Instantiate fins, if necessary -->
-    <xacro:fin_macro namespace="${namespace}" fin_id="0">
-      <origin xyz="0 0 0" rpy="0 0 0" />
-    </xacro:fin_macro>
-    <xacro:fin_macro namespace="${namespace}" fin_id="1">
-      <origin xyz="0 0 0" rpy="0 0 0" />
-    </xacro:fin_macro>
-    <xacro:fin_macro namespace="${namespace}" fin_id="2">
-      <origin xyz="0 0 0" rpy="0 0 0" />
-    </xacro:fin_macro>
-    <xacro:fin_macro namespace="${namespace}" fin_id="3">
-      <origin xyz="0 0 0" rpy="0 0 0" />
-    </xacro:fin_macro>
+    <xacro:thruster_macro robot_namespace="${namespace}" thruster_id="3">
+        <origin xyz="-0.03138 0.27898 -0.03151" rpy="0 ${0.5*pi} 0" />
+    </xacro:thruster_macro>
+    <xacro:thruster_macro robot_namespace="${namespace}" thruster_id="4">
+        <origin xyz="-0.18139 -0.29113 0.01005" rpy="0 0 -${0.25*pi}" />
+    </xacro:thruster_macro>
+    <xacro:thruster_macro robot_namespace="${namespace}" thruster_id="5">
+    <origin xyz="-0.18139 0.30932 0.01005" rpy="0 0 ${0.25*pi}" />
+    </xacro:thruster_macro>
 </robot>

File: vtec_u3_description/urdf/base.xacro (robot description, xacro)
@@ -62,5 +62,5 @@
     <xacro:insert_block name="gazebo"/>
     <!-- Include the thruster modules -->
-    <!-- <xacro:include filename="$(find vtec_u3_description)/urdf/actuators.xacro"/> -->
+    <xacro:include filename="$(find vtec_u3_description)/urdf/actuators.xacro"/>
     <!-- Include the sensor modules -->
     <!-- <xacro:include filename="$(find vtec_u3_description)/urdf/sensors.xacro"/> -->

File: vtec_u3_description/urdf/snippets.xacro (robot description, xacro)
@@ -7,5 +7,6 @@
   over propeller's frame X-axis in DAE (Collada) or STL format.
   -->
-  <xacro:property name="prop_mesh_file" value="file://$(find vtec_s3_description)/meshes/bluerob_propcw.dae"/>
+  <!-- To improve: add mirror propeller -->
+  <xacro:property name="prop_mesh_file" value="file://$(find vtec_u3_description)/meshes/bluerob_propcw.dae"/>
   <!--
     Thruster macro with integration of joint and link. The thrusters should

Commit message: Sensors

File: vtec_u3_description/urdf/actuators.xacro (robot description, xacro)
@@ -9,11 +9,20 @@
     -->
     <xacro:thruster_macro robot_namespace="${namespace}" thruster_id="0">
-        <origin xyz="0 0 0" rpy="0 0 ${pi}" />
+        <origin xyz="0.19789 -0.28839 0.01070" rpy="0 0 ${pi}" />
     </xacro:thruster_macro>
     <xacro:thruster_macro robot_namespace="${namespace}" thruster_id="1">
-        <origin xyz="0 0 0" rpy="0 0 ${pi}" />
+        <origin xyz="0.04583 -0.26083 -0.02765" rpy="0 0 ${pi}" />
     </xacro:thruster_macro>
     <xacro:thruster_macro robot_namespace="${namespace}" thruster_id="2">
-    <origin xyz="0 0 0" rpy="0 -${0.5*pi} 0" />
+      <origin xyz="-0.18414 -0.28844 0.01070" rpy="0 -${0.5*pi} 0" />
+    </xacro:thruster_macro>
+    <xacro:thruster_macro robot_namespace="${namespace}" thruster_id="3">
+      <origin xyz="0.19790 0.30658 0.01070" rpy="0 -${0.5*pi} 0" />
+    </xacro:thruster_macro>
+    <xacro:thruster_macro robot_namespace="${namespace}" thruster_id="4">
+        <origin xyz="-0.03203 0.279 -0.02765" rpy="0 0 ${pi}" />
+    </xacro:thruster_macro>
+    <xacro:thruster_macro robot_namespace="${namespace}" thruster_id="5">
+        <origin xyz="-0.18409 0.30657 0.01070" rpy="0 0 ${pi}" />
     </xacro:thruster_macro>
     <!-- Instantiate fins, if necessary -->

File: vtec_u3_description/urdf/base.xacro (robot description, xacro)
@@ -64,5 +64,5 @@
     <xacro:include filename="$(find vtec_u3_description)/urdf/actuators.xacro"/>
     <!-- Include the sensor modules -->
-    <!-- <xacro:include filename="$(find vtec_u3_description)/urdf/sensors.xacro"/> -->
+    <xacro:include filename="$(find vtec_u3_description)/urdf/sensors.xacro"/>
   </xacro:macro>
 </robot>

File: vtec_u3_description/urdf/sensors.xacro (robot description, xacro)
@@ -8,30 +8,30 @@
   -->
   <!-- Mount a GPS. -->
-  <xacro:default_gps namespace="${namespace}" parent_link="${namespace}/base_link" />
+  <!--<xacro:default_gps namespace="${namespace}" parent_link="${namespace}/base_link" />-->
   <!-- Mount a Pose 3D sensor. -->
-  <xacro:default_pose_3d namespace="${namespace}" parent_link="${namespace}/base_link" />
+  <!--<xacro:default_pose_3d namespace="${namespace}" parent_link="${namespace}/base_link" /> -->
   <!-- Forward-looking sonar sensor -->
-  <xacro:forward_multibeam_p900 namespace="${namespace}" parent_link="${namespace}/base_link">
-    <origin xyz="0 0 0" rpy="0 0 0"/>
-  </xacro:forward_multibeam_p900>
+  <!--<xacro:forward_multibeam_p900 namespace="${namespace}" parent_link="${namespace}/base_link">
+    <origin xyz="0 0 0" rpy="0 0 0"/> -->
+  <!--</xacro:forward_multibeam_p900> -->
   <!-- DVL  -->
-  <xacro:default_dvl namespace="${namespace}" parent_link="${namespace}/base_link">
-    <origin xyz="0 0 0" rpy="0 0 0"/>
-  </xacro:default_dvl>
-  <!-- RPT  -->
-  <xacro:default_rpt namespace="${namespace}" parent_link="${namespace}/base_link">
-    <origin xyz="0 0 0" rpy="0 0 0"/>
-  </xacro:default_rpt>
+  <!--<xacro:default_dvl namespace="${namespace}" parent_link="${namespace}/base_link">
+    <origin xyz="0 0 0" rpy="0 0 0"/>-->
+  <!--</xacro:default_dvl> -->
+   <!-- RPT  -->
+  <!--<xacro:default_rpt namespace="${namespace}" parent_link="${namespace}/base_link">
+    <origin xyz="0 0 0" rpy="0 0 0"/>-->
+  <!--</xacro:default_rpt>-->
   <!-- Pressure  -->
   <xacro:default_pressure namespace="${namespace}" parent_link="${namespace}/base_link">
-    <origin xyz="0 0 0" rpy="0 0 0"/>
+    <origin xyz="-0.10278 0.03138 0.10095" rpy="0 0 0"/>
   </xacro:default_pressure>
   <!-- IMU  -->
   <xacro:default_imu namespace="${namespace}" parent_link="${namespace}/base_link">
-    <origin xyz="0 0 0" rpy="0 0 0"/>
+    <origin xyz="0.08992 0.00853 0.05671" rpy="0 0 0"/>
   </xacro:default_imu>
   <!-- Mount a camera  -->
   <xacro:default_camera namespace="${namespace}" parent_link="${namespace}/base_link" suffix="">
-    <origin xyz="0 0 0" rpy="0 0 0"/>
+    <origin xyz="0.19281 0.01961 0.06659" rpy="0 0 0"/>
   </xacro:default_camera>
 </robot>

File: vtec_u3_description/urdf/snippets.xacro (robot description, xacro)
@@ -7,5 +7,5 @@
   over propeller's frame X-axis in DAE (Collada) or STL format.
   -->
-  <xacro:property name="prop_mesh_file" value="file://$(find vtec_u3_description)/meshes/bluerob_propcw.dae"/>
+ <!-- <xacro:property name="prop_mesh_file" value="file://$(find vtec_u3_description)/meshes/bluerob_propcw.dae"/>-->
   <!--
     Thruster macro with integration of joint and link. The thrusters should

Commit message: Reverted merge conflicts modification
This reverts commit 5493e5c108a3daedc4c9150d9bbdd8ed80246f42, reversing
changes made to 36441c7fbd007b27b599f7a96ef79cc146354c3d.

File: vtec_u3_description/urdf/actuators.xacro (robot description, xacro)
@@ -8,22 +8,34 @@
           aware that Gazebo does not use the SNAME convention per default.
     -->
-    <!-- Note: measurements are as exact as were possible from SolidWorks. Just check the result -->
     <xacro:thruster_macro robot_namespace="${namespace}" thruster_id="0">
-        <origin xyz="0.18829 0.30023 0" rpy="0 0 ${0.75*pi}" />
+        <origin xyz="0.19789 -0.28839 0.01070" rpy="0 0 ${pi}" />
     </xacro:thruster_macro>
     <xacro:thruster_macro robot_namespace="${namespace}" thruster_id="1">
-        <origin xyz="0.18829 -0.30023 0" rpy="0 0 -${0.75*pi}" />
+        <origin xyz="0.04583 -0.26083 -0.02765" rpy="0 0 ${pi}" />
     </xacro:thruster_macro>
     <xacro:thruster_macro robot_namespace="${namespace}" thruster_id="2">
-        <origin xyz="-0.03828 0.26988 -0.04156" rpy="0 ${0.5*pi} 0" />
+      <origin xyz="-0.18414 -0.28844 0.01070" rpy="0 -${0.5*pi} 0" />
     </xacro:thruster_macro>
     <xacro:thruster_macro robot_namespace="${namespace}" thruster_id="3">
-        <origin xyz="0.03828 -0.26988 -0.04156" rpy="0 ${0.5*pi} 0" />
+      <origin xyz="0.19790 0.30658 0.01070" rpy="0 -${0.5*pi} 0" />
     </xacro:thruster_macro>
     <xacro:thruster_macro robot_namespace="${namespace}" thruster_id="4">
-        <origin xyz="-0.18829 0.30023 0" rpy="0 0 ${0.25*pi}" />
+        <origin xyz="-0.03203 0.279 -0.02765" rpy="0 0 ${pi}" />
     </xacro:thruster_macro>
     <xacro:thruster_macro robot_namespace="${namespace}" thruster_id="5">
-        <origin xyz="-0.18829 -0.30023 0" rpy="0 0 -${0.25*pi}" />
+        <origin xyz="-0.18409 0.30657 0.01070" rpy="0 0 ${pi}" />
     </xacro:thruster_macro>
+    <!-- Instantiate fins, if necessary -->
+    <!-- <xacro:fin_macro namespace="${namespace}" fin_id="0">
+      <origin xyz="0 0 0" rpy="0 0 0" />
+    </xacro:fin_macro>
+    <xacro:fin_macro namespace="${namespace}" fin_id="1">
+      <origin xyz="0 0 0" rpy="0 0 0" />
+    </xacro:fin_macro>
+    <xacro:fin_macro namespace="${namespace}" fin_id="2">
+      <origin xyz="0 0 0" rpy="0 0 0" />
+    </xacro:fin_macro>
+    <xacro:fin_macro namespace="${namespace}" fin_id="3">
+      <origin xyz="0 0 0" rpy="0 0 0" />
+    </xacro:fin_macro> -->
 </robot>

File: vtec_u3_description/urdf/base.xacro (robot description, xacro)
@@ -13,14 +13,6 @@
   -->
   <xacro:property name="mass" value="18.74"/>
-<<<<<<< HEAD
   <!-- Center of gravity -->
   <xacro:property name="cog" value="0 0 0"/>
-=======
-  <!-- The origin of the model is at 0,0,0 in ENU, which is coincident with the COG of the CAD model, but to increase stability, the COG is assumed
-       to be in the same position as the geometric center of the UUV, hence the little offset presented when the COG is described below -->
-  <!-- Center of gravity -->
-  <xacro:property name="cog" value="0 0 0"/> <!-- At the quasi geometric center -> we'll take it as the COG-->
-  <xacro:property name="geocenter" value="-0.0069 -0.00909 -0.01005"/>
->>>>>>> e946dcf003282f3560dc7e3e7b27018b34966df5
   <!-- Fluid density -->
   <xacro:property name="rho" value="1000"/>
@@ -46,16 +38,11 @@
         <inertial>
           <mass value="${mass}" />
-          <origin xyz="0 0 0" rpy="0 0 0"/>
-          <!-- From Pedro's report -->
-          <!-- <inertia ixx="0.49770495" ixy="0.00275177" ixz="-0.0574426"
+          <origin xyz="${cog}" rpy="0 0 0"/>
+          <inertia ixx="0.49770495" ixy="0.00275177" ixz="-0.0574426"
                    iyy="0.37089716" iyz="-0.0036791"
-                   izz="0.64879823" /> -->
-          <!-- For COM nearly in geometric center -->
-            <inertia ixx="0.83639798529" ixy="-0.00503680373" ixz="0.0560001532"
-                      iyy="0.46118483068" iyz="-0.01377965358"
-                      izz="1.02986207702" />
+                   izz="0.64879823" />
         </inertial>
         <visual>
-          <origin xyz="${geocenter}" rpy="0 0 0"/>
+          <origin xyz="0 0 0" rpy="0 0 0"/>
           <geometry>
             <mesh filename="${visual_mesh_file}" scale="0.001 0.001 0.001" />

File: vtec_u3_description/urdf/gazebo.xacro (robot description, xacro)
@@ -1,14 +1,11 @@
 <?xml version="1.0"?>
 <robot xmlns:xacro="http://www.ros.org/wiki/xacro">
-    <!-- Center of buoyancy (must be set with respect to COG)-->
-    <xacro:property name="vtec_u3_cob" value="0 0 0.22"/> <!-- For stability, it should remain as far as possible from COM in z -->
-    <!-- In solidworks, the COB proved to be in 0.00777 0.00725 0.0146 with respect to the origin of the CAD (the real COG), which means
-         unstability will be presented. COB should be in the same place as COG in the XY plane and as possible from it in z -->
-    <!-- Having a COB so close to COG means problems in pitch-->
+    <!-- Center of buoyancy -->
+    <xacro:property name="vtec_u3_cob" value="0 0 0"/>
     <!-- Vehicle's actual volume (Gazebo cannot compute the volume out of the mesh) -->
     <xacro:property name="vtec_u3_volume" value="0.01209"/>
     <!-- Describing the dimensions of the vehicle's bounding box -->
-    <xacro:property name="vtec_u3_length" value="0.7"/>
-    <xacro:property name="vtec_u3_width"  value="0.45"/>
+    <xacro:property name="vtec_u3_length" value="0.45"/>
+    <xacro:property name="vtec_u3_width"  value="0.7"/>
     <xacro:property name="vtec_u3_height" value="0.34"/>
     <xacro:macro name="vtec_u3_hydro_model" params="namespace">

File: vtec_u3_description/urdf/sensors.xacro (robot description, xacro)
@@ -7,21 +7,20 @@
     more examples or add you own custom sensor units.
   -->
-  <!-- Must be set with respect to COG -->
   <!-- Mount a GPS. -->
-  <xacro:default_gps namespace="${namespace}" parent_link="${namespace}/base_link" />
+  <!--<xacro:default_gps namespace="${namespace}" parent_link="${namespace}/base_link" />-->
   <!-- Mount a Pose 3D sensor. -->
-  <xacro:default_pose_3d namespace="${namespace}" parent_link="${namespace}/base_link" />
+  <!--<xacro:default_pose_3d namespace="${namespace}" parent_link="${namespace}/base_link" /> -->
   <!-- Forward-looking sonar sensor -->
-  <xacro:forward_multibeam_p900 namespace="${namespace}" parent_link="${namespace}/base_link">
-    <origin xyz="0 0 0" rpy="0 0 0"/>
-  </xacro:forward_multibeam_p900>
+  <!--<xacro:forward_multibeam_p900 namespace="${namespace}" parent_link="${namespace}/base_link">
+    <origin xyz="0 0 0" rpy="0 0 0"/> -->
+  <!--</xacro:forward_multibeam_p900> -->
   <!-- DVL  -->
-  <xacro:default_dvl namespace="${namespace}" parent_link="${namespace}/base_link">
-    <origin xyz="0 0 0" rpy="0 0 0"/>
-  </xacro:default_dvl>
-  <!-- RPT  -->
-  <xacro:default_rpt namespace="${namespace}" parent_link="${namespace}/base_link">
-    <origin xyz="0 0 0" rpy="0 0 0"/>
-  </xacro:default_rpt>
+  <!--<xacro:default_dvl namespace="${namespace}" parent_link="${namespace}/base_link">
+    <origin xyz="0 0 0" rpy="0 0 0"/>-->
+  <!--</xacro:default_dvl> -->
+   <!-- RPT  -->
+  <!--<xacro:default_rpt namespace="${namespace}" parent_link="${namespace}/base_link">
+    <origin xyz="0 0 0" rpy="0 0 0"/>-->
+  <!--</xacro:default_rpt>-->
   <!-- Pressure  -->
   <xacro:default_pressure namespace="${namespace}" parent_link="${namespace}/base_link">

File: vtec_u3_description/urdf/snippets.xacro (robot description, xacro)
@@ -7,6 +7,5 @@
   over propeller's frame X-axis in DAE (Collada) or STL format.
   -->
-  <!-- To improve: add mirror propeller -->
-  <xacro:property name="prop_mesh_file" value="file://$(find vtec_u3_description)/meshes/bluerob_propcw.dae"/>
+ <!-- <xacro:property name="prop_mesh_file" value="file://$(find vtec_u3_description)/meshes/bluerob_propcw.dae"/>-->
   <!--
     Thruster macro with integration of joint and link. The thrusters should
@@ -56,6 +55,6 @@
         <!-- <clampMin>3000</clampMin> -->
         <!-- Minimum and maximum thrust force output allowed -->
-        <thrustMin>-100</thrustMin>
-        <thrustMax>100</thrustMax>
+        <thrustMin>-30</thrustMin>
+        <thrustMax>36.5</thrustMax>
         <!--
         Value from 0 to 1 to set the efficiency of the output thrust force
@@ -122,5 +121,5 @@
         <conversion>
           <type>Basic</type>
-          <rotorConstant>0.02892</rotorConstant>
+          <rotorConstant>0.002</rotorConstant>
         </conversion>
         <!-- 2) Dead-zone nonlinearity described in Bessa, 2006
