Commit message: add sensors

File: vtec_u3_description/urdf/sensors.xacro (robot description, xacro)
@@ -7,21 +7,20 @@
     more examples or add you own custom sensor units.
   -->
-  <!-- Must be set with respect to COG -->
   <!-- Mount a GPS. -->
-  <xacro:default_gps namespace="${namespace}" parent_link="${namespace}/base_link" />
+  <!--<xacro:default_gps namespace="${namespace}" parent_link="${namespace}/base_link" />-->
   <!-- Mount a Pose 3D sensor. -->
-  <xacro:default_pose_3d namespace="${namespace}" parent_link="${namespace}/base_link" />
+  <!--<xacro:default_pose_3d namespace="${namespace}" parent_link="${namespace}/base_link" /> -->
   <!-- Forward-looking sonar sensor -->
-  <xacro:forward_multibeam_p900 namespace="${namespace}" parent_link="${namespace}/base_link">
-    <origin xyz="0 0 0" rpy="0 0 0"/>
-  </xacro:forward_multibeam_p900>
+  <!--<xacro:forward_multibeam_p900 namespace="${namespace}" parent_link="${namespace}/base_link">
+    <origin xyz="0 0 0" rpy="0 0 0"/> -->
+  <!--</xacro:forward_multibeam_p900> -->
   <!-- DVL  -->
-  <xacro:default_dvl namespace="${namespace}" parent_link="${namespace}/base_link">
-    <origin xyz="0 0 0" rpy="0 0 0"/>
-  </xacro:default_dvl>
-  <!-- RPT  -->
-  <xacro:default_rpt namespace="${namespace}" parent_link="${namespace}/base_link">
-    <origin xyz="0 0 0" rpy="0 0 0"/>
-  </xacro:default_rpt>
+  <!--<xacro:default_dvl namespace="${namespace}" parent_link="${namespace}/base_link">
+    <origin xyz="0 0 0" rpy="0 0 0"/>-->
+  <!--</xacro:default_dvl> -->
+   <!-- RPT  -->
+  <!--<xacro:default_rpt namespace="${namespace}" parent_link="${namespace}/base_link">
+    <origin xyz="0 0 0" rpy="0 0 0"/>-->
+  <!--</xacro:default_rpt>-->
   <!-- Pressure  -->
   <xacro:default_pressure namespace="${namespace}" parent_link="${namespace}/base_link">

Commit message: Aiming system integration

File: vtec_u3_description/urdf/sensors.xacro (robot description, xacro)
@@ -25,13 +25,25 @@
   <!-- Pressure  -->
   <xacro:default_pressure namespace="${namespace}" parent_link="${namespace}/base_link">
-    <origin xyz="0 0 0" rpy="0 0 0"/>
+    <origin xyz="-0.10278 0.03138 0.10095" rpy="0 0 0"/>
   </xacro:default_pressure>
   <!-- IMU  -->
   <xacro:default_imu namespace="${namespace}" parent_link="${namespace}/base_link">
-    <origin xyz="0 0 0" rpy="0 0 0"/>
+    <origin xyz="0.08992 0.00853 0.05671" rpy="0 0 0"/>
   </xacro:default_imu>
   <!-- Mount a camera  -->
   <xacro:default_camera namespace="${namespace}" parent_link="${namespace}/base_link" suffix="">
-    <origin xyz="0 0 0" rpy="0 0 0"/>
+    <origin xyz="0.19281 0.01961 0.06659" rpy="0 0 0"/>
   </xacro:default_camera>
+  <!-- Mount base torpedos  -->
+  <xacro:base_torpedos namespace="${namespace}" parent_link="${namespace}/base_link" suffix="">
+    <origin xyz="0.19281 0.01961 -0.16659" rpy="0 0 1.5757"/>
+  </xacro:base_torpedos>
+  <!-- Mount torpedo1  -->
+  <xacro:torpedo1 namespace="${namespace}" parent_link="${namespace}/base_link" suffix="">
+    <origin xyz="0.27781 0.01961 -0.16659" rpy="0 0 0"/>
+  </xacro:torpedo1>
+  <!-- Mount torpedo2  -->
+  <xacro:torpedo2 namespace="${namespace}" parent_link="${namespace}/base_link" suffix="">
+    <origin xyz="0.10781 0.01961 -0.16659" rpy="0 0 0"/>
+  </xacro:torpedo2>
 </robot>

Commit message: Gate obstacle-torpedosbaselocation

File: vtec_u3_description/urdf/sensors.xacro (robot description, xacro)
@@ -37,5 +37,5 @@
   <!-- Mount base torpedos  -->
   <xacro:base_torpedos namespace="${namespace}" parent_link="${namespace}/base_link" suffix="">
-    <origin xyz="0.19281 0.01961 -0.16659" rpy="0 0 1.5757"/>
+    <origin xyz="0.1031 0.022 0.21" rpy="0 0 -1.5757"/>
   </xacro:base_torpedos>
   <!-- Mount torpedo1  -->

Commit message: two cameras sub, pointcloud enable just one

File: vtec_u3_description/urdf/sensors.xacro (robot description, xacro)
@@ -31,11 +31,19 @@
     <origin xyz="0.08992 0.00853 0.05671" rpy="0 0 0"/>
   </xacro:default_imu>
+  <!-- Realsense R200 1-->
+  <xacro:realsense_camera namespace="${namespace}" parent_link="${namespace}/base_link" suffix="front">
+    <origin xyz="0.19281 0.01961 0.06659" rpy="0 0 0"/>
+  </xacro:realsense_camera>
+  <!-- Realsense R200 -->
+  <xacro:realsense_camera namespace="${namespace}" parent_link="${namespace}/base_link" suffix="down">
+    <origin xyz="2.19281 0.01961 0.06659" rpy="0 1.57 0"/>
+  </xacro:realsense_camera>
   <!-- Realsense R200 -->
   <!-- Import macro for realsense-RS200 camera-->
-  <xacro:include filename="$(find realsense_gazebo_plugin)/urdf/realsense-RS200.macro.xacro"/>
+ <!-- <xacro:include filename="$(find realsense_gazebo_plugin)/urdf/realsense-RS200.macro.xacro"/>-->
   <!-- Create camera instance -->
-  <xacro:realsense-rs200 prefix="" parent="${namespace}/base_link">
-    <origin xyz="0.19281 0.01961 0.06659" rpy="0 0 0"/>
-  </xacro:realsense-rs200>
+  <!--<xacro:realsense-rs200 prefix="" parent="${namespace}/base_link">-->
+  <!--  <origin xyz="0.19281 0.01961 0.06659" rpy="0 0 0"/>-->
+  <!--</xacro:realsense-rs200>-->
   <!-- Mount a camera  -->
   <!-- <xacro:default_camera namespace="${namespace}" parent_link="${namespace}/base_link" suffix="">

Commit message: color

File: vtec_u3_description/urdf/sensors.xacro (robot description, xacro)
@@ -37,5 +37,5 @@
   <!-- Realsense R200 -->
   <xacro:realsense_camera namespace="${namespace}" parent_link="${namespace}/base_link" suffix="down">
-    <origin xyz="2.19281 0.01961 0.06659" rpy="0 1.57 0"/>
+    <origin xyz="0.0 0.01961 0.18" rpy="0 -1.57 0"/>
   </xacro:realsense_camera>
   <!-- Realsense R200 -->
