Commit message: Changed damping coefficient sign and erased a comment

File: vtec_u3_description/urdf/base.xacro (robot description, xacro)
@@ -46,8 +46,4 @@
                    iyy="0.37089716" iyz="-0.0036791"
                    izz="0.64879823" /> -->
-          <!-- From Solidworks -->
-          <!-- <inertia ixx="0.66676616706" ixy="0.00116837789" ixz="0.05627875991"
-                   iyy="0.41083355789" iyz="-0.01350290989"
-                   izz="0.81311081679" /> -->
           <!-- For COM nearly in geometric center -->
             <inertia ixx="0.83639798529" ixy="-0.00503680373" ixz="0.0560001532"

File: vtec_u3_description/urdf/gazebo.xacro (robot description, xacro)
@@ -68,5 +68,5 @@
           -->
           <quadratic_damping>
-            -45.808 -41.282 -42.243 0.3185 -0.4752 -0.607
+            -45.808 -41.282 -42.243 -0.3185 -0.4752 -0.607
           </quadratic_damping>
           <!--

Commit message: Changes

File: vtec_u3_description/urdf/base.xacro (robot description, xacro)
@@ -8,13 +8,17 @@
   <xacro:include filename="$(find uuv_gazebo_ros_plugins)/urdf/snippets.xacro"/>
   <!-- Loading vehicle's specific macros -->
-  <xacro:include filename="$(find vtec_u3_description)/urdf/snippets.xacro"/>
+  <xacro:include filename="$(find vtec_s3_description)/urdf/snippets.xacro"/>
   <!--
     Vehicle's parameters (remember to enter the model parameters below)
   -->
-  <xacro:property name="mass" value="18.74"/>
+  <xacro:property name="mass" value="30"/>
   <!-- Center of gravity -->
-  <xacro:property name="cog" value="0 0 0"/>
+  <xacro:property name="cog" value="0 0 0.19"/> <!-- Superficie del barco esta a 0.19 m de COM en Z-->
   <!-- Fluid density -->
   <xacro:property name="rho" value="1000"/>
+  <!-- For the collision cube -->
+  <xacro:property name="x_size" value="1"/>
+  <xacro:property name="y_size" value="0.75"/>
+  <xacro:property name="z_size" value="0.5"/>
   <!--
     Visual mesh file for the vehicle, usually in DAE (Collada) format. Be sure to store the
@@ -23,11 +27,11 @@
     Open the meshes for the RexROV vehicle in Blender to see an example on the mesh placement.
   -->
-  <xacro:property name="visual_mesh_file" value="file://$(find vtec_u3_description)/meshes/vtec_u3_spl.dae"/>
+  <xacro:property name="visual_mesh_file" value="file://$(find vtec_s3_description)/meshes/VTECSIII_NOPROP.dae"/>
   <!-- Collision geometry mesh, usually in STL format (it is recommended to keep
   this geometry as simple as possible to improve the performance the physics engine
   regarding the computation of collision forces) -->
-  <xacro:property name="collision_mesh_file" value="file://$(find vtec_u3_description)/meshes/vtec_u3_spl.stl"/>
+  <xacro:property name="collision_mesh_file" value="file://$(find vtec_s3_description)/meshes/VTECSIII_NOPROP.stl"/>
   <!-- Vehicle macro -->
-  <xacro:macro name="vtec_u3_base" params="namespace *gazebo">
+  <xacro:macro name="vtec_s3_base" params="namespace *gazebo">
       <!-- Rigid body description of the base link -->
       <link name="${namespace}/base_link">
@@ -38,21 +42,25 @@
         <inertial>
           <mass value="${mass}" />
-          <origin xyz="${cog}" rpy="0 0 0"/>
-          <inertia ixx="0.49770495" ixy="0.00275177" ixz="-0.0574426"
-                   iyy="0.37089716" iyz="-0.0036791"
-                   izz="0.64879823" />
+          <origin xyz="0.05 0 0.19" rpy="0 0 0"/>
+          <!-- From SolidWorks -->
+          <inertia  ixx="2.5" ixy="-0.04046722475" ixz="-0.248111803"
+                    iyy="3.704654962" iyz="0.083214169"
+                    izz="4.1" />
         </inertial>
         <visual>
-          <origin xyz="0 0 0" rpy="0 0 0"/>
+          <!-- <origin xyz="0.55 -0.375 0.2" rpy="1.57075 3.141592 -1.57075"/> -->
+          <origin xyz="${cog}" rpy="0 0 0"/>
           <geometry>
+            <!-- <box size="1 0.75 0.5" />   -->
             <mesh filename="${visual_mesh_file}" scale="0.001 0.001 0.001" />
           </geometry>
         </visual>
-        <!-- <collision>
-          <origin xyz="0 0 0" rpy="0 0 0"/>
+        <collision>
+          <origin xyz="0.05 0 0.19" rpy="0 0 0"/>
           <geometry>
-            <mesh filename="${collision_mesh_file}" scale="0.001 0.001 0.001" />
+            <box size="${x_size} ${y_size} ${z_size}"/>
+            <!-- <mesh filename="${collision_mesh_file}" scale="0.001 0.001 0.001" /> --> <!-- To improve performance, we replaced it by a box -->
           </geometry>
-        </collision> -->
+        </collision>
       </link>
     <gazebo reference="${namespace}/base_link">
@@ -62,7 +70,7 @@
     <xacro:insert_block name="gazebo"/>
     <!-- Include the thruster modules -->
-    <xacro:include filename="$(find vtec_u3_description)/urdf/actuators.xacro"/>
+    <xacro:include filename="$(find vtec_s3_description)/urdf/actuators.xacro"/>
     <!-- Include the sensor modules -->
-    <xacro:include filename="$(find vtec_u3_description)/urdf/sensors.xacro"/>
+    <!-- <xacro:include filename="$(find vtec_s3_description)/urdf/sensors.xacro"/> -->
   </xacro:macro>
 </robot>

File: vtec_u3_description/urdf/sensors.xacro (robot description, xacro)
@@ -32,6 +32,9 @@
   </xacro:default_imu>
   <!-- Mount a camera  -->
+  <!--<xacro:stereo_camera namespace="${namespace}" parent_link="${namespace}/base_link" suffix="">-->
+  <!--  <origin xyz="0.19281 0.01961 0.06659" rpy="0 0 0"/>-->
+  <!-- </xacro:stereo_camera>-->
   <xacro:default_camera namespace="${namespace}" parent_link="${namespace}/base_link" suffix="">
-    <origin xyz="0.19281 0.01961 0.06659" rpy="0 0 0"/>
+   <origin xyz="0.19281 0.01961 0.06659" rpy="0 0 0"/>
   </xacro:default_camera>
 </robot>

File: vtec_u3_description/urdf/snippets.xacro (robot description, xacro)
@@ -7,5 +7,5 @@
   over propeller's frame X-axis in DAE (Collada) or STL format.
   -->
- <!-- <xacro:property name="prop_mesh_file" value="file://$(find vtec_u3_description)/meshes/bluerob_propcw.dae"/>-->
+ <xacro:property name="prop_mesh_file" value="file://$(find vtec_u3_description)/meshes/bluerob_propcw.dae"/>
   <!--
     Thruster macro with integration of joint and link. The thrusters should

Commit message: Changes2

File: vtec_u3_description/urdf/base.xacro (robot description, xacro)
@@ -8,5 +8,5 @@
   <xacro:include filename="$(find uuv_gazebo_ros_plugins)/urdf/snippets.xacro"/>
   <!-- Loading vehicle's specific macros -->
-  <xacro:include filename="$(find vtec_s3_description)/urdf/snippets.xacro"/>
+  <xacro:include filename="$(find vtec_u3_description)/urdf/snippets.xacro"/>
   <!--
     Vehicle's parameters (remember to enter the model parameters below)
@@ -27,11 +27,11 @@
     Open the meshes for the RexROV vehicle in Blender to see an example on the mesh placement.
   -->
-  <xacro:property name="visual_mesh_file" value="file://$(find vtec_s3_description)/meshes/VTECSIII_NOPROP.dae"/>
+  <xacro:property name="visual_mesh_file" value="file://$(find vtec_u3_description)/meshes/VTECSIII_NOPROP.dae"/>
   <!-- Collision geometry mesh, usually in STL format (it is recommended to keep
   this geometry as simple as possible to improve the performance the physics engine
   regarding the computation of collision forces) -->
-  <xacro:property name="collision_mesh_file" value="file://$(find vtec_s3_description)/meshes/VTECSIII_NOPROP.stl"/>
+  <xacro:property name="collision_mesh_file" value="file://$(find vtec_u3_description)/meshes/VTECSIII_NOPROP.stl"/>
   <!-- Vehicle macro -->
-  <xacro:macro name="vtec_s3_base" params="namespace *gazebo">
+  <xacro:macro name="vtec_u3_base" params="namespace *gazebo">
       <!-- Rigid body description of the base link -->
       <link name="${namespace}/base_link">
@@ -70,7 +70,7 @@
     <xacro:insert_block name="gazebo"/>
     <!-- Include the thruster modules -->
-    <xacro:include filename="$(find vtec_s3_description)/urdf/actuators.xacro"/>
+    <xacro:include filename="$(find vtec_u3_description)/urdf/actuators.xacro"/>
     <!-- Include the sensor modules -->
-    <!-- <xacro:include filename="$(find vtec_s3_description)/urdf/sensors.xacro"/> -->
+    <!-- <xacro:include filename="$(find vtec_u3_description)/urdf/sensors.xacro"/> -->
   </xacro:macro>
 </robot>

Commit message: Changes3

File: vtec_u3_description/urdf/base.xacro (robot description, xacro)
@@ -12,13 +12,12 @@
     Vehicle's parameters (remember to enter the model parameters below)
   -->
-  <xacro:property name="mass" value="30"/>
+  <xacro:property name="mass" value="18.74"/>
+  <!-- The origin of the model is at 0,0,0 in ENU, which is coincident with the COG of the CAD model, but to increase stability, the COG is assumed
+       to be in the same position as the geometric center of the UUV, hence the little offset presented when the COG is described below -->
   <!-- Center of gravity -->
-  <xacro:property name="cog" value="0 0 0.19"/> <!-- Superficie del barco esta a 0.19 m de COM en Z-->
+  <xacro:property name="cog" value="0 0 0"/> <!-- At the quasi geometric center -> we'll take it as the COG-->
+  <xacro:property name="geocenter" value="-0.0069 -0.00909 -0.01005"/>
   <!-- Fluid density -->
   <xacro:property name="rho" value="1000"/>
-  <!-- For the collision cube -->
-  <xacro:property name="x_size" value="1"/>
-  <xacro:property name="y_size" value="0.75"/>
-  <xacro:property name="z_size" value="0.5"/>
   <!--
     Visual mesh file for the vehicle, usually in DAE (Collada) format. Be sure to store the
@@ -27,9 +26,9 @@
     Open the meshes for the RexROV vehicle in Blender to see an example on the mesh placement.
   -->
-  <xacro:property name="visual_mesh_file" value="file://$(find vtec_u3_description)/meshes/VTECSIII_NOPROP.dae"/>
+  <xacro:property name="visual_mesh_file" value="file://$(find vtec_u3_description)/meshes/vtec_u3_spl.dae"/>
   <!-- Collision geometry mesh, usually in STL format (it is recommended to keep
   this geometry as simple as possible to improve the performance the physics engine
   regarding the computation of collision forces) -->
-  <xacro:property name="collision_mesh_file" value="file://$(find vtec_u3_description)/meshes/VTECSIII_NOPROP.stl"/>
+  <xacro:property name="collision_mesh_file" value="file://$(find vtec_u3_description)/meshes/vtec_u3_spl.stl"/>
   <!-- Vehicle macro -->
   <xacro:macro name="vtec_u3_base" params="namespace *gazebo">
@@ -42,25 +41,26 @@
         <inertial>
           <mass value="${mass}" />
-          <origin xyz="0.05 0 0.19" rpy="0 0 0"/>
-          <!-- From SolidWorks -->
-          <inertia  ixx="2.5" ixy="-0.04046722475" ixz="-0.248111803"
-                    iyy="3.704654962" iyz="0.083214169"
-                    izz="4.1" />
+          <origin xyz="0 0 0" rpy="0 0 0"/>
+          <!-- From Pedro's report -->
+          <!-- <inertia ixx="0.49770495" ixy="0.00275177" ixz="-0.0574426"
+                   iyy="0.37089716" iyz="-0.0036791"
+                   izz="0.64879823" /> -->
+          <!-- For COM nearly in geometric center -->
+            <inertia ixx="0.83639798529" ixy="-0.00503680373" ixz="0.0560001532"
+                      iyy="0.46118483068" iyz="-0.01377965358"
+                      izz="1.02986207702" />
         </inertial>
         <visual>
-          <!-- <origin xyz="0.55 -0.375 0.2" rpy="1.57075 3.141592 -1.57075"/> -->
-          <origin xyz="${cog}" rpy="0 0 0"/>
+          <origin xyz="${geocenter}" rpy="0 0 0"/>
           <geometry>
-            <!-- <box size="1 0.75 0.5" />   -->
             <mesh filename="${visual_mesh_file}" scale="0.001 0.001 0.001" />
           </geometry>
         </visual>
-        <collision>
-          <origin xyz="0.05 0 0.19" rpy="0 0 0"/>
+        <!-- <collision>
+          <origin xyz="0 0 0" rpy="0 0 0"/>
           <geometry>
-            <box size="${x_size} ${y_size} ${z_size}"/>
-            <!-- <mesh filename="${collision_mesh_file}" scale="0.001 0.001 0.001" /> --> <!-- To improve performance, we replaced it by a box -->
+            <mesh filename="${collision_mesh_file}" scale="0.001 0.001 0.001" />
           </geometry>
-        </collision>
+        </collision> -->
       </link>
     <gazebo reference="${namespace}/base_link">

Commit message: Camara integration

File: vtec_u3_description/urdf/base.xacro (robot description, xacro)
@@ -72,5 +72,5 @@
     <xacro:include filename="$(find vtec_u3_description)/urdf/actuators.xacro"/>
     <!-- Include the sensor modules -->
-    <!-- <xacro:include filename="$(find vtec_u3_description)/urdf/sensors.xacro"/> -->
+    <xacro:include filename="$(find vtec_u3_description)/urdf/sensors.xacro"/>
   </xacro:macro>
 </robot>

File: vtec_u3_description/urdf/sensors.xacro (robot description, xacro)
@@ -26,13 +26,13 @@
   <!-- Pressure  -->
   <xacro:default_pressure namespace="${namespace}" parent_link="${namespace}/base_link">
-    <origin xyz="0 0 0" rpy="0 0 0"/>
+    <origin xyz="-0.10278 0.03138 0.10095" rpy="0 0 0"/>
   </xacro:default_pressure>
   <!-- IMU  -->
   <xacro:default_imu namespace="${namespace}" parent_link="${namespace}/base_link">
-    <origin xyz="0 0 0" rpy="0 0 0"/>
+    <origin xyz="0.08992 0.00853 0.05671" rpy="0 0 0"/>
   </xacro:default_imu>
   <!-- Mount a camera  -->
   <xacro:default_camera namespace="${namespace}" parent_link="${namespace}/base_link" suffix="">
-    <origin xyz="0 0 0" rpy="0 0 0"/>
+    <origin xyz="0.19281 0.01961 0.06659" rpy="0 0 0"/>
   </xacro:default_camera>
 </robot>

Commit message: Lots of changes

File: vtec_u3_description/urdf/base.xacro (robot description, xacro)
@@ -2,9 +2,5 @@
 <robot xmlns:xacro="http://www.ros.org/wiki/xacro">
   <!-- Loading file with sensor macros -->
-  <xacro:include filename="$(find uuv_sensor_ros_plugins)/urdf/sensor_snippets.xacro"/>
-  <!-- Loading the UUV simulator ROS plugin macros -->
-  <xacro:include filename="$(find uuv_gazebo_ros_plugins)/urdf/snippets.xacro"/>  <!-- Don't take it out or it won't work  -->
-  <!-- Loading vehicle's specific macros -->
-  <!-- <xacro:include filename="$(find vtec_u3_description)/urdf/snippets.xacro"/> -->
+  <!-- <xacro:include filename="$(find uuv_sensor_ros_plugins)/urdf/sensor_snippets.xacro"/> -->
   <!--
     Vehicle's parameters (remember to enter the model parameters below)
@@ -16,6 +12,4 @@
   <xacro:property name="cog" value="0 0 0"/> <!-- At the quasi geometric center -> we'll take it as the COG-->
   <xacro:property name="geocenter" value="-0.0069 -0.00909 -0.01005"/>
-  <!-- Fluid density -->
-  <!-- <xacro:property name="rho" value="1000"/> -->
   <!--
     Visual mesh file for the vehicle, usually in DAE (Collada) format. Be sure to store the
@@ -65,7 +59,6 @@
       <selfCollide>0</selfCollide>
       <turnGravityOff>1</turnGravityOff>
-    </gazebo>
-    <gazebo>
-      <plugin name="sixDOFMov" filename="libsixDOFMov.so">
+      <!-- CUSTOM PLUG-IN -->
+      <!-- <plugin name="sixDOFMov" filename="libsixDOFMov.so">
         <commandTopic>/uuv_desired_velocity</commandTopic>
         <odometryTopic>odom</odometryTopic>
@@ -74,10 +67,6 @@
         <robotBaseFrame>${namespace}/base_link</robotBaseFrame>
         <publishTF>false</publishTF>
-      </plugin>
+      </plugin> -->
     </gazebo>
-    <!-- Set up hydrodynamic plugin given as input parameter -->
-    <!-- <xacro:insert_block name="gazebo"/> -->
-    <!-- Include the thruster modules -->
-    <!-- <xacro:include filename="$(find vtec_u3_description)/urdf/actuators.xacro"/> -->
     <!-- Include the sensor modules -->
     <xacro:include filename="$(find vtec_u3_description)/urdf/sensors.xacro"/>

File: vtec_u3_description/urdf/sensors.xacro (robot description, xacro)
@@ -31,19 +31,18 @@
     <origin xyz="0.08992 0.00853 0.05671" rpy="0 0 0"/>
   </xacro:default_imu>
+  <!-- Realsense R200 -->
+  <!-- Import macro for realsense-RS200 camera-->
+  <xacro:include filename="$(find realsense_gazebo_plugin)/urdf/realsense-RS200.macro.xacro"/>
+  <!-- Create camera instance -->
+  <xacro:realsense-rs200 prefix="" parent="${namespace}/base_link">
+    <origin xyz="0.19281 0.01961 0.06659" rpy="0 0 0"/>
+  </xacro:realsense-rs200>
   <!-- Mount a camera  -->
-  <xacro:default_camera namespace="${namespace}" parent_link="${namespace}/base_link" suffix="">
+  <!-- <xacro:default_camera namespace="${namespace}" parent_link="${namespace}/base_link" suffix="">
     <origin xyz="0.19281 0.01961 0.06659" rpy="0 0 0"/>
-  </xacro:default_camera>
+  </xacro:default_camera> -->
   <!-- Mount base torpedos  -->
-  <xacro:base_torpedos namespace="${namespace}" parent_link="${namespace}/base_link" suffix="">
+  <!-- <xacro:base_torpedos namespace="${namespace}" parent_link="${namespace}/base_link" suffix="">
     <origin xyz="0.1031 0.022 0.21" rpy="0 0 -1.5757"/>
-  </xacro:base_torpedos>
-  <!-- Mount torpedo1  -->
-  <!-- <xacro:torpedo1 namespace="${namespace}" parent_link="${namespace}/base_link" suffix="">
-    <origin xyz="0.27781 0.01961 -0.16659" rpy="0 0 0"/>
-  </xacro:torpedo1>-->
-  <!-- Mount torpedo2  -->
-  <!--<xacro:torpedo2 namespace="${namespace}" parent_link="${namespace}/base_link" suffix="">
-    <origin xyz="0.10781 0.01961 -0.16659" rpy="0 0 0"/>
-  </xacro:torpedo2>-->
+  </xacro:base_torpedos> -->
 </robot>

Commit message: cambios cambios

File: vtec_u3_description/urdf/base.xacro (robot description, xacro)
@@ -39,12 +39,13 @@
                    izz="0.64879823" /> -->
           <!-- For COM nearly in geometric center -->
-            <inertia ixx="0.83639798529" ixy="-0.00503680373" ixz="0.0560001532"
+            <!-- inertia ixx="0.83639798529" ixy="-0.00503680373" ixz="0.0560001532"
                       iyy="0.46118483068" iyz="-0.01377965358"
-                      izz="1.02986207702" />
+                      izz="1.02986207702" /-->
         </inertial>
         <visual>
           <origin xyz="${geocenter}" rpy="0 0 0"/>
           <geometry>
-            <mesh filename="${visual_mesh_file}" scale="0.001 0.001 0.001" />
+            <box size= "0.6 0.6 0.6"/>
+            <!-- mesh filename="${visual_mesh_file}" scale="0.001 0.001 0.001" /-->
           </geometry>
         </visual>

File: vtec_u3_description/urdf/sensors.xacro (robot description, xacro)
@@ -35,8 +35,8 @@
     <origin xyz="0.19281 0.01961 0.06659" rpy="0 0 0"/>
   </xacro:realsense_camera>
-  <!-- Realsense R200 -->
+  <!-- Realsense R200 - ->
   <xacro:realsense_camera namespace="${namespace}" parent_link="${namespace}/base_link" suffix="down">
     <origin xyz="2.19281 0.01961 0.06659" rpy="0 1.57 0"/>
-  </xacro:realsense_camera>
+  </xacro:realsense_camera-->
   <!-- Realsense R200 -->
   <!-- Import macro for realsense-RS200 camera-->

Commit message: working

File: vtec_u3_description/urdf/base.xacro (robot description, xacro)
@@ -44,5 +44,5 @@
         </inertial>
         <visual>
-          <origin xyz="${geocenter}" rpy="0 0 0"/>
+          <origin xyz="${geocenter}" rpy="0 1.57 0"/>
           <geometry>
             <box size= "0.6 0.6 0.6"/>
