Commit message: Changed size of target

File: props_gazebo/urdf/gman.xacro (robot description, xacro)
@@ -7,5 +7,5 @@
             <origin xyz="0.0 0.0 0.23" rpy="0.0 0.0 0.0"/>
             <geometry>
-                <mesh filename="${visual_mesh_file}" scale="0.5 0.5 0.5"/>
+                <mesh filename="${visual_mesh_file}" scale="0.3 0.3 0.3"/>
             </geometry>
         </visual>
@@ -13,5 +13,5 @@
             <origin xyz="0 0 0.23" rpy="0 0 0"/>
             <geometry>
-                <mesh filename="${visual_mesh_file}" scale="0.5 0.5 0.5"/>
+                <mesh filename="${visual_mesh_file}" scale="0.3 0.3 0.3"/>
             </geometry>
         </collision>
