Commit message: Different group torpedos

File: shooter_description/urdf/torpedoes.xacro (robot description, xacro)
@@ -4,5 +4,5 @@
 <xacro:include filename="$(find shooter_description)/urdf/macro_torpedoes.xacro"/>
 <xacro:macro_torpedoes id="1">
-  <origin xyz="0.085 0 0" rpy="0.0 0.0 1.5757"/>
+  <origin xyz="0.27781 0.01961 -2.16659" rpy="0.0 0.0 1.5757"/>
 </xacro:macro_torpedoes>
 <gazebo>

File: shooter_description/urdf/torpedoes_1.xacro (robot description, xacro)
@@ -5,5 +5,5 @@
 <xacro:macro_torpedoes id="2">
   <!--<origin xyz="-0.085 0 0" rpy="0.0 0.0 1.5757"/>-->
-  <origin xyz="-0.085 0 0" rpy="0.0 0.0 1.5757"/>
+  <origin xyz="0.10781 0.01961 -2.16659" rpy="0.0 0.0 1.5757"/>
 </xacro:macro_torpedoes>
 <gazebo>

File: vtec_u3_description/urdf/sensors.xacro (robot description, xacro)
@@ -40,10 +40,10 @@
   </xacro:base_torpedos>
   <!-- Mount torpedo1  -->
-  <xacro:torpedo1 namespace="${namespace}" parent_link="${namespace}/base_link" suffix="">
+  <!-- <xacro:torpedo1 namespace="${namespace}" parent_link="${namespace}/base_link" suffix="">
     <origin xyz="0.27781 0.01961 -0.16659" rpy="0 0 0"/>
-  </xacro:torpedo1>
+  </xacro:torpedo1>-->
   <!-- Mount torpedo2  -->
-  <xacro:torpedo2 namespace="${namespace}" parent_link="${namespace}/base_link" suffix="">
+  <!--<xacro:torpedo2 namespace="${namespace}" parent_link="${namespace}/base_link" suffix="">
     <origin xyz="0.10781 0.01961 -0.16659" rpy="0 0 0"/>
-  </xacro:torpedo2>
+  </xacro:torpedo2>-->
 </robot>
