Commit message: Tasks ready

File: uuv_world/urdf/bin1.xacro (robot description, xacro)
@@ -4,7 +4,7 @@
 <xacro:property name="visual_mesh_file" value="file://$(find uuv_world)/models/meshes/bin.dae" />
 <!-- <origin xyz="0.085 (0 -0.085) 0 0" rpy="0.0 0.0 1.57075"/> -->
-<link name="gate_base">
+<link name="bin1_base">
     <visual>
-        <origin xyz="0.0 0.0 0.23" rpy="0.0 0.0 0.0"/>
+        <origin xyz="22.180420 -2.960028 -4.0" rpy="0.0 0.0 -1.57"/>
         <geometry>
             <mesh filename="${visual_mesh_file}" scale="1 1 1" />
@@ -13,5 +13,5 @@
         <!-- Se deben cambiar los parametros reales-->
     <collision>
-      <origin xyz="0.0 0.0 0.23" rpy="0.0 0.0 0.0"/>
+      <origin xyz="22.180420 -2.960028 -4.0" rpy="0.0 0.0 -1.57"/>
       <geometry>
         <mesh filename="${visual_mesh_file}" scale="1 1 1" />
@@ -19,5 +19,5 @@
     </collision>
     <inertial>
-      <origin xyz="0.0 0.0 0.23" rpy="0.0 0.0 0.0"/>
+      <origin xyz="22.180420 -2.960028 -4.0" rpy="0.0 0.0 -1.57"/>
       <mass value="1"/>
       <inertia

File: uuv_world/urdf/bin2.xacro (robot description, xacro)
@@ -4,7 +4,7 @@
 <xacro:property name="visual_mesh_file" value="file://$(find uuv_world)/models/meshes/bin02.dae" />
 <!-- <origin xyz="0.085 (0 -0.085) 0 0" rpy="0.0 0.0 1.57075"/> -->
-<link name="gate_base">
+<link name="bin2_base">
     <visual>
-        <origin xyz="0.0 0.0 0.23" rpy="0.0 0.0 0.0"/>
+        <origin xyz="22.180420 4.643661 -4.0" rpy="0.0 0.0 -1.57"/>
         <geometry>
             <mesh filename="${visual_mesh_file}" scale="1 1 1" />
@@ -13,5 +13,5 @@
         <!-- Se deben cambiar los parametros reales-->
     <collision>
-      <origin xyz="0.0 0.0 0.23" rpy="0.0 0.0 0.0"/>
+      <origin xyz="22.180420 4.643661 -4.0" rpy="0.0 0.0 -1.57"/>
       <geometry>
         <mesh filename="${visual_mesh_file}" scale="1 1 1" />
@@ -19,5 +19,5 @@
     </collision>
     <inertial>
-      <origin xyz="0.0 0.0 0.23" rpy="0.0 0.0 0.0"/>
+      <origin xyz="22.180420 4.643661 -4.0" rpy="0.0 0.0 -1.57"/>
       <mass value="1"/>
       <inertia

File: uuv_world/urdf/buoy.xacro (robot description, xacro)
@@ -4,7 +4,7 @@
 <xacro:property name="visual_mesh_file" value="file://$(find uuv_world)/models/meshes/buoy1.dae" />
 <!-- <origin xyz="0.085 (0 -0.085) 0 0" rpy="0.0 0.0 1.57075"/> -->
-<link name="gate_base">
+<link name="buoy1_base">
     <visual>
-        <origin xyz="0.0 0.0 0.23" rpy="0.0 0.0 0.0"/>
+        <origin xyz="14.349550 -1.744834 -3.126359" rpy="0.0 0.0 1.57"/>
         <geometry>
             <mesh filename="${visual_mesh_file}" scale="1 1 1" />
@@ -13,5 +13,5 @@
         <!-- Se deben cambiar los parametros reales-->
     <collision>
-      <origin xyz="0.0 0.0 0.23" rpy="0.0 0.0 0.0"/>
+      <origin xyz="14.349550 -1.744834 -3.126359" rpy="0.0 0.0 1.57"/>
       <geometry>
         <mesh filename="${visual_mesh_file}" scale="1 1 1" />
@@ -19,5 +19,5 @@
     </collision>
     <inertial>
-      <origin xyz="0.0 0.0 0.23" rpy="0.0 0.0 0.0"/>
+      <origin xyz="14.349550 -1.744834 -3.126359" rpy="0.0 0.0 1.57"/>
       <mass value="1"/>
       <inertia

File: uuv_world/urdf/buoy2.xacro (robot description, xacro)
@@ -4,7 +4,7 @@
 <xacro:property name="visual_mesh_file" value="file://$(find uuv_world)/models/meshes/buoy2.dae" />
 <!-- <origin xyz="0.085 (0 -0.085) 0 0" rpy="0.0 0.0 1.57075"/> -->
-<link name="gate_base">
+<link name="buoy2_base">
     <visual>
-        <origin xyz="0.0 0.0 0.23" rpy="0.0 0.0 0.0"/>
+        <origin xyz="14.349550 -0.497678 -3.126359" rpy="0.0 0.0 1.57"/>
         <geometry>
             <mesh filename="${visual_mesh_file}" scale="1 1 1" />
@@ -13,5 +13,5 @@
         <!-- Se deben cambiar los parametros reales-->
     <collision>
-      <origin xyz="0.0 0.0 0.23" rpy="0.0 0.0 0.0"/>
+      <origin xyz="14.349550 -0.497678 -3.126359" rpy="0.0 0.0 1.57"/>
       <geometry>
         <mesh filename="${visual_mesh_file}" scale="1 1 1" />
@@ -19,5 +19,5 @@
     </collision>
     <inertial>
-      <origin xyz="0.0 0.0 0.23" rpy="0.0 0.0 0.0"/>
+      <origin xyz="14.349550 -0.497678 -3.126359" rpy="0.0 0.0 1.57"/>
       <mass value="1"/>
       <inertia

File: uuv_world/urdf/octagon.xacro (robot description, xacro)
@@ -4,7 +4,7 @@
 <xacro:property name="visual_mesh_file" value="file://$(find uuv_world)/models/meshes/MyOctagon.dae" />
 <!-- <origin xyz="0.085 (0 -0.085) 0 0" rpy="0.0 0.0 1.57075"/> -->
-<link name="gate_base">
+<link name="octagon_base">
     <visual>
-        <origin xyz="0.0 0.0 0.23" rpy="0.0 0.0 0.0"/>
+        <origin xyz="28.593435 -0.004454 -4.0" rpy="0.0 0.0 1.57"/>
         <geometry>
             <mesh filename="${visual_mesh_file}" scale="1 1 1" />
@@ -13,5 +13,5 @@
         <!-- Se deben cambiar los parametros reales-->
     <collision>
-      <origin xyz="0.0 0.0 0.23" rpy="0.0 0.0 0.0"/>
+      <origin xyz="28.593435 -0.004454 -4.0" rpy="0.0 0.0 1.57"/>
       <geometry>
         <mesh filename="${visual_mesh_file}" scale="1 1 1" />
@@ -19,5 +19,5 @@
     </collision>
     <inertial>
-      <origin xyz="0.0 0.0 0.23" rpy="0.0 0.0 0.0"/>
+      <origin xyz="28.593435 -0.004454 -4.0" rpy="0.0 0.0 1.57"/>
       <mass value="1"/>
       <inertia

File: uuv_world/urdf/torpedos1.xacro (robot description, xacro)
@@ -1,10 +1,10 @@
 <?xml version="1.0"?>
-<robot name="gate_1" xmlns:xacro="http://www.ros.org/wiki/xacro">
+<robot name="torpedos_1" xmlns:xacro="http://www.ros.org/wiki/xacro">
 <!-- Introducir meshes -->
-<xacro:property name="visual_mesh_file" value="file://$(find uuv_world)/models/meshes/Gate.dae" />
+<xacro:property name="visual_mesh_file" value="file://$(find uuv_world)/models/meshes/Mytorpedo1.dae" />
 <!-- <origin xyz="0.085 (0 -0.085) 0 0" rpy="0.0 0.0 1.57075"/> -->
-<link name="gate_base">
+<link name="torpedos1_base">
     <visual>
-        <origin xyz="7.526688 -1.294371 -1.583826" rpy="0.0 0.0 1.57"/>
+        <origin xyz="25.180420 1.835166 -4.0" rpy="0.0 0.0 1.57"/>
         <geometry>
             <mesh filename="${visual_mesh_file}" scale="1 1 1" />
@@ -13,5 +13,5 @@
         <!-- Se deben cambiar los parametros reales-->
     <collision>
-      <origin xyz="7.526688 -1.294371 -1.583826" rpy="0.0 0.0 1.57"/>
+      <origin xyz="25.180420 1.835166 -4.0" rpy="0.0 0.0 1.57"/>
       <geometry>
         <mesh filename="${visual_mesh_file}" scale="1 1 1" />
@@ -19,5 +19,5 @@
     </collision>
     <inertial>
-      <origin xyz="7.526688 -1.294371 -1.583826" rpy="0.0 0.0 1.57"/>
+      <origin xyz="25.180420 1.835166 -4.0" rpy="0.0 0.0 1.57"/>
       <mass value="1"/>
       <inertia

File: uuv_world/urdf/torpedos2.xacro (robot description, xacro)
@@ -1,10 +1,10 @@
 <?xml version="1.0"?>
-<robot name="gate_1" xmlns:xacro="http://www.ros.org/wiki/xacro">
+<robot name="torpedos_2" xmlns:xacro="http://www.ros.org/wiki/xacro">
 <!-- Introducir meshes -->
-<xacro:property name="visual_mesh_file" value="file://$(find uuv_world)/models/meshes/Gate.dae" />
+<xacro:property name="visual_mesh_file" value="file://$(find uuv_world)/models/meshes/Mytorpedos2.dae" />
 <!-- <origin xyz="0.085 (0 -0.085) 0 0" rpy="0.0 0.0 1.57075"/> -->
-<link name="gate_base">
+<link name="torpedos2_base">
     <visual>
-        <origin xyz="7.526688 -1.294371 -1.583826" rpy="0.0 0.0 1.57"/>
+        <origin xyz="25.180420 3.082322 -4.0" rpy="0.0 0.0 1.57"/>
         <geometry>
             <mesh filename="${visual_mesh_file}" scale="1 1 1" />
@@ -13,5 +13,5 @@
         <!-- Se deben cambiar los parametros reales-->
     <collision>
-      <origin xyz="7.526688 -1.294371 -1.583826" rpy="0.0 0.0 1.57"/>
+      <origin xyz="25.180420 3.082322 -4.0" rpy="0.0 0.0 1.57"/>
       <geometry>
         <mesh filename="${visual_mesh_file}" scale="1 1 1" />
@@ -19,5 +19,5 @@
     </collision>
     <inertial>
-      <origin xyz="7.526688 -1.294371 -1.583826" rpy="0.0 0.0 1.57"/>
+      <origin xyz="25.180420 3.082322 -4.0" rpy="0.0 0.0 1.57"/>
       <mass value="1"/>
       <inertia
