Commit message: Added LiDAR VLP-16 and IMU

File: vtec_s3_description/robots/vtec_s3_default.xacro (robot description, xacro)
@@ -3,5 +3,5 @@
   <xacro:arg name="debug" default="0"/>
   <xacro:arg name="namespace" default="vtec_s3"/>
-  <xacro:arg name="inertial_reference_frame" default="map"/>
+  <xacro:arg name="inertial_reference_frame" default="world_ned"/>
   <!-- Include the USV macro file -->
   <xacro:include filename="$(find vtec_s3_description)/urdf/base.xacro"/>

File: vtec_s3_description/urdf/base.xacro (robot description, xacro)
@@ -2,5 +2,5 @@
 <robot xmlns:xacro="http://www.ros.org/wiki/xacro">
   <!-- Loading file with sensor macros -->
-  <!-- <xacro:include filename="$(find uuv_sensor_ros_plugins)/urdf/sensor_snippets.xacro"/> -->
+  <xacro:include filename="$(find sensor_plugins)/sensor_ros_plugins/urdf/sensor_snippets.xacro"/>
   <!--
     Vehicle's parameters (remember to enter the model parameters below)
@@ -63,5 +63,5 @@
     </gazebo>
     <!-- Include the sensor modules -->
-    <!-- <xacro:include filename="$(find vtec_s3_description)/urdf/sensors.xacro"/> -->
+    <xacro:include filename="$(find vtec_s3_description)/urdf/sensors.xacro"/>
   </xacro:macro>
 </robot>

File: vtec_s3_description/urdf/sensors.xacro (robot description, xacro)
@@ -8,30 +8,35 @@
   -->
   <!-- Mount a GPS. -->
-  <xacro:default_gps namespace="${namespace}" parent_link="${namespace}/base_link" />
+  <!-- <xacro:default_gps namespace="${namespace}" parent_link="${namespace}/base_link" /> -->
   <!-- Mount a Pose 3D sensor. -->
-  <xacro:default_pose_3d namespace="${namespace}" parent_link="${namespace}/base_link" />
+  <!-- <xacro:default_pose_3d namespace="${namespace}" parent_link="${namespace}/base_link" /> -->
   <!-- Forward-looking sonar sensor -->
-  <xacro:forward_multibeam_p900 namespace="${namespace}" parent_link="${namespace}/base_link">
+  <!-- <xacro:forward_multibeam_p900 namespace="${namespace}" parent_link="${namespace}/base_link">
     <origin xyz="0 0 0" rpy="0 0 0"/>
-  </xacro:forward_multibeam_p900>
+  </xacro:forward_multibeam_p900> -->
   <!-- DVL  -->
-  <xacro:default_dvl namespace="${namespace}" parent_link="${namespace}/base_link">
+  <!-- <xacro:default_dvl namespace="${namespace}" parent_link="${namespace}/base_link">
     <origin xyz="0 0 0" rpy="0 0 0"/>
-  </xacro:default_dvl>
+  </xacro:default_dvl> -->
   <!-- RPT  -->
-  <xacro:default_rpt namespace="${namespace}" parent_link="${namespace}/base_link">
+  <!-- <xacro:default_rpt namespace="${namespace}" parent_link="${namespace}/base_link">
     <origin xyz="0 0 0" rpy="0 0 0"/>
-  </xacro:default_rpt>
+  </xacro:default_rpt> -->
   <!-- Pressure  -->
-  <xacro:default_pressure namespace="${namespace}" parent_link="${namespace}/base_link">
+  <!-- <xacro:default_pressure namespace="${namespace}" parent_link="${namespace}/base_link">
     <origin xyz="0 0 0" rpy="0 0 0"/>
-  </xacro:default_pressure>
+  </xacro:default_pressure> -->
   <!-- IMU  -->
   <xacro:default_imu namespace="${namespace}" parent_link="${namespace}/base_link">
     <origin xyz="0 0 0" rpy="0 0 0"/>
   </xacro:default_imu>
+  <!-- LiDAR VLP-16 -->
+  <xacro:include filename="$(find velodyne_description)/urdf/VLP-16.urdf.xacro"/>
+  <VLP-16 parent="${namespace}/base_link" name="velodyne" topic="/velodyne_points" hz="10" samples="440" gpu="0">
+    <origin xyz="0 0 0.4" rpy="0 0 0" />
+  </VLP-16>
   <!-- Mount a camera  -->
-  <xacro:default_camera namespace="${namespace}" parent_link="${namespace}/base_link" suffix="">
+  <!-- <xacro:default_camera namespace="${namespace}" parent_link="${namespace}/base_link" suffix="">
     <origin xyz="0 0 0" rpy="0 0 0"/>
-  </xacro:default_camera>
+  </xacro:default_camera> -->
 </robot>
