Commit message: USV ready with sensors

File: sensor_plugins/sensor_ros_plugins/urdf/imu_snippets.xacro (robot description, xacro)
@@ -131,5 +131,4 @@
     </link>
     <gazebo reference="${namespace}/imu${imu_suffix}_link">
-      <selfCollide>0</selfCollide>
       <turnGravityOff>1</turnGravityOff>
     </gazebo>

File: vtec_s3_description/urdf/base.xacro (robot description, xacro)
@@ -21,9 +21,9 @@
     Open the meshes for the RexROV vehicle in Blender to see an example on the mesh placement.
   -->
-  <xacro:property name="visual_mesh_file" value="file://$(find vtec_s3_description)/meshes/VTECSIII_NOPROP.dae"/>
+  <xacro:property name="visual_mesh_file" value="file://$(find vtec_s3_description)/meshes/vtec_s3.dae"/>
   <!-- Collision geometry mesh, usually in STL format (it is recommended to keep
   this geometry as simple as possible to improve the performance the physics engine
   regarding the computation of collision forces) -->
-  <xacro:property name="collision_mesh_file" value="file://$(find vtec_s3_description)/meshes/VTECSIII_NOPROP.stl"/>
+  <xacro:property name="collision_mesh_file" value="file://$(find vtec_s3_description)/meshes/vtec_s3.stl"/>
   <!-- Vehicle macro -->
   <xacro:macro name="vtec_s3_base" params="namespace *gazebo">

File: vtec_s3_description/urdf/sensors.xacro (robot description, xacro)
@@ -34,6 +34,13 @@
   <xacro:include filename="$(find velodyne_description)/urdf/VLP-16.urdf.xacro"/>
   <VLP-16 parent="${namespace}/base_link" name="velodyne" topic="/velodyne_points" hz="10" samples="440" gpu="0">
-    <origin xyz="0 0 0.4" rpy="0 0 0" />
+    <origin xyz="0.25 0 0.38" rpy="0 0 0" />
   </VLP-16>
+  <!-- Realsense R200 -->
+  <!-- Import macro for realsense-RS200 camera-->
+  <xacro:include filename="$(find realsense_gazebo_plugin)/urdf/realsense-RS200.macro.xacro"/>
+  <!-- Create camera instance -->
+  <xacro:realsense-rs200 prefix="" parent="${namespace}/base_link">
+      <origin xyz="0.52 0 0.22" rpy="0 0 0" />
+  </xacro:realsense-rs200>
   <!-- Mount a camera  -->
   <!-- <xacro:default_camera namespace="${namespace}" parent_link="${namespace}/base_link" suffix="">
