Commit message: Point clouds fixed

File: sensors/sensor_plugins/sensor_ros_plugins/urdf/sensor_snippets.xacro (robot description, xacro)
@@ -17,4 +17,5 @@
   <xacro:include filename="$(find sensor_plugins)/sensor_ros_plugins/urdf/pressure_snippets.xacro" />
   <xacro:include filename="$(find sensor_plugins)/sensor_ros_plugins/urdf/camera_snippets.xacro" />
+  <xacro:include filename="$(find sensor_plugins)/sensor_ros_plugins/urdf/realsense_camera.xacro" />
   <xacro:include filename="$(find sensor_plugins)/sensor_ros_plugins/urdf/dvl_snippets.xacro" />
   <xacro:include filename="$(find sensor_plugins)/sensor_ros_plugins/urdf/rpt_snippets.xacro" />

File: vtec_s3_description/urdf/sensors.xacro (robot description, xacro)
@@ -37,10 +37,7 @@
   </VLP-16>
   <!-- Realsense R200 -->
-  <!-- Import macro for realsense-RS200 camera-->
-  <xacro:include filename="$(find realsense_gazebo_plugin)/urdf/realsense-RS200.macro.xacro"/>
-  <!-- Create camera instance -->
-  <xacro:realsense-rs200 prefix="" parent="${namespace}/base_link">
-      <origin xyz="0.52 0 0.22" rpy="0 0 0" />
-  </xacro:realsense-rs200>
+  <xacro:realsense_camera namespace="${namespace}" parent_link="${namespace}/base_link" suffix="">
+    <origin xyz="0.52 0 0.22" rpy="0 0 0"/>
+  </xacro:realsense_camera>
   <!-- Mount a camera  -->
   <!-- <xacro:default_camera namespace="${namespace}" parent_link="${namespace}/base_link" suffix="">
