Commit message: missing just path marker

File: sim_challenges/urdf/gate.xacro (robot description, xacro)
@@ -2,5 +2,5 @@
 <robot name="gate_1" xmlns:xacro="http://www.ros.org/wiki/xacro">
 <!-- Introducir meshes -->
-<xacro:property name="visual_mesh_file" value="file://$(find sim_challenges)/models/meshes/Gate.dae" />
+<xacro:property name="visual_mesh_file" value="file://$(find sim_challenges)/models/meshes/mygate1.dae" />
 <!-- <origin xyz="0.085 (0 -0.085) 0 0" rpy="0.0 0.0 1.57075"/> -->
 <link name="gate_base">

File: sim_challenges/urdf/octagon.xacro (robot description, xacro)
@@ -2,5 +2,5 @@
 <robot name="octagon_1" xmlns:xacro="http://www.ros.org/wiki/xacro">
 <!-- Introducir meshes -->
-<xacro:property name="visual_mesh_file" value="file://$(find sim_challenges)/models/meshes/MyOctagon.dae" />
+<xacro:property name="visual_mesh_file" value="file://$(find sim_challenges)/models/meshes/Myoctagon2.dae" />
 <!-- <origin xyz="0.085 (0 -0.085) 0 0" rpy="0.0 0.0 1.57075"/> -->
 <link name="octagon_base">

Commit message: uploaded gate and octagon.xacro

File: sim_challenges/urdf/gate.xacro (robot description, xacro)
@@ -2,9 +2,9 @@
 <robot name="gate_1" xmlns:xacro="http://www.ros.org/wiki/xacro">
 <!-- Introducir meshes -->
-<xacro:property name="visual_mesh_file" value="file://$(find sim_challenges)/models/meshes/Gate.dae" />
+<xacro:property name="visual_mesh_file" value="file://$(find sim_challenges)/models/meshes/mygate1.dae" />
 <!-- <origin xyz="0.085 (0 -0.085) 0 0" rpy="0.0 0.0 1.57075"/> -->
 <link name="gate_base">
     <visual>
-        <origin xyz="7.00 0 -22.0" rpy="0.0 0.0 1.57"/>
+        <origin xyz="0 0 -4" rpy="0.0 0.0 1.57"/>
         <geometry>
             <mesh filename="${visual_mesh_file}" scale="1 1 1" />
@@ -13,5 +13,5 @@
         <!-- Se deben cambiar los parametros reales-->
     <collision>
-      <origin xyz="7.00 0 -22.0" rpy="0.0 0.0 1.57"/>
+      <origin xyz="0 0 -4" rpy="0.0 0.0 1.57"/>
       <geometry>
         <mesh filename="${visual_mesh_file}" scale="1 1 1" />
@@ -19,5 +19,5 @@
     </collision>
     <inertial>
-      <origin xyz="7.00 0 -22.0" rpy="0.0 0.0 1.57"/>
+      <origin xyz="0 0 -4" rpy="0.0 0.0 1.57"/>
       <mass value="1"/>
       <inertia

File: sim_challenges/urdf/octagon.xacro (robot description, xacro)
@@ -2,9 +2,9 @@
 <robot name="octagon_1" xmlns:xacro="http://www.ros.org/wiki/xacro">
 <!-- Introducir meshes -->
-<xacro:property name="visual_mesh_file" value="file://$(find sim_challenges)/models/meshes/MyOctagon.dae" />
+<xacro:property name="visual_mesh_file" value="file://$(find sim_challenges)/models/meshes/Myoctagon2.dae" />
 <!-- <origin xyz="0.085 (0 -0.085) 0 0" rpy="0.0 0.0 1.57075"/> -->
 <link name="octagon_base">
     <visual>
-        <origin xyz="28.593435 -0.004454 -4.0" rpy="0.0 0.0 1.57"/>
+        <origin xyz="0 0 -4" rpy="0.0 0.0 1.57"/>
         <geometry>
             <mesh filename="${visual_mesh_file}" scale="1 1 1" />
@@ -13,5 +13,5 @@
         <!-- Se deben cambiar los parametros reales-->
     <collision>
-      <origin xyz="28.593435 -0.004454 -4.0" rpy="0.0 0.0 1.57"/>
+      <origin xyz="0 0 -4" rpy="0.0 0.0 1.57"/>
       <geometry>
         <mesh filename="${visual_mesh_file}" scale="1 1 1" />
@@ -19,5 +19,5 @@
     </collision>
     <inertial>
-      <origin xyz="28.593435 -0.004454 -4.0" rpy="0.0 0.0 1.57"/>
+      <origin xyz="0 0 -4" rpy="0.0 0.0 1.57"/>
       <mass value="1"/>
       <inertia
