Commit message: Cambios cambios

File: sim_challenges/urdf/buoy.xacro (robot description, xacro)
@@ -1,4 +1,5 @@
 <?xml version="1.0"?>
 <robot name="buoy_1" xmlns:xacro="http://www.ros.org/wiki/xacro">
+<!-- GUN -->
 <!-- Introducir meshes -->
 <xacro:property name="visual_mesh_file" value="file://$(find sim_challenges)/models/meshes/buoy1.dae" />
@@ -6,5 +7,5 @@
 <link name="buoy1_base">
     <visual>
-        <origin xyz="14.349550 -1.744834 -3.126359" rpy="0.0 0.0 1.57"/>
+        <origin xyz="7.00 0 -3.0" rpy="0.0 0.0 1.57"/>
         <geometry>
             <mesh filename="${visual_mesh_file}" scale="1 1 1" />
@@ -13,5 +14,5 @@
         <!-- Se deben cambiar los parametros reales-->
     <collision>
-      <origin xyz="14.349550 -1.744834 -3.126359" rpy="0.0 0.0 1.57"/>
+      <origin xyz="7.00 0 -3.0" rpy="0.0 0.0 1.57"/>
       <geometry>
         <mesh filename="${visual_mesh_file}" scale="1 1 1" />
@@ -19,5 +20,5 @@
     </collision>
     <inertial>
-      <origin xyz="14.349550 -1.744834 -3.126359" rpy="0.0 0.0 1.57"/>
+      <origin xyz="7.00 0 -3.0" rpy="0.0 0.0 1.57"/>
       <mass value="1"/>
       <inertia

File: sim_challenges/urdf/buoy2.xacro (robot description, xacro)
@@ -1,4 +1,5 @@
 <?xml version="1.0"?>
 <robot name="buoy_2" xmlns:xacro="http://www.ros.org/wiki/xacro">
+<!-- Badge -->
 <!-- Introducir meshes -->
 <xacro:property name="visual_mesh_file" value="file://$(find sim_challenges)/models/meshes/buoy2.dae" />
@@ -6,5 +7,5 @@
 <link name="buoy2_base">
     <visual>
-        <origin xyz="14.349550 -0.497678 -3.126359" rpy="0.0 0.0 1.57"/>
+        <origin xyz="7.00 2 -3.0" rpy="0.0 0.0 1.57"/>
         <geometry>
             <mesh filename="${visual_mesh_file}" scale="1 1 1" />
@@ -13,5 +14,5 @@
         <!-- Se deben cambiar los parametros reales-->
     <collision>
-      <origin xyz="14.349550 -0.497678 -3.126359" rpy="0.0 0.0 1.57"/>
+      <origin xyz="7.00 2 -3.0" rpy="0.0 0.0 1.57"/>
       <geometry>
         <mesh filename="${visual_mesh_file}" scale="1 1 1" />
@@ -19,5 +20,5 @@
     </collision>
     <inertial>
-      <origin xyz="14.349550 -0.497678 -3.126359" rpy="0.0 0.0 1.57"/>
+      <origin xyz="7.00 2 -3.0" rpy="0.0 0.0 1.57"/>
       <mass value="1"/>
       <inertia

File: sim_challenges/urdf/gate.xacro (robot description, xacro)
@@ -6,5 +6,5 @@
 <link name="gate_base">
     <visual>
-        <origin xyz="0 0 -4" rpy="0.0 0.0 1.57"/>
+        <origin xyz="7.00 0 -3.0" rpy="0.0 0.0 1.57"/>
         <geometry>
             <mesh filename="${visual_mesh_file}" scale="1 1 1" />
@@ -13,5 +13,5 @@
         <!-- Se deben cambiar los parametros reales-->
     <collision>
-      <origin xyz="0 0 -4" rpy="0.0 0.0 1.57"/>
+      <origin xyz="7.00 0 -3.0" rpy="0.0 0.0 1.57"/>
       <geometry>
         <mesh filename="${visual_mesh_file}" scale="1 1 1" />
@@ -19,5 +19,5 @@
     </collision>
     <inertial>
-      <origin xyz="0 0 -4" rpy="0.0 0.0 1.57"/>
+      <origin xyz="7.00 0 -3.0" rpy="0.0 0.0 1.57"/>
       <mass value="1"/>
       <inertia
