Commit message: .

File: sim_challenges/urdf/octagon.xacro (robot description, xacro)
@@ -6,5 +6,5 @@
 <link name="octagon_base">
     <visual>
-        <origin xyz="0 0 -4" rpy="0.0 0.0 1.57"/>
+        <origin xyz="8 0 8" rpy="1.57 0 1.57"/>
         <geometry>
             <mesh filename="${visual_mesh_file}" scale="1 1 1" />
@@ -13,5 +13,5 @@
         <!-- Se deben cambiar los parametros reales-->
     <collision>
-      <origin xyz="0 0 -4" rpy="0.0 0.0 1.57"/>
+      <origin xyz="8 0 8" rpy="1.57 0.0 1.57"/>
       <geometry>
         <mesh filename="${visual_mesh_file}" scale="1 1 1" />
@@ -19,5 +19,5 @@
     </collision>
     <inertial>
-      <origin xyz="0 0 -4" rpy="0.0 0.0 1.57"/>
+      <origin xyz="8 0 8" rpy="1.57 0.0 1.57"/>
       <mass value="1"/>
       <inertia
