Commit message: missions ready to simulate with new repository

File: sim_challenges/urdf/bin1.xacro (robot description, xacro)
@@ -2,5 +2,5 @@
 <robot name="bin_1" xmlns:xacro="http://www.ros.org/wiki/xacro">
 <!-- Introducir meshes -->
-<xacro:property name="visual_mesh_file" value="file://$(find uuv_world)/models/meshes/bin.dae" />
+<xacro:property name="visual_mesh_file" value="file://$(find sim_challenges)/models/meshes/bin.dae" />
 <!-- <origin xyz="0.085 (0 -0.085) 0 0" rpy="0.0 0.0 1.57075"/> -->
 <link name="bin1_base">
@@ -27,3 +27,7 @@
     </inertial>
 </link>
+<gazebo reference="bin1_base">
+  <selfCollide>0</selfCollide>
+  <turnGravityOff>1</turnGravityOff>
+</gazebo>
 </robot>

File: sim_challenges/urdf/bin2.xacro (robot description, xacro)
@@ -2,5 +2,5 @@
 <robot name="bin_2" xmlns:xacro="http://www.ros.org/wiki/xacro">
 <!-- Introducir meshes -->
-<xacro:property name="visual_mesh_file" value="file://$(find uuv_world)/models/meshes/bin02.dae" />
+<xacro:property name="visual_mesh_file" value="file://$(find sim_challenges)/models/meshes/bin02.dae" />
 <!-- <origin xyz="0.085 (0 -0.085) 0 0" rpy="0.0 0.0 1.57075"/> -->
 <link name="bin2_base">
@@ -27,3 +27,7 @@
     </inertial>
 </link>
+<gazebo reference="bin2_base">
+  <selfCollide>0</selfCollide>
+  <turnGravityOff>1</turnGravityOff>
+</gazebo>
 </robot>

File: sim_challenges/urdf/buoy.xacro (robot description, xacro)
@@ -2,5 +2,5 @@
 <robot name="buoy_1" xmlns:xacro="http://www.ros.org/wiki/xacro">
 <!-- Introducir meshes -->
-<xacro:property name="visual_mesh_file" value="file://$(find uuv_world)/models/meshes/buoy1.dae" />
+<xacro:property name="visual_mesh_file" value="file://$(find sim_challenges)/models/meshes/buoy1.dae" />
 <!-- <origin xyz="0.085 (0 -0.085) 0 0" rpy="0.0 0.0 1.57075"/> -->
 <link name="buoy1_base">
@@ -27,3 +27,7 @@
     </inertial>
 </link>
+<gazebo reference="buoy1_base">
+  <selfCollide>0</selfCollide>
+  <turnGravityOff>1</turnGravityOff>
+</gazebo>
 </robot>

File: sim_challenges/urdf/buoy2.xacro (robot description, xacro)
@@ -2,5 +2,5 @@
 <robot name="buoy_2" xmlns:xacro="http://www.ros.org/wiki/xacro">
 <!-- Introducir meshes -->
-<xacro:property name="visual_mesh_file" value="file://$(find uuv_world)/models/meshes/buoy2.dae" />
+<xacro:property name="visual_mesh_file" value="file://$(find sim_challenges)/models/meshes/buoy2.dae" />
 <!-- <origin xyz="0.085 (0 -0.085) 0 0" rpy="0.0 0.0 1.57075"/> -->
 <link name="buoy2_base">
@@ -27,3 +27,7 @@
     </inertial>
 </link>
+<gazebo reference="buoy2_base">
+  <selfCollide>0</selfCollide>
+  <turnGravityOff>1</turnGravityOff>
+</gazebo>
 </robot>

File: sim_challenges/urdf/gate.xacro (robot description, xacro)
@@ -2,5 +2,5 @@
 <robot name="gate_1" xmlns:xacro="http://www.ros.org/wiki/xacro">
 <!-- Introducir meshes -->
-<xacro:property name="visual_mesh_file" value="file://$(find uuv_world)/models/meshes/Gate.dae" />
+<xacro:property name="visual_mesh_file" value="file://$(find sim_challenges)/models/meshes/Gate.dae" />
 <!-- <origin xyz="0.085 (0 -0.085) 0 0" rpy="0.0 0.0 1.57075"/> -->
 <link name="gate_base">
@@ -27,3 +27,7 @@
     </inertial>
 </link>
+<gazebo reference="gate_base">
+  <selfCollide>0</selfCollide>
+  <turnGravityOff>1</turnGravityOff>
+</gazebo>
 </robot>

File: sim_challenges/urdf/octagon.xacro (robot description, xacro)
@@ -2,5 +2,5 @@
 <robot name="octagon_1" xmlns:xacro="http://www.ros.org/wiki/xacro">
 <!-- Introducir meshes -->
-<xacro:property name="visual_mesh_file" value="file://$(find uuv_world)/models/meshes/MyOctagon.dae" />
+<xacro:property name="visual_mesh_file" value="file://$(find sim_challenges)/models/meshes/MyOctagon.dae" />
 <!-- <origin xyz="0.085 (0 -0.085) 0 0" rpy="0.0 0.0 1.57075"/> -->
 <link name="octagon_base">
@@ -27,3 +27,7 @@
     </inertial>
 </link>
+<gazebo reference="octagon_base">
+  <selfCollide>0</selfCollide>
+  <turnGravityOff>1</turnGravityOff>
+</gazebo>
 </robot>

File: sim_challenges/urdf/torpedos1.xacro (robot description, xacro)
@@ -2,5 +2,5 @@
 <robot name="torpedos_1" xmlns:xacro="http://www.ros.org/wiki/xacro">
 <!-- Introducir meshes -->
-<xacro:property name="visual_mesh_file" value="file://$(find uuv_world)/models/meshes/Mytorpedo1.dae" />
+<xacro:property name="visual_mesh_file" value="file://$(find sim_challenges)/models/meshes/Mytorpedo1.dae" />
 <!-- <origin xyz="0.085 (0 -0.085) 0 0" rpy="0.0 0.0 1.57075"/> -->
 <link name="torpedos1_base">
@@ -27,3 +27,7 @@
     </inertial>
 </link>
+<gazebo reference="torpedos1_base">
+  <selfCollide>0</selfCollide>
+  <turnGravityOff>1</turnGravityOff>
+</gazebo>
 </robot>

File: sim_challenges/urdf/torpedos2.xacro (robot description, xacro)
@@ -2,5 +2,5 @@
 <robot name="torpedos_2" xmlns:xacro="http://www.ros.org/wiki/xacro">
 <!-- Introducir meshes -->
-<xacro:property name="visual_mesh_file" value="file://$(find uuv_world)/models/meshes/Mytorpedos2.dae" />
+<xacro:property name="visual_mesh_file" value="file://$(find sim_challenges)/models/meshes/Mytorpedos2.dae" />
 <!-- <origin xyz="0.085 (0 -0.085) 0 0" rpy="0.0 0.0 1.57075"/> -->
 <link name="torpedos2_base">
@@ -27,3 +27,7 @@
     </inertial>
 </link>
+<gazebo reference="torpedos2_base">
+  <selfCollide>0</selfCollide>
+  <turnGravityOff>1</turnGravityOff>
+</gazebo>
 </robot>

Commit message: Task2021

File: sim_challenges/urdf/bin1.xacro (robot description, xacro)
@@ -6,5 +6,5 @@
 <link name="bin1_base">
     <visual>
-        <origin xyz="22.180420 -2.960028 -4.0" rpy="0.0 0.0 -1.57"/>
+        <origin xyz="0 0 0" rpy="0.0 0.0 -1.57"/>
         <geometry>
             <mesh filename="${visual_mesh_file}" scale="1 1 1" />
@@ -13,5 +13,5 @@
         <!-- Se deben cambiar los parametros reales-->
     <collision>
-      <origin xyz="22.180420 -2.960028 -4.0" rpy="0.0 0.0 -1.57"/>
+      <origin xyz="0 0 0" rpy="0.0 0.0 -1.57"/>
       <geometry>
         <mesh filename="${visual_mesh_file}" scale="1 1 1" />
@@ -19,5 +19,5 @@
     </collision>
     <inertial>
-      <origin xyz="22.180420 -2.960028 -4.0" rpy="0.0 0.0 -1.57"/>
+      <origin xyz="0 0 0" rpy="0.0 0.0 -1.57"/>
       <mass value="1"/>
       <inertia

File: sim_challenges/urdf/bin2.xacro (robot description, xacro)
@@ -6,5 +6,5 @@
 <link name="bin2_base">
     <visual>
-        <origin xyz="22.180420 4.643661 -4.0" rpy="0.0 0.0 -1.57"/>
+        <origin xyz="0 0 0" rpy="0.0 0.0 -1.57"/>
         <geometry>
             <mesh filename="${visual_mesh_file}" scale="1 1 1" />
@@ -13,5 +13,5 @@
         <!-- Se deben cambiar los parametros reales-->
     <collision>
-      <origin xyz="22.180420 4.643661 -4.0" rpy="0.0 0.0 -1.57"/>
+      <origin xyz="0 0 0" rpy="0.0 0.0 -1.57"/>
       <geometry>
         <mesh filename="${visual_mesh_file}" scale="1 1 1" />
@@ -19,5 +19,5 @@
     </collision>
     <inertial>
-      <origin xyz="22.180420 4.643661 -4.0" rpy="0.0 0.0 -1.57"/>
+      <origin xyz="0 0 0" rpy="0.0 0.0 -1.57"/>
       <mass value="1"/>
       <inertia

File: sim_challenges/urdf/buoy2.xacro (robot description, xacro)
@@ -6,5 +6,5 @@
 <link name="buoy2_base">
     <visual>
-        <origin xyz="14.349550 -0.497678 -3.126359" rpy="0.0 0.0 1.57"/>
+        <origin xyz="0 0 -4" rpy="0.0 0.0 1.57"/>
         <geometry>
             <mesh filename="${visual_mesh_file}" scale="1 1 1" />
@@ -13,5 +13,5 @@
         <!-- Se deben cambiar los parametros reales-->
     <collision>
-      <origin xyz="14.349550 -0.497678 -3.126359" rpy="0.0 0.0 1.57"/>
+      <origin xyz="0 0 -4" rpy="0.0 0.0 1.57"/>
       <geometry>
         <mesh filename="${visual_mesh_file}" scale="1 1 1" />
@@ -19,5 +19,5 @@
     </collision>
     <inertial>
-      <origin xyz="14.349550 -0.497678 -3.126359" rpy="0.0 0.0 1.57"/>
+      <origin xyz="0 0 -4" rpy="0.0 0.0 1.57"/>
       <mass value="1"/>
       <inertia

File: sim_challenges/urdf/gate.xacro (robot description, xacro)
@@ -6,5 +6,5 @@
 <link name="gate_base">
     <visual>
-        <origin xyz="7.526688 -1.294371 -1.583826" rpy="0.0 0.0 1.57"/>
+        <origin xyz="0 0 -4" rpy="0.0 0.0 1.57"/>
         <geometry>
             <mesh filename="${visual_mesh_file}" scale="1 1 1" />
@@ -13,5 +13,5 @@
         <!-- Se deben cambiar los parametros reales-->
     <collision>
-      <origin xyz="7.526688 -1.294371 -1.583826" rpy="0.0 0.0 1.57"/>
+      <origin xyz="0 0 -4" rpy="0.0 0.0 1.57"/>
       <geometry>
         <mesh filename="${visual_mesh_file}" scale="1 1 1" />
@@ -19,5 +19,5 @@
     </collision>
     <inertial>
-      <origin xyz="7.526688 -1.294371 -1.583826" rpy="0.0 0.0 1.57"/>
+      <origin xyz="0 0 -4" rpy="0.0 0.0 1.57"/>
       <mass value="1"/>
       <inertia

File: sim_challenges/urdf/octagon.xacro (robot description, xacro)
@@ -6,5 +6,5 @@
 <link name="octagon_base">
     <visual>
-        <origin xyz="28.593435 -0.004454 -4.0" rpy="0.0 0.0 1.57"/>
+        <origin xyz="0 0 -4" rpy="0.0 0.0 1.57"/>
         <geometry>
             <mesh filename="${visual_mesh_file}" scale="1 1 1" />
@@ -13,5 +13,5 @@
         <!-- Se deben cambiar los parametros reales-->
     <collision>
-      <origin xyz="28.593435 -0.004454 -4.0" rpy="0.0 0.0 1.57"/>
+      <origin xyz="0 0 -4" rpy="0.0 0.0 1.57"/>
       <geometry>
         <mesh filename="${visual_mesh_file}" scale="1 1 1" />
@@ -19,5 +19,5 @@
     </collision>
     <inertial>
-      <origin xyz="28.593435 -0.004454 -4.0" rpy="0.0 0.0 1.57"/>
+      <origin xyz="0 0 -4" rpy="0.0 0.0 1.57"/>
       <mass value="1"/>
       <inertia

File: sim_challenges/urdf/pathmarkers/pathmarker1.xacro (robot description, xacro)
@@ -1,8 +1,8 @@
 <?xml version="1.0"?>
-<robot name="buoy_1" xmlns:xacro="http://www.ros.org/wiki/xacro">
+<robot name="path_marker" xmlns:xacro="http://www.ros.org/wiki/xacro">
 <!-- Introducir meshes -->
-<xacro:property name="visual_mesh_file" value="file://$(find sim_challenges)/models/meshes/buoy1.dae" />
-<!-- <origin xyz="0.085 (0 -0.085) 0 0" rpy="0.0 0.0 1.57075"/> -->
-<link name="buoy1_base">
+<xacro:property name="visual_mesh_file" value="file://$(find sim_challenges)/models/meshes/pathmarkers/pathmarker1.dae" />
+<!-- <origin xyz="0.085 (0 -0.085) 0 0" rpy="0.0 0.0 0.0075"/> -->
+<link name="path_marker_base">
     <visual>
         <origin xyz="0 0 -4" rpy="0.0 0.0 1.57"/>
@@ -27,5 +27,5 @@
     </inertial>
 </link>
-<gazebo reference="buoy1_base">
+<gazebo reference="path_marker_base">
   <selfCollide>0</selfCollide>
   <turnGravityOff>1</turnGravityOff>

File: sim_challenges/urdf/pathmarkers/pathmarker10.xacro (robot description, xacro)
@@ -1,8 +1,8 @@
 <?xml version="1.0"?>
-<robot name="buoy_1" xmlns:xacro="http://www.ros.org/wiki/xacro">
+<robot name="path_marker10" xmlns:xacro="http://www.ros.org/wiki/xacro">
 <!-- Introducir meshes -->
-<xacro:property name="visual_mesh_file" value="file://$(find sim_challenges)/models/meshes/buoy1.dae" />
-<!-- <origin xyz="0.085 (0 -0.085) 0 0" rpy="0.0 0.0 1.57075"/> -->
-<link name="buoy1_base">
+<xacro:property name="visual_mesh_file" value="file://$(find sim_challenges)/models/meshes/pathmarkers/pathmarker10.dae" />
+<!-- <origin xyz="0.085 (0 -0.085) 0 0" rpy="0.0 0.0 0.0075"/> -->
+<link name="path_marker_base10">
     <visual>
         <origin xyz="0 0 -4" rpy="0.0 0.0 1.57"/>
@@ -27,5 +27,5 @@
     </inertial>
 </link>
-<gazebo reference="buoy1_base">
+<gazebo reference="path_marker_base10">
   <selfCollide>0</selfCollide>
   <turnGravityOff>1</turnGravityOff>

File: sim_challenges/urdf/pathmarkers/pathmarker2.xacro (robot description, xacro)
@@ -1,8 +1,8 @@
 <?xml version="1.0"?>
-<robot name="buoy_1" xmlns:xacro="http://www.ros.org/wiki/xacro">
+<robot name="path_marker2" xmlns:xacro="http://www.ros.org/wiki/xacro">
 <!-- Introducir meshes -->
-<xacro:property name="visual_mesh_file" value="file://$(find sim_challenges)/models/meshes/buoy1.dae" />
-<!-- <origin xyz="0.085 (0 -0.085) 0 0" rpy="0.0 0.0 1.57075"/> -->
-<link name="buoy1_base">
+<xacro:property name="visual_mesh_file" value="file://$(find sim_challenges)/models/meshes/pathmarkers/pathmarker2.dae" />
+<!-- <origin xyz="0.085 (0 -0.085) 0 0" rpy="0.0 0.0 0.0075"/> -->
+<link name="path_marker_base2">
     <visual>
         <origin xyz="0 0 -4" rpy="0.0 0.0 1.57"/>
@@ -27,5 +27,5 @@
     </inertial>
 </link>
-<gazebo reference="buoy1_base">
+<gazebo reference="path_marker_base2">
   <selfCollide>0</selfCollide>
   <turnGravityOff>1</turnGravityOff>

File: sim_challenges/urdf/pathmarkers/pathmarker3.xacro (robot description, xacro)
@@ -1,8 +1,8 @@
 <?xml version="1.0"?>
-<robot name="buoy_1" xmlns:xacro="http://www.ros.org/wiki/xacro">
+<robot name="path_marker3" xmlns:xacro="http://www.ros.org/wiki/xacro">
 <!-- Introducir meshes -->
-<xacro:property name="visual_mesh_file" value="file://$(find sim_challenges)/models/meshes/buoy1.dae" />
-<!-- <origin xyz="0.085 (0 -0.085) 0 0" rpy="0.0 0.0 1.57075"/> -->
-<link name="buoy1_base">
+<xacro:property name="visual_mesh_file" value="file://$(find sim_challenges)/models/meshes/pathmarkers/pathmarker3.dae" />
+<!-- <origin xyz="0.085 (0 -0.085) 0 0" rpy="0.0 0.0 0.0075"/> -->
+<link name="path_marker_base3">
     <visual>
         <origin xyz="0 0 -4" rpy="0.0 0.0 1.57"/>
@@ -27,5 +27,5 @@
     </inertial>
 </link>
-<gazebo reference="buoy1_base">
+<gazebo reference="path_marker_base3">
   <selfCollide>0</selfCollide>
   <turnGravityOff>1</turnGravityOff>

File: sim_challenges/urdf/pathmarkers/pathmarker4.xacro (robot description, xacro)
@@ -1,10 +1,10 @@
 <?xml version="1.0"?>
-<robot name="path_marker" xmlns:xacro="http://www.ros.org/wiki/xacro">
+<robot name="path_marker4" xmlns:xacro="http://www.ros.org/wiki/xacro">
 <!-- Introducir meshes -->
-<xacro:property name="visual_mesh_file" value="file://$(find sim_challenges)/models/meshes/pathmarker.dae" />
-<!-- <origin xyz="0.085 (0 -0.085) 0 0" rpy="0.0 0.0 1.57075"/> -->
-<link name="path_marker_base">
+<xacro:property name="visual_mesh_file" value="file://$(find sim_challenges)/models/meshes/pathmarkers/pathmarker4.dae" />
+<!-- <origin xyz="0.085 (0 -0.085) 0 0" rpy="0.0 0.0 0.0075"/> -->
+<link name="path_marker_base4">
     <visual>
-        <origin xyz="14.349550 -1.744834 -3.126359" rpy="0.0 0.0 1.57"/>
+        <origin xyz="0 0 -4" rpy="0.0 0.0 1.57"/>
         <geometry>
             <mesh filename="${visual_mesh_file}" scale="1 1 1" />
@@ -13,5 +13,5 @@
         <!-- Se deben cambiar los parametros reales-->
     <collision>
-      <origin xyz="14.349550 -1.744834 -3.126359" rpy="0.0 0.0 1.57"/>
+      <origin xyz="0 0 -4" rpy="0.0 0.0 1.57"/>
       <geometry>
         <mesh filename="${visual_mesh_file}" scale="1 1 1" />
@@ -19,5 +19,5 @@
     </collision>
     <inertial>
-      <origin xyz="14.349550 -1.744834 -3.126359" rpy="0.0 0.0 1.57"/>
+      <origin xyz="0 0 -4" rpy="0.0 0.0 1.57"/>
       <mass value="1"/>
       <inertia
@@ -27,5 +27,5 @@
     </inertial>
 </link>
-<gazebo reference="path_marker_base">
+<gazebo reference="path_marker_base4">
   <selfCollide>0</selfCollide>
   <turnGravityOff>1</turnGravityOff>

File: sim_challenges/urdf/pathmarkers/pathmarker5.xacro (robot description, xacro)
@@ -1,8 +1,8 @@
 <?xml version="1.0"?>
-<robot name="buoy_1" xmlns:xacro="http://www.ros.org/wiki/xacro">
+<robot name="path_marker5" xmlns:xacro="http://www.ros.org/wiki/xacro">
 <!-- Introducir meshes -->
-<xacro:property name="visual_mesh_file" value="file://$(find sim_challenges)/models/meshes/buoy1.dae" />
-<!-- <origin xyz="0.085 (0 -0.085) 0 0" rpy="0.0 0.0 1.57075"/> -->
-<link name="buoy1_base">
+<xacro:property name="visual_mesh_file" value="file://$(find sim_challenges)/models/meshes/pathmarkers/pathmarker5.dae" />
+<!-- <origin xyz="0.085 (0 -0.085) 0 0" rpy="0.0 0.0 0.0075"/> -->
+<link name="path_marker_base5">
     <visual>
         <origin xyz="0 0 -4" rpy="0.0 0.0 1.57"/>
@@ -27,5 +27,5 @@
     </inertial>
 </link>
-<gazebo reference="buoy1_base">
+<gazebo reference="path_marker_base5">
   <selfCollide>0</selfCollide>
   <turnGravityOff>1</turnGravityOff>

File: sim_challenges/urdf/pathmarkers/pathmarker6.xacro (robot description, xacro)
@@ -1,8 +1,8 @@
 <?xml version="1.0"?>
-<robot name="buoy_1" xmlns:xacro="http://www.ros.org/wiki/xacro">
+<robot name="path_marker6" xmlns:xacro="http://www.ros.org/wiki/xacro">
 <!-- Introducir meshes -->
-<xacro:property name="visual_mesh_file" value="file://$(find sim_challenges)/models/meshes/buoy1.dae" />
-<!-- <origin xyz="0.085 (0 -0.085) 0 0" rpy="0.0 0.0 1.57075"/> -->
-<link name="buoy1_base">
+<xacro:property name="visual_mesh_file" value="file://$(find sim_challenges)/models/meshes/pathmarkers/pathmarker6.dae" />
+<!-- <origin xyz="0.085 (0 -0.085) 0 0" rpy="0.0 0.0 0.0075"/> -->
+<link name="path_marker_base6">
     <visual>
         <origin xyz="0 0 -4" rpy="0.0 0.0 1.57"/>
@@ -27,5 +27,5 @@
     </inertial>
 </link>
-<gazebo reference="buoy1_base">
+<gazebo reference="path_marker_base6">
   <selfCollide>0</selfCollide>
   <turnGravityOff>1</turnGravityOff>

File: sim_challenges/urdf/pathmarkers/pathmarker7.xacro (robot description, xacro)
@@ -1,8 +1,8 @@
 <?xml version="1.0"?>
-<robot name="buoy_1" xmlns:xacro="http://www.ros.org/wiki/xacro">
+<robot name="path_marker7" xmlns:xacro="http://www.ros.org/wiki/xacro">
 <!-- Introducir meshes -->
-<xacro:property name="visual_mesh_file" value="file://$(find sim_challenges)/models/meshes/buoy1.dae" />
-<!-- <origin xyz="0.085 (0 -0.085) 0 0" rpy="0.0 0.0 1.57075"/> -->
-<link name="buoy1_base">
+<xacro:property name="visual_mesh_file" value="file://$(find sim_challenges)/models/meshes/pathmarkers/pathmarker7.dae" />
+<!-- <origin xyz="0.085 (0 -0.085) 0 0" rpy="0.0 0.0 0.0075"/> -->
+<link name="path_marker_base7">
     <visual>
         <origin xyz="0 0 -4" rpy="0.0 0.0 1.57"/>
@@ -27,5 +27,5 @@
     </inertial>
 </link>
-<gazebo reference="buoy1_base">
+<gazebo reference="path_marker_base7">
   <selfCollide>0</selfCollide>
   <turnGravityOff>1</turnGravityOff>

File: sim_challenges/urdf/pathmarkers/pathmarker8.xacro (robot description, xacro)
@@ -1,8 +1,8 @@
 <?xml version="1.0"?>
-<robot name="buoy_1" xmlns:xacro="http://www.ros.org/wiki/xacro">
+<robot name="path_marker8" xmlns:xacro="http://www.ros.org/wiki/xacro">
 <!-- Introducir meshes -->
-<xacro:property name="visual_mesh_file" value="file://$(find sim_challenges)/models/meshes/buoy1.dae" />
-<!-- <origin xyz="0.085 (0 -0.085) 0 0" rpy="0.0 0.0 1.57075"/> -->
-<link name="buoy1_base">
+<xacro:property name="visual_mesh_file" value="file://$(find sim_challenges)/models/meshes/pathmarkers/pathmarker8.dae" />
+<!-- <origin xyz="0.085 (0 -0.085) 0 0" rpy="0.0 0.0 0.0075"/> -->
+<link name="path_marker_base8">
     <visual>
         <origin xyz="0 0 -4" rpy="0.0 0.0 1.57"/>
@@ -27,5 +27,5 @@
     </inertial>
 </link>
-<gazebo reference="buoy1_base">
+<gazebo reference="path_marker_base8">
   <selfCollide>0</selfCollide>
   <turnGravityOff>1</turnGravityOff>

File: sim_challenges/urdf/pathmarkers/pathmarker9.xacro (robot description, xacro)
@@ -1,8 +1,8 @@
 <?xml version="1.0"?>
-<robot name="buoy_1" xmlns:xacro="http://www.ros.org/wiki/xacro">
+<robot name="path_marker9" xmlns:xacro="http://www.ros.org/wiki/xacro">
 <!-- Introducir meshes -->
-<xacro:property name="visual_mesh_file" value="file://$(find sim_challenges)/models/meshes/buoy1.dae" />
-<!-- <origin xyz="0.085 (0 -0.085) 0 0" rpy="0.0 0.0 1.57075"/> -->
-<link name="buoy1_base">
+<xacro:property name="visual_mesh_file" value="file://$(find sim_challenges)/models/meshes/pathmarkers/pathmarker9.dae" />
+<!-- <origin xyz="0.085 (0 -0.085) 0 0" rpy="0.0 0.0 0.0075"/> -->
+<link name="path_marker_base9">
     <visual>
         <origin xyz="0 0 -4" rpy="0.0 0.0 1.57"/>
@@ -27,5 +27,5 @@
     </inertial>
 </link>
-<gazebo reference="buoy1_base">
+<gazebo reference="path_marker_base9">
   <selfCollide>0</selfCollide>
   <turnGravityOff>1</turnGravityOff>

File: sim_challenges/urdf/torpedos1.xacro (robot description, xacro)
@@ -6,5 +6,5 @@
 <link name="torpedos1_base">
     <visual>
-        <origin xyz="25.180420 1.835166 -4.0" rpy="0.0 0.0 1.57"/>
+        <origin xyz="0 0 -4" rpy="0.0 0.0 1.57"/>
         <geometry>
             <mesh filename="${visual_mesh_file}" scale="1 1 1" />
@@ -13,5 +13,5 @@
         <!-- Se deben cambiar los parametros reales-->
     <collision>
-      <origin xyz="25.180420 1.835166 -4.0" rpy="0.0 0.0 1.57"/>
+      <origin xyz="0 0 -4" rpy="0.0 0.0 1.57"/>
       <geometry>
         <mesh filename="${visual_mesh_file}" scale="1 1 1" />
@@ -19,5 +19,5 @@
     </collision>
     <inertial>
-      <origin xyz="25.180420 1.835166 -4.0" rpy="0.0 0.0 1.57"/>
+      <origin xyz="0 0 -4" rpy="0.0 0.0 1.57"/>
       <mass value="1"/>
       <inertia

File: sim_challenges/urdf/torpedos2.xacro (robot description, xacro)
@@ -6,5 +6,5 @@
 <link name="torpedos2_base">
     <visual>
-        <origin xyz="25.180420 3.082322 -4.0" rpy="0.0 0.0 1.57"/>
+        <origin xyz="0 0 -4" rpy="0.0 0.0 1.57"/>
         <geometry>
             <mesh filename="${visual_mesh_file}" scale="1 1 1" />
@@ -13,5 +13,5 @@
         <!-- Se deben cambiar los parametros reales-->
     <collision>
-      <origin xyz="25.180420 3.082322 -4.0" rpy="0.0 0.0 1.57"/>
+      <origin xyz="0 0 -4" rpy="0.0 0.0 1.57"/>
       <geometry>
         <mesh filename="${visual_mesh_file}" scale="1 1 1" />
@@ -19,5 +19,5 @@
     </collision>
     <inertial>
-      <origin xyz="25.180420 3.082322 -4.0" rpy="0.0 0.0 1.57"/>
+      <origin xyz="0 0 -4" rpy="0.0 0.0 1.57"/>
       <mass value="1"/>
       <inertia
