Commit message: Cambios cambios

File: sim_challenges/urdf/bin1.xacro (robot description, xacro)
@@ -6,5 +6,5 @@
 <link name="bin1_base">
     <visual>
-        <origin xyz="22.180420 -2.960028 -4.0" rpy="0.0 0.0 -1.57"/>
+        <origin xyz="5.00 0 -22.0" rpy="0.0 0.0 -1.57"/>
         <geometry>
             <mesh filename="${visual_mesh_file}" scale="1 1 1" />
@@ -13,5 +13,5 @@
         <!-- Se deben cambiar los parametros reales-->
     <collision>
-      <origin xyz="22.180420 -2.960028 -4.0" rpy="0.0 0.0 -1.57"/>
+      <origin xyz="5.00 0 -22.0" rpy="0.0 0.0 -1.57"/>
       <geometry>
         <mesh filename="${visual_mesh_file}" scale="1 1 1" />
@@ -19,5 +19,5 @@
     </collision>
     <inertial>
-      <origin xyz="22.180420 -2.960028 -4.0" rpy="0.0 0.0 -1.57"/>
+      <origin xyz="5.00 0 -22.0" rpy="0.0 0.0 -1.57"/>
       <mass value="1"/>
       <inertia

File: sim_challenges/urdf/bin2.xacro (robot description, xacro)
@@ -6,5 +6,5 @@
 <link name="bin2_base">
     <visual>
-        <origin xyz="22.180420 4.643661 -4.0" rpy="0.0 0.0 -1.57"/>
+        <origin xyz="5.00 0 -22.0" rpy="0.0 0.0 -1.57"/>
         <geometry>
             <mesh filename="${visual_mesh_file}" scale="1 1 1" />
@@ -13,5 +13,5 @@
         <!-- Se deben cambiar los parametros reales-->
     <collision>
-      <origin xyz="22.180420 4.643661 -4.0" rpy="0.0 0.0 -1.57"/>
+      <origin xyz="5.00 0 -22.0" rpy="0.0 0.0 -1.57"/>
       <geometry>
         <mesh filename="${visual_mesh_file}" scale="1 1 1" />
@@ -19,5 +19,5 @@
     </collision>
     <inertial>
-      <origin xyz="22.180420 4.643661 -4.0" rpy="0.0 0.0 -1.57"/>
+      <origin xyz="5.00 0 -22.0" rpy="0.0 0.0 -1.57"/>
       <mass value="1"/>
       <inertia

File: sim_challenges/urdf/gate.xacro (robot description, xacro)
@@ -6,5 +6,5 @@
 <link name="gate_base">
     <visual>
-        <origin xyz="7.526688 -1.294371 -1.583826" rpy="0.0 0.0 1.57"/>
+        <origin xyz="7.00 0 -22.0" rpy="0.0 0.0 1.57"/>
         <geometry>
             <mesh filename="${visual_mesh_file}" scale="1 1 1" />
@@ -13,5 +13,5 @@
         <!-- Se deben cambiar los parametros reales-->
     <collision>
-      <origin xyz="7.526688 -1.294371 -1.583826" rpy="0.0 0.0 1.57"/>
+      <origin xyz="7.00 0 -22.0" rpy="0.0 0.0 1.57"/>
       <geometry>
         <mesh filename="${visual_mesh_file}" scale="1 1 1" />
@@ -19,5 +19,5 @@
     </collision>
     <inertial>
-      <origin xyz="7.526688 -1.294371 -1.583826" rpy="0.0 0.0 1.57"/>
+      <origin xyz="7.00 0 -22.0" rpy="0.0 0.0 1.57"/>
       <mass value="1"/>
       <inertia

File: sim_challenges/urdf/pathmarker.xacro (robot description, xacro)
@@ -6,5 +6,5 @@
 <link name="path_marker_base">
     <visual>
-        <origin xyz="14.349550 -1.744834 -3.126359" rpy="3.1416 0.0 0.0"/>
+        <origin xyz="7.00 0 -22.0" rpy="3.1416 0.0 0.0"/>
         <geometry>
             <mesh filename="${visual_mesh_file}" scale="1 1 1" />
@@ -13,5 +13,5 @@
         <!-- Se deben cambiar los parametros reales-->
     <collision>
-      <origin xyz="14.349550 -1.744834 -3.126359" rpy="3.1416 0.0 0.0"/>
+      <origin xyz="7.00 0 -22.0" rpy="3.1416 0.0 0.0"/>
       <geometry>
         <mesh filename="${visual_mesh_file}" scale="1 1 1" />
@@ -19,5 +19,5 @@
     </collision>
     <inertial>
-      <origin xyz="14.349550 -1.744834 -3.126359" rpy="3.1416 0.0 0.0"/>
+      <origin xyz="7.00 0 -22.0" rpy="3.1416 0.0 0.0"/>
       <mass value="1"/>
       <inertia

File: sim_challenges/urdf/pathmarker2.xacro (robot description, xacro)
@@ -6,5 +6,5 @@
 <link name="path_marker_base2">
     <visual>
-        <origin xyz="14.349550 1.744834 -3.126359" rpy="1.57 0.0 0.0"/>
+        <origin xyz="7.00 0 -22.0" rpy="1.57 0.0 0.0"/>
         <geometry>
             <mesh filename="${visual_mesh_file}" scale="1 1 1" />
@@ -13,5 +13,5 @@
         <!-- Se deben cambiar los parametros reales-->
     <collision>
-      <origin xyz="14.349550 1.744834 -3.126359" rpy="1.57 0.0 0.0"/>
+      <origin xyz="7.00 0 -22.0" rpy="1.57 0.0 0.0"/>
       <geometry>
         <mesh filename="${visual_mesh_file}" scale="1 1 1" />
@@ -19,5 +19,5 @@
     </collision>
     <inertial>
-      <origin xyz="14.349550 1.744834 -3.126359" rpy="1.57 0.0 0.0"/>
+      <origin xyz="7.00 0 -22.0" rpy="1.57 0.0 0.0"/>
       <mass value="1"/>
       <inertia

Commit message: Added bins, black gate, and path markers

File: sim_challenges/urdf/bin1.xacro (robot description, xacro)
@@ -1,10 +1,11 @@
 <?xml version="1.0"?>
 <robot name="bin_1" xmlns:xacro="http://www.ros.org/wiki/xacro">
+<!--Change .dae to binopen.dae, bintapadod.dae, bintapadoi.dae depending on the situation-->
 <!-- Introducir meshes -->
-<xacro:property name="visual_mesh_file" value="file://$(find sim_challenges)/models/meshes/bin.dae" />
+<xacro:property name="visual_mesh_file" value="file://$(find sim_challenges)/models/meshes/bintapadoi.dae" />
 <!-- <origin xyz="0.085 (0 -0.085) 0 0" rpy="0.0 0.0 1.57075"/> -->
 <link name="bin1_base">
     <visual>
-        <origin xyz="0 0 0" rpy="0.0 0.0 -1.57"/>
+        <origin xyz="0 0 -4" rpy="0.0 0.0 1.57"/>
         <geometry>
             <mesh filename="${visual_mesh_file}" scale="1 1 1" />
@@ -13,5 +14,5 @@
         <!-- Se deben cambiar los parametros reales-->
     <collision>
-      <origin xyz="0 0 0" rpy="0.0 0.0 -1.57"/>
+      <origin xyz="0 0 -4" rpy="0.0 0.0 1.57"/>
       <geometry>
         <mesh filename="${visual_mesh_file}" scale="1 1 1" />
@@ -19,5 +20,5 @@
     </collision>
     <inertial>
-      <origin xyz="0 0 0" rpy="0.0 0.0 -1.57"/>
+      <origin xyz="0 0 -4" rpy="0.0 0.0 1.57"/>
       <mass value="1"/>
       <inertia

Commit message: Fix positions task

File: sim_challenges/urdf/bin1.xacro (robot description, xacro)
@@ -7,5 +7,5 @@
 <link name="bin1_base">
     <visual>
-        <origin xyz="0 0 -4" rpy="0.0 0.0 1.57"/>
+        <origin xyz="0 0 -4" rpy="0.0 0.0 0.0"/>
         <geometry>
             <mesh filename="${visual_mesh_file}" scale="1 1 1" />
@@ -14,5 +14,5 @@
         <!-- Se deben cambiar los parametros reales-->
     <collision>
-      <origin xyz="0 0 -4" rpy="0.0 0.0 1.57"/>
+      <origin xyz="0 0 -4" rpy="0.0 0.0 0.0"/>
       <geometry>
         <mesh filename="${visual_mesh_file}" scale="1 1 1" />
@@ -20,5 +20,5 @@
     </collision>
     <inertial>
-      <origin xyz="0 0 -4" rpy="0.0 0.0 1.57"/>
+      <origin xyz="0 0 -4" rpy="0.0 0.0 0.0"/>
       <mass value="1"/>
       <inertia

File: sim_challenges/urdf/buoy.xacro (robot description, xacro)
@@ -6,5 +6,5 @@
 <link name="buoy1_base">
     <visual>
-        <origin xyz="0 0 -4" rpy="0.0 0.0 1.57"/>
+        <origin xyz="0 0 -4" rpy="0.0 0.0 0.0"/>
         <geometry>
             <mesh filename="${visual_mesh_file}" scale="1 1 1" />
@@ -13,5 +13,5 @@
         <!-- Se deben cambiar los parametros reales-->
     <collision>
-      <origin xyz="0 0 -4" rpy="0.0 0.0 1.57"/>
+      <origin xyz="0 0 -4" rpy="0.0 0.0 0.0"/>
       <geometry>
         <mesh filename="${visual_mesh_file}" scale="1 1 1" />
@@ -19,5 +19,5 @@
     </collision>
     <inertial>
-      <origin xyz="0 0 -4" rpy="0.0 0.0 1.57"/>
+      <origin xyz="0 0 -4" rpy="0.0 0.0 0.0"/>
       <mass value="1"/>
       <inertia

File: sim_challenges/urdf/buoy2.xacro (robot description, xacro)
@@ -6,5 +6,5 @@
 <link name="buoy2_base">
     <visual>
-        <origin xyz="0 0 -4" rpy="0.0 0.0 1.57"/>
+        <origin xyz="0 0 -4" rpy="0.0 0.0 0.0"/>
         <geometry>
             <mesh filename="${visual_mesh_file}" scale="1 1 1" />
@@ -13,5 +13,5 @@
         <!-- Se deben cambiar los parametros reales-->
     <collision>
-      <origin xyz="0 0 -4" rpy="0.0 0.0 1.57"/>
+      <origin xyz="0 0 -4" rpy="0.0 0.0 0.0"/>
       <geometry>
         <mesh filename="${visual_mesh_file}" scale="1 1 1" />
@@ -19,5 +19,5 @@
     </collision>
     <inertial>
-      <origin xyz="0 0 -4" rpy="0.0 0.0 1.57"/>
+      <origin xyz="0 0 -4" rpy="0.0 0.0 0.0"/>
       <mass value="1"/>
       <inertia

File: sim_challenges/urdf/gate.xacro (robot description, xacro)
@@ -6,5 +6,5 @@
 <link name="gate_base">
     <visual>
-        <origin xyz="0 0 -4" rpy="0.0 0.0 1.57"/>
+        <origin xyz="0 0 -4" rpy="0.0 0.0 0"/>
         <geometry>
             <mesh filename="${visual_mesh_file}" scale="1 1 1" />
@@ -13,5 +13,5 @@
         <!-- Se deben cambiar los parametros reales-->
     <collision>
-      <origin xyz="0 0 -4" rpy="0.0 0.0 1.57"/>
+      <origin xyz="0 0 -4" rpy="0.0 0.0 0.0"/>
       <geometry>
         <mesh filename="${visual_mesh_file}" scale="1 1 1" />
@@ -19,5 +19,5 @@
     </collision>
     <inertial>
-      <origin xyz="0 0 -4" rpy="0.0 0.0 1.57"/>
+      <origin xyz="0 0 -4" rpy="0.0 0.0 0.0"/>
       <mass value="1"/>
       <inertia

File: sim_challenges/urdf/octagon.xacro (robot description, xacro)
@@ -6,5 +6,5 @@
 <link name="octagon_base">
     <visual>
-        <origin xyz="0 0 -4" rpy="0.0 0.0 1.57"/>
+        <origin xyz="0 0 -4" rpy="0.0 0.0 0.0"/>
         <geometry>
             <mesh filename="${visual_mesh_file}" scale="1 1 1" />
@@ -13,5 +13,5 @@
         <!-- Se deben cambiar los parametros reales-->
     <collision>
-      <origin xyz="0 0 -4" rpy="0.0 0.0 1.57"/>
+      <origin xyz="0 0 -4" rpy="0.0 0.0 0.0"/>
       <geometry>
         <mesh filename="${visual_mesh_file}" scale="1 1 1" />
@@ -19,5 +19,5 @@
     </collision>
     <inertial>
-      <origin xyz="0 0 -4" rpy="0.0 0.0 1.57"/>
+      <origin xyz="0 0 -4" rpy="0.0 0.0 0.0"/>
       <mass value="1"/>
       <inertia

File: sim_challenges/urdf/pathmarkers/pathmarker1.xacro (robot description, xacro)
@@ -6,5 +6,5 @@
 <link name="path_marker_base">
     <visual>
-        <origin xyz="0 0 -4" rpy="0.0 0.0 1.57"/>
+        <origin xyz="0 0 -4" rpy="0.0 0.0 0.0"/>
         <geometry>
             <mesh filename="${visual_mesh_file}" scale="1 1 1" />
@@ -13,5 +13,5 @@
         <!-- Se deben cambiar los parametros reales-->
     <collision>
-      <origin xyz="0 0 -4" rpy="0.0 0.0 1.57"/>
+      <origin xyz="0 0 -4" rpy="0.0 0.0 0.0"/>
       <geometry>
         <mesh filename="${visual_mesh_file}" scale="1 1 1" />
@@ -19,5 +19,5 @@
     </collision>
     <inertial>
-      <origin xyz="0 0 -4" rpy="0.0 0.0 1.57"/>
+      <origin xyz="0 0 -4" rpy="0.0 0.0 0.0"/>
       <mass value="1"/>
       <inertia

File: sim_challenges/urdf/pathmarkers/pathmarker10.xacro (robot description, xacro)
@@ -6,5 +6,5 @@
 <link name="path_marker_base10">
     <visual>
-        <origin xyz="0 0 -4" rpy="0.0 0.0 1.57"/>
+        <origin xyz="0 0 -4" rpy="0.0 0.0 0.0"/>
         <geometry>
             <mesh filename="${visual_mesh_file}" scale="1 1 1" />
@@ -13,5 +13,5 @@
         <!-- Se deben cambiar los parametros reales-->
     <collision>
-      <origin xyz="0 0 -4" rpy="0.0 0.0 1.57"/>
+      <origin xyz="0 0 -4" rpy="0.0 0.0 0.0"/>
       <geometry>
         <mesh filename="${visual_mesh_file}" scale="1 1 1" />
@@ -19,5 +19,5 @@
     </collision>
     <inertial>
-      <origin xyz="0 0 -4" rpy="0.0 0.0 1.57"/>
+      <origin xyz="0 0 -4" rpy="0.0 0.0 0.0"/>
       <mass value="1"/>
       <inertia

File: sim_challenges/urdf/pathmarkers/pathmarker2.xacro (robot description, xacro)
@@ -6,5 +6,5 @@
 <link name="path_marker_base2">
     <visual>
-        <origin xyz="0 0 -4" rpy="0.0 0.0 1.57"/>
+        <origin xyz="0 0 -4" rpy="0.0 0.0 0.0"/>
         <geometry>
             <mesh filename="${visual_mesh_file}" scale="1 1 1" />
@@ -13,5 +13,5 @@
         <!-- Se deben cambiar los parametros reales-->
     <collision>
-      <origin xyz="0 0 -4" rpy="0.0 0.0 1.57"/>
+      <origin xyz="0 0 -4" rpy="0.0 0.0 0.0"/>
       <geometry>
         <mesh filename="${visual_mesh_file}" scale="1 1 1" />
@@ -19,5 +19,5 @@
     </collision>
     <inertial>
-      <origin xyz="0 0 -4" rpy="0.0 0.0 1.57"/>
+      <origin xyz="0 0 -4" rpy="0.0 0.0 0.0"/>
       <mass value="1"/>
       <inertia

File: sim_challenges/urdf/pathmarkers/pathmarker3.xacro (robot description, xacro)
@@ -6,5 +6,5 @@
 <link name="path_marker_base3">
     <visual>
-        <origin xyz="0 0 -4" rpy="0.0 0.0 1.57"/>
+        <origin xyz="0 0 -4" rpy="0.0 0.0 0.0"/>
         <geometry>
             <mesh filename="${visual_mesh_file}" scale="1 1 1" />
@@ -13,5 +13,5 @@
         <!-- Se deben cambiar los parametros reales-->
     <collision>
-      <origin xyz="0 0 -4" rpy="0.0 0.0 1.57"/>
+      <origin xyz="0 0 -4" rpy="0.0 0.0 0.0"/>
       <geometry>
         <mesh filename="${visual_mesh_file}" scale="1 1 1" />
@@ -19,5 +19,5 @@
     </collision>
     <inertial>
-      <origin xyz="0 0 -4" rpy="0.0 0.0 1.57"/>
+      <origin xyz="0 0 -4" rpy="0.0 0.0 0.0"/>
       <mass value="1"/>
       <inertia

File: sim_challenges/urdf/pathmarkers/pathmarker4.xacro (robot description, xacro)
@@ -6,5 +6,5 @@
 <link name="path_marker_base4">
     <visual>
-        <origin xyz="0 0 -4" rpy="0.0 0.0 1.57"/>
+        <origin xyz="0 0 -4" rpy="0.0 0.0 0.0"/>
         <geometry>
             <mesh filename="${visual_mesh_file}" scale="1 1 1" />
@@ -13,5 +13,5 @@
         <!-- Se deben cambiar los parametros reales-->
     <collision>
-      <origin xyz="0 0 -4" rpy="0.0 0.0 1.57"/>
+      <origin xyz="0 0 -4" rpy="0.0 0.0 0.0"/>
       <geometry>
         <mesh filename="${visual_mesh_file}" scale="1 1 1" />
@@ -19,5 +19,5 @@
     </collision>
     <inertial>
-      <origin xyz="0 0 -4" rpy="0.0 0.0 1.57"/>
+      <origin xyz="0 0 -4" rpy="0.0 0.0 0.0"/>
       <mass value="1"/>
       <inertia

File: sim_challenges/urdf/pathmarkers/pathmarker5.xacro (robot description, xacro)
@@ -6,5 +6,5 @@
 <link name="path_marker_base5">
     <visual>
-        <origin xyz="0 0 -4" rpy="0.0 0.0 1.57"/>
+        <origin xyz="0 0 -4" rpy="0.0 0.0 0.0"/>
         <geometry>
             <mesh filename="${visual_mesh_file}" scale="1 1 1" />
@@ -13,5 +13,5 @@
         <!-- Se deben cambiar los parametros reales-->
     <collision>
-      <origin xyz="0 0 -4" rpy="0.0 0.0 1.57"/>
+      <origin xyz="0 0 -4" rpy="0.0 0.0 0.0"/>
       <geometry>
         <mesh filename="${visual_mesh_file}" scale="1 1 1" />
@@ -19,5 +19,5 @@
     </collision>
     <inertial>
-      <origin xyz="0 0 -4" rpy="0.0 0.0 1.57"/>
+      <origin xyz="0 0 -4" rpy="0.0 0.0 0.0"/>
       <mass value="1"/>
       <inertia

File: sim_challenges/urdf/pathmarkers/pathmarker6.xacro (robot description, xacro)
@@ -6,5 +6,5 @@
 <link name="path_marker_base6">
     <visual>
-        <origin xyz="0 0 -4" rpy="0.0 0.0 1.57"/>
+        <origin xyz="0 0 -4" rpy="0.0 0.0 0.0"/>
         <geometry>
             <mesh filename="${visual_mesh_file}" scale="1 1 1" />
@@ -13,5 +13,5 @@
         <!-- Se deben cambiar los parametros reales-->
     <collision>
-      <origin xyz="0 0 -4" rpy="0.0 0.0 1.57"/>
+      <origin xyz="0 0 -4" rpy="0.0 0.0 0.0"/>
       <geometry>
         <mesh filename="${visual_mesh_file}" scale="1 1 1" />
@@ -19,5 +19,5 @@
     </collision>
     <inertial>
-      <origin xyz="0 0 -4" rpy="0.0 0.0 1.57"/>
+      <origin xyz="0 0 -4" rpy="0.0 0.0 0.0"/>
       <mass value="1"/>
       <inertia

File: sim_challenges/urdf/pathmarkers/pathmarker7.xacro (robot description, xacro)
@@ -6,5 +6,5 @@
 <link name="path_marker_base7">
     <visual>
-        <origin xyz="0 0 -4" rpy="0.0 0.0 1.57"/>
+        <origin xyz="0 0 -4" rpy="0.0 0.0 0.0"/>
         <geometry>
             <mesh filename="${visual_mesh_file}" scale="1 1 1" />
@@ -13,5 +13,5 @@
         <!-- Se deben cambiar los parametros reales-->
     <collision>
-      <origin xyz="0 0 -4" rpy="0.0 0.0 1.57"/>
+      <origin xyz="0 0 -4" rpy="0.0 0.0 0.0"/>
       <geometry>
         <mesh filename="${visual_mesh_file}" scale="1 1 1" />
@@ -19,5 +19,5 @@
     </collision>
     <inertial>
-      <origin xyz="0 0 -4" rpy="0.0 0.0 1.57"/>
+      <origin xyz="0 0 -4" rpy="0.0 0.0 0.0"/>
       <mass value="1"/>
       <inertia

File: sim_challenges/urdf/pathmarkers/pathmarker8.xacro (robot description, xacro)
@@ -6,5 +6,5 @@
 <link name="path_marker_base8">
     <visual>
-        <origin xyz="0 0 -4" rpy="0.0 0.0 1.57"/>
+        <origin xyz="0 0 -4" rpy="0.0 0.0 0.0"/>
         <geometry>
             <mesh filename="${visual_mesh_file}" scale="1 1 1" />
@@ -13,5 +13,5 @@
         <!-- Se deben cambiar los parametros reales-->
     <collision>
-      <origin xyz="0 0 -4" rpy="0.0 0.0 1.57"/>
+      <origin xyz="0 0 -4" rpy="0.0 0.0 0.0"/>
       <geometry>
         <mesh filename="${visual_mesh_file}" scale="1 1 1" />
@@ -19,5 +19,5 @@
     </collision>
     <inertial>
-      <origin xyz="0 0 -4" rpy="0.0 0.0 1.57"/>
+      <origin xyz="0 0 -4" rpy="0.0 0.0 0.0"/>
       <mass value="1"/>
       <inertia

File: sim_challenges/urdf/pathmarkers/pathmarker9.xacro (robot description, xacro)
@@ -6,5 +6,5 @@
 <link name="path_marker_base9">
     <visual>
-        <origin xyz="0 0 -4" rpy="0.0 0.0 1.57"/>
+        <origin xyz="0 0 -4" rpy="0.0 0.0 0.0"/>
         <geometry>
             <mesh filename="${visual_mesh_file}" scale="1 1 1" />
@@ -13,5 +13,5 @@
         <!-- Se deben cambiar los parametros reales-->
     <collision>
-      <origin xyz="0 0 -4" rpy="0.0 0.0 1.57"/>
+      <origin xyz="0 0 -4" rpy="0.0 0.0 0.0"/>
       <geometry>
         <mesh filename="${visual_mesh_file}" scale="1 1 1" />
@@ -19,5 +19,5 @@
     </collision>
     <inertial>
-      <origin xyz="0 0 -4" rpy="0.0 0.0 1.57"/>
+      <origin xyz="0 0 -4" rpy="0.0 0.0 0.0"/>
       <mass value="1"/>
       <inertia

File: sim_challenges/urdf/torpedos1.xacro (robot description, xacro)
@@ -6,5 +6,5 @@
 <link name="torpedos1_base">
     <visual>
-        <origin xyz="0 0 -4" rpy="0.0 0.0 1.57"/>
+        <origin xyz="0 0 -4" rpy="0.0 0.0 0.0"/>
         <geometry>
             <mesh filename="${visual_mesh_file}" scale="1 1 1" />
@@ -13,5 +13,5 @@
         <!-- Se deben cambiar los parametros reales-->
     <collision>
-      <origin xyz="0 0 -4" rpy="0.0 0.0 1.57"/>
+      <origin xyz="0 0 -4" rpy="0.0 0.0 0.0"/>
       <geometry>
         <mesh filename="${visual_mesh_file}" scale="1 1 1" />
@@ -19,5 +19,5 @@
     </collision>
     <inertial>
-      <origin xyz="0 0 -4" rpy="0.0 0.0 1.57"/>
+      <origin xyz="0 0 -4" rpy="0.0 0.0 0.0"/>
       <mass value="1"/>
       <inertia

File: sim_challenges/urdf/torpedos2.xacro (robot description, xacro)
@@ -6,5 +6,5 @@
 <link name="torpedos2_base">
     <visual>
-        <origin xyz="0 0 -4" rpy="0.0 0.0 1.57"/>
+        <origin xyz="0 0 -4" rpy="0.0 0.0 0.0"/>
         <geometry>
             <mesh filename="${visual_mesh_file}" scale="1 1 1" />
@@ -13,5 +13,5 @@
         <!-- Se deben cambiar los parametros reales-->
     <collision>
-      <origin xyz="0 0 -4" rpy="0.0 0.0 1.57"/>
+      <origin xyz="0 0 -4" rpy="0.0 0.0 0.0"/>
       <geometry>
         <mesh filename="${visual_mesh_file}" scale="1 1 1" />
@@ -19,5 +19,5 @@
     </collision>
     <inertial>
-      <origin xyz="0 0 -4" rpy="0.0 0.0 1.57"/>
+      <origin xyz="0 0 -4" rpy="0.0 0.0 0.0"/>
       <mass value="1"/>
       <inertia

Commit message: Octagon included-models.dae

File: sim_challenges/urdf/bin1.xacro (robot description, xacro)
@@ -7,5 +7,5 @@
 <link name="bin1_base">
     <visual>
-        <origin xyz="0 0 -4" rpy="0.0 0.0 0.0"/>
+        <origin xyz="0 0 -5.5" rpy="0.0 0.0 0.0"/>
         <geometry>
             <mesh filename="${visual_mesh_file}" scale="1 1 1" />
@@ -14,5 +14,5 @@
         <!-- Se deben cambiar los parametros reales-->
     <collision>
-      <origin xyz="0 0 -4" rpy="0.0 0.0 0.0"/>
+      <origin xyz="0 0 -5.5" rpy="0.0 0.0 0.0"/>
       <geometry>
         <mesh filename="${visual_mesh_file}" scale="1 1 1" />
@@ -20,5 +20,5 @@
     </collision>
     <inertial>
-      <origin xyz="0 0 -4" rpy="0.0 0.0 0.0"/>
+      <origin xyz="0 0 -5.5" rpy="0.0 0.0 0.0"/>
       <mass value="1"/>
       <inertia

File: sim_challenges/urdf/bin2.xacro (robot description, xacro)
@@ -6,5 +6,5 @@
 <link name="bin2_base">
     <visual>
-        <origin xyz="0 0 0" rpy="0.0 0.0 -1.57"/>
+        <origin xyz="0 0 -5.5" rpy="0.0 0.0 0.0"/>
         <geometry>
             <mesh filename="${visual_mesh_file}" scale="1 1 1" />
@@ -13,5 +13,5 @@
         <!-- Se deben cambiar los parametros reales-->
     <collision>
-      <origin xyz="0 0 0" rpy="0.0 0.0 -1.57"/>
+      <origin xyz="0 0 -5.5" rpy="0.0 0.0 0.0"/>
       <geometry>
         <mesh filename="${visual_mesh_file}" scale="1 1 1" />
@@ -19,5 +19,5 @@
     </collision>
     <inertial>
-      <origin xyz="0 0 0" rpy="0.0 0.0 -1.57"/>
+      <origin xyz="0 0 -5.5" rpy="0.0 0.0 0.0"/>
       <mass value="1"/>
       <inertia
