Commit message: Gate vision code upgrade

File: sim_challenges/urdf/bin1.xacro (robot description, xacro)
@@ -7,5 +7,5 @@
 <link name="bin1_base">
     <visual>
-        <origin xyz="0 0 -5.5" rpy="0.0 0.0 0.0"/>
+        <origin xyz="0 0 -8.5" rpy="0.0 0.0 0.0"/>
         <geometry>
             <mesh filename="${visual_mesh_file}" scale="1 1 1" />
@@ -14,5 +14,5 @@
         <!-- Se deben cambiar los parametros reales-->
     <collision>
-      <origin xyz="0 0 -5.5" rpy="0.0 0.0 0.0"/>
+      <origin xyz="0 0 -8.5" rpy="0.0 0.0 0.0"/>
       <geometry>
         <mesh filename="${visual_mesh_file}" scale="1 1 1" />
@@ -20,5 +20,5 @@
     </collision>
     <inertial>
-      <origin xyz="0 0 -5.5" rpy="0.0 0.0 0.0"/>
+      <origin xyz="0 0 -8.5" rpy="0.0 0.0 0.0"/>
       <mass value="1"/>
       <inertia

File: sim_challenges/urdf/bin2.xacro (robot description, xacro)
@@ -6,5 +6,5 @@
 <link name="bin2_base">
     <visual>
-        <origin xyz="0 0 -5.5" rpy="0.0 0.0 0.0"/>
+        <origin xyz="0 0 -8.5" rpy="0.0 0.0 0.0"/>
         <geometry>
             <mesh filename="${visual_mesh_file}" scale="1 1 1" />
@@ -13,5 +13,5 @@
         <!-- Se deben cambiar los parametros reales-->
     <collision>
-      <origin xyz="0 0 -5.5" rpy="0.0 0.0 0.0"/>
+      <origin xyz="0 0 -8.5" rpy="0.0 0.0 0.0"/>
       <geometry>
         <mesh filename="${visual_mesh_file}" scale="1 1 1" />
@@ -19,5 +19,5 @@
     </collision>
     <inertial>
-      <origin xyz="0 0 -5.5" rpy="0.0 0.0 0.0"/>
+      <origin xyz="0 0 -8.5" rpy="0.0 0.0 0.0"/>
       <mass value="1"/>
       <inertia

File: sim_challenges/urdf/buoy.xacro (robot description, xacro)
@@ -6,5 +6,5 @@
 <link name="buoy1_base">
     <visual>
-        <origin xyz="0 0 -4" rpy="0.0 0.0 0.0"/>
+        <origin xyz="0 0 -7" rpy="0.0 0.0 0.0"/>
         <geometry>
             <mesh filename="${visual_mesh_file}" scale="1 1 1" />
@@ -13,5 +13,5 @@
         <!-- Se deben cambiar los parametros reales-->
     <collision>
-      <origin xyz="0 0 -4" rpy="0.0 0.0 0.0"/>
+      <origin xyz="0 0 -7" rpy="0.0 0.0 0.0"/>
       <geometry>
         <mesh filename="${visual_mesh_file}" scale="1 1 1" />
@@ -19,5 +19,5 @@
     </collision>
     <inertial>
-      <origin xyz="0 0 -4" rpy="0.0 0.0 0.0"/>
+      <origin xyz="0 0 -7" rpy="0.0 0.0 0.0"/>
       <mass value="1"/>
       <inertia

File: sim_challenges/urdf/buoy2.xacro (robot description, xacro)
@@ -6,5 +6,5 @@
 <link name="buoy2_base">
     <visual>
-        <origin xyz="0 0 -4" rpy="0.0 0.0 0.0"/>
+        <origin xyz="0 0 -7" rpy="0.0 0.0 0.0"/>
         <geometry>
             <mesh filename="${visual_mesh_file}" scale="1 1 1" />
@@ -13,5 +13,5 @@
         <!-- Se deben cambiar los parametros reales-->
     <collision>
-      <origin xyz="0 0 -4" rpy="0.0 0.0 0.0"/>
+      <origin xyz="0 0 -7" rpy="0.0 0.0 0.0"/>
       <geometry>
         <mesh filename="${visual_mesh_file}" scale="1 1 1" />
@@ -19,5 +19,5 @@
     </collision>
     <inertial>
-      <origin xyz="0 0 -4" rpy="0.0 0.0 0.0"/>
+      <origin xyz="0 0 -7" rpy="0.0 0.0 0.0"/>
       <mass value="1"/>
       <inertia

File: sim_challenges/urdf/gate.xacro (robot description, xacro)
@@ -6,5 +6,5 @@
 <link name="gate_base">
     <visual>
-        <origin xyz="0 0 -4" rpy="0.0 0.0 0"/>
+        <origin xyz="0 0 -7" rpy="0.0 0.0 0"/>
         <geometry>
             <mesh filename="${visual_mesh_file}" scale="1 1 1" />
@@ -13,5 +13,5 @@
         <!-- Se deben cambiar los parametros reales-->
     <collision>
-      <origin xyz="0 0 -4" rpy="0.0 0.0 0.0"/>
+      <origin xyz="0 0 -7" rpy="0.0 0.0 0.0"/>
       <geometry>
         <mesh filename="${visual_mesh_file}" scale="1 1 1" />
@@ -19,5 +19,5 @@
     </collision>
     <inertial>
-      <origin xyz="0 0 -4" rpy="0.0 0.0 0.0"/>
+      <origin xyz="0 0 -7" rpy="0.0 0.0 0.0"/>
       <mass value="1"/>
       <inertia

File: sim_challenges/urdf/octagon.xacro (robot description, xacro)
@@ -6,5 +6,5 @@
 <link name="octagon_base">
     <visual>
-        <origin xyz="0 0 -4" rpy="0.0 0.0 0.0"/>
+        <origin xyz="0 0 -7" rpy="0.0 0.0 0.0"/>
         <geometry>
             <mesh filename="${visual_mesh_file}" scale="1 1 1" />
@@ -13,5 +13,5 @@
         <!-- Se deben cambiar los parametros reales-->
     <collision>
-      <origin xyz="0 0 -4" rpy="0.0 0.0 0.0"/>
+      <origin xyz="0 0 -7" rpy="0.0 0.0 0.0"/>
       <geometry>
         <mesh filename="${visual_mesh_file}" scale="1 1 1" />
@@ -19,5 +19,5 @@
     </collision>
     <inertial>
-      <origin xyz="0 0 -4" rpy="0.0 0.0 0.0"/>
+      <origin xyz="0 0 -7" rpy="0.0 0.0 0.0"/>
       <mass value="1"/>
       <inertia

File: sim_challenges/urdf/pathmarkers/pathmarker1.xacro (robot description, xacro)
@@ -6,5 +6,5 @@
 <link name="path_marker_base">
     <visual>
-        <origin xyz="0 0 -5.5" rpy="0.0 0.0 0.0"/>
+        <origin xyz="0 0 -8.5" rpy="0.0 0.0 0.0"/>
         <geometry>
             <mesh filename="${visual_mesh_file}" scale="1 1 1" />
@@ -13,5 +13,5 @@
         <!-- Se deben cambiar los parametros reales-->
     <collision>
-      <origin xyz="0 0 -5.5" rpy="0.0 0.0 0.0"/>
+      <origin xyz="0 0 -8.5" rpy="0.0 0.0 0.0"/>
       <geometry>
         <mesh filename="${visual_mesh_file}" scale="1 1 1" />
@@ -19,5 +19,5 @@
     </collision>
     <inertial>
-      <origin xyz="0 0 -5.5" rpy="0.0 0.0 0.0"/>
+      <origin xyz="0 0 -8.5" rpy="0.0 0.0 0.0"/>
       <mass value="1"/>
       <inertia

File: sim_challenges/urdf/pathmarkers/pathmarker3.xacro (robot description, xacro)
@@ -6,5 +6,5 @@
 <link name="path_marker_base3">
     <visual>
-        <origin xyz="0 0 -5.5" rpy="0.0 0.0 0.0"/>
+        <origin xyz="0 0 -8.5" rpy="0.0 0.0 0.0"/>
         <geometry>
             <mesh filename="${visual_mesh_file}" scale="1 1 1" />
@@ -13,5 +13,5 @@
         <!-- Se deben cambiar los parametros reales-->
     <collision>
-      <origin xyz="0 0 -5.5" rpy="0.0 0.0 0.0"/>
+      <origin xyz="0 0 -8.5" rpy="0.0 0.0 0.0"/>
       <geometry>
         <mesh filename="${visual_mesh_file}" scale="1 1 1" />
@@ -19,5 +19,5 @@
     </collision>
     <inertial>
-      <origin xyz="0 0 -5.5" rpy="0.0 0.0 0.0"/>
+      <origin xyz="0 0 -8.5" rpy="0.0 0.0 0.0"/>
       <mass value="1"/>
       <inertia

File: sim_challenges/urdf/torpedos1.xacro (robot description, xacro)
@@ -6,5 +6,5 @@
 <link name="torpedos1_base">
     <visual>
-        <origin xyz="0 0 -4" rpy="0.0 0.0 0.0"/>
+        <origin xyz="0 0 -7" rpy="0.0 0.0 0.0"/>
         <geometry>
             <mesh filename="${visual_mesh_file}" scale="1 1 1" />
@@ -13,5 +13,5 @@
         <!-- Se deben cambiar los parametros reales-->
     <collision>
-      <origin xyz="0 0 -4" rpy="0.0 0.0 0.0"/>
+      <origin xyz="0 0 -7" rpy="0.0 0.0 0.0"/>
       <geometry>
         <mesh filename="${visual_mesh_file}" scale="1 1 1" />
@@ -19,5 +19,5 @@
     </collision>
     <inertial>
-      <origin xyz="0 0 -4" rpy="0.0 0.0 0.0"/>
+      <origin xyz="0 0 -7" rpy="0.0 0.0 0.0"/>
       <mass value="1"/>
       <inertia

File: sim_challenges/urdf/torpedos2.xacro (robot description, xacro)
@@ -6,5 +6,5 @@
 <link name="torpedos2_base">
     <visual>
-        <origin xyz="0 0 -4" rpy="0.0 0.0 0.0"/>
+        <origin xyz="0 0 -7" rpy="0.0 0.0 0.0"/>
         <geometry>
             <mesh filename="${visual_mesh_file}" scale="1 1 1" />
@@ -13,5 +13,5 @@
         <!-- Se deben cambiar los parametros reales-->
     <collision>
-      <origin xyz="0 0 -4" rpy="0.0 0.0 0.0"/>
+      <origin xyz="0 0 -7" rpy="0.0 0.0 0.0"/>
       <geometry>
         <mesh filename="${visual_mesh_file}" scale="1 1 1" />
@@ -19,5 +19,5 @@
     </collision>
     <inertial>
-      <origin xyz="0 0 -4" rpy="0.0 0.0 0.0"/>
+      <origin xyz="0 0 -7" rpy="0.0 0.0 0.0"/>
       <mass value="1"/>
       <inertia

Commit message: Torpedos

File: sim_challenges/urdf/bin1.xacro (robot description, xacro)
@@ -7,5 +7,5 @@
 <link name="bin1_base">
     <visual>
-        <origin xyz="0 0 -8.5" rpy="0.0 0.0 0.0"/>
+        <origin xyz="0 0 -7" rpy="0.0 0.0 0.0"/>
         <geometry>
             <mesh filename="${visual_mesh_file}" scale="1 1 1" />
@@ -14,5 +14,5 @@
         <!-- Se deben cambiar los parametros reales-->
     <collision>
-      <origin xyz="0 0 -8.5" rpy="0.0 0.0 0.0"/>
+      <origin xyz="0 0 -7" rpy="0.0 0.0 0.0"/>
       <geometry>
         <mesh filename="${visual_mesh_file}" scale="1 1 1" />
@@ -20,5 +20,5 @@
     </collision>
     <inertial>
-      <origin xyz="0 0 -8.5" rpy="0.0 0.0 0.0"/>
+      <origin xyz="0 0 -7" rpy="0.0 0.0 0.0"/>
       <mass value="1"/>
       <inertia

File: sim_challenges/urdf/bin2.xacro (robot description, xacro)
@@ -6,5 +6,5 @@
 <link name="bin2_base">
     <visual>
-        <origin xyz="0 0 -8.5" rpy="0.0 0.0 0.0"/>
+        <origin xyz="0 0 -7" rpy="0.0 0.0 0.0"/>
         <geometry>
             <mesh filename="${visual_mesh_file}" scale="1 1 1" />
@@ -13,5 +13,5 @@
         <!-- Se deben cambiar los parametros reales-->
     <collision>
-      <origin xyz="0 0 -8.5" rpy="0.0 0.0 0.0"/>
+      <origin xyz="0 0 -7" rpy="0.0 0.0 0.0"/>
       <geometry>
         <mesh filename="${visual_mesh_file}" scale="1 1 1" />
@@ -19,5 +19,5 @@
     </collision>
     <inertial>
-      <origin xyz="0 0 -8.5" rpy="0.0 0.0 0.0"/>
+      <origin xyz="0 0 -7" rpy="0.0 0.0 0.0"/>
       <mass value="1"/>
       <inertia

File: sim_challenges/urdf/torpedos1.xacro (robot description, xacro)
@@ -2,5 +2,5 @@
 <robot name="torpedos_1" xmlns:xacro="http://www.ros.org/wiki/xacro">
 <!-- Introducir meshes -->
-<xacro:property name="visual_mesh_file" value="file://$(find sim_challenges)/models/meshes/Mytorpedo1.dae" />
+<xacro:property name="visual_mesh_file" value="file://$(find sim_challenges)/models/meshes/finaltorpedos.dae" />
 <!-- <origin xyz="0.085 (0 -0.085) 0 0" rpy="0.0 0.0 1.57075"/> -->
 <link name="torpedos1_base">

Commit message: Change pathmarker and location obstacles

File: sim_challenges/urdf/bin1.xacro (robot description, xacro)
@@ -7,5 +7,5 @@
 <link name="bin1_base">
     <visual>
-        <origin xyz="0 0 -7" rpy="0.0 0.0 0.0"/>
+        <origin xyz="0 2 -7" rpy="0.0 0.0 0.0"/>
         <geometry>
             <mesh filename="${visual_mesh_file}" scale="1 1 1" />
@@ -14,5 +14,5 @@
         <!-- Se deben cambiar los parametros reales-->
     <collision>
-      <origin xyz="0 0 -7" rpy="0.0 0.0 0.0"/>
+      <origin xyz="0 2 -7" rpy="0.0 0.0 0.0"/>
       <geometry>
         <mesh filename="${visual_mesh_file}" scale="1 1 1" />
@@ -20,5 +20,5 @@
     </collision>
     <inertial>
-      <origin xyz="0 0 -7" rpy="0.0 0.0 0.0"/>
+      <origin xyz="0 2 -7" rpy="0.0 0.0 0.0"/>
       <mass value="1"/>
       <inertia

File: sim_challenges/urdf/bin2.xacro (robot description, xacro)
@@ -6,5 +6,5 @@
 <link name="bin2_base">
     <visual>
-        <origin xyz="0 0 -7" rpy="0.0 0.0 0.0"/>
+        <origin xyz="0 2 -7" rpy="0.0 0.0 0.0"/>
         <geometry>
             <mesh filename="${visual_mesh_file}" scale="1 1 1" />
@@ -13,5 +13,5 @@
         <!-- Se deben cambiar los parametros reales-->
     <collision>
-      <origin xyz="0 0 -7" rpy="0.0 0.0 0.0"/>
+      <origin xyz="0 2 -7" rpy="0.0 0.0 0.0"/>
       <geometry>
         <mesh filename="${visual_mesh_file}" scale="1 1 1" />
@@ -19,5 +19,5 @@
     </collision>
     <inertial>
-      <origin xyz="0 0 -7" rpy="0.0 0.0 0.0"/>
+      <origin xyz="0 2 -7" rpy="0.0 0.0 0.0"/>
       <mass value="1"/>
       <inertia

File: sim_challenges/urdf/buoy.xacro (robot description, xacro)
@@ -6,5 +6,5 @@
 <link name="buoy1_base">
     <visual>
-        <origin xyz="0 0 -7" rpy="0.0 0.0 0.0"/>
+        <origin xyz="0 2 -7" rpy="0.0 0.0 0.0"/>
         <geometry>
             <mesh filename="${visual_mesh_file}" scale="1 1 1" />
@@ -13,5 +13,5 @@
         <!-- Se deben cambiar los parametros reales-->
     <collision>
-      <origin xyz="0 0 -7" rpy="0.0 0.0 0.0"/>
+      <origin xyz="0 2 -7" rpy="0.0 0.0 0.0"/>
       <geometry>
         <mesh filename="${visual_mesh_file}" scale="1 1 1" />
@@ -19,5 +19,5 @@
     </collision>
     <inertial>
-      <origin xyz="0 0 -7" rpy="0.0 0.0 0.0"/>
+      <origin xyz="0 2 -7" rpy="0.0 0.0 0.0"/>
       <mass value="1"/>
       <inertia

File: sim_challenges/urdf/buoy2.xacro (robot description, xacro)
@@ -6,5 +6,5 @@
 <link name="buoy2_base">
     <visual>
-        <origin xyz="0 0 -7" rpy="0.0 0.0 0.0"/>
+        <origin xyz="0 2 -7" rpy="0.0 0.0 0.0"/>
         <geometry>
             <mesh filename="${visual_mesh_file}" scale="1 1 1" />
@@ -13,5 +13,5 @@
         <!-- Se deben cambiar los parametros reales-->
     <collision>
-      <origin xyz="0 0 -7" rpy="0.0 0.0 0.0"/>
+      <origin xyz="0 2 -7" rpy="0.0 0.0 0.0"/>
       <geometry>
         <mesh filename="${visual_mesh_file}" scale="1 1 1" />
@@ -19,5 +19,5 @@
     </collision>
     <inertial>
-      <origin xyz="0 0 -7" rpy="0.0 0.0 0.0"/>
+      <origin xyz="0 2 -7" rpy="0.0 0.0 0.0"/>
       <mass value="1"/>
       <inertia

File: sim_challenges/urdf/octagon.xacro (robot description, xacro)
@@ -6,5 +6,5 @@
 <link name="octagon_base">
     <visual>
-        <origin xyz="0 0 -7" rpy="0.0 0.0 0.0"/>
+        <origin xyz="0 2 -7" rpy="0.0 0.0 0.0"/>
         <geometry>
             <mesh filename="${visual_mesh_file}" scale="1 1 1" />
@@ -13,5 +13,5 @@
         <!-- Se deben cambiar los parametros reales-->
     <collision>
-      <origin xyz="0 0 -7" rpy="0.0 0.0 0.0"/>
+      <origin xyz="0 2 -7" rpy="0.0 0.0 0.0"/>
       <geometry>
         <mesh filename="${visual_mesh_file}" scale="1 1 1" />
@@ -19,5 +19,5 @@
     </collision>
     <inertial>
-      <origin xyz="0 0 -7" rpy="0.0 0.0 0.0"/>
+      <origin xyz="0 2 -7" rpy="0.0 0.0 0.0"/>
       <mass value="1"/>
       <inertia

File: sim_challenges/urdf/pathmarkers/pathmarker3.xacro (robot description, xacro)
@@ -6,5 +6,5 @@
 <link name="path_marker_base3">
     <visual>
-        <origin xyz="0 0 -8.5" rpy="0.0 0.0 0.0"/>
+        <origin xyz="0 2 -8.5" rpy="0.0 0.0 0.0"/>
         <geometry>
             <mesh filename="${visual_mesh_file}" scale="1 1 1" />
@@ -13,5 +13,5 @@
         <!-- Se deben cambiar los parametros reales-->
     <collision>
-      <origin xyz="0 0 -8.5" rpy="0.0 0.0 0.0"/>
+      <origin xyz="0 2 -8.5" rpy="0.0 0.0 0.0"/>
       <geometry>
         <mesh filename="${visual_mesh_file}" scale="1 1 1" />
@@ -19,5 +19,5 @@
     </collision>
     <inertial>
-      <origin xyz="0 0 -8.5" rpy="0.0 0.0 0.0"/>
+      <origin xyz="0 2 -8.5" rpy="0.0 0.0 0.0"/>
       <mass value="1"/>
       <inertia

File: sim_challenges/urdf/torpedos1.xacro (robot description, xacro)
@@ -6,5 +6,5 @@
 <link name="torpedos1_base">
     <visual>
-        <origin xyz="0 0 -7" rpy="0.0 0.0 0.0"/>
+        <origin xyz="0 2 -7" rpy="0.0 0.0 0.0"/>
         <geometry>
             <mesh filename="${visual_mesh_file}" scale="1 1 1" />
@@ -13,5 +13,5 @@
         <!-- Se deben cambiar los parametros reales-->
     <collision>
-      <origin xyz="0 0 -7" rpy="0.0 0.0 0.0"/>
+      <origin xyz="0 2 -7" rpy="0.0 0.0 0.0"/>
       <geometry>
         <mesh filename="${visual_mesh_file}" scale="1 1 1" />
@@ -19,5 +19,5 @@
     </collision>
     <inertial>
-      <origin xyz="0 0 -7" rpy="0.0 0.0 0.0"/>
+      <origin xyz="0 2 -7" rpy="0.0 0.0 0.0"/>
       <mass value="1"/>
       <inertia

File: sim_challenges/urdf/torpedos2.xacro (robot description, xacro)
@@ -6,5 +6,5 @@
 <link name="torpedos2_base">
     <visual>
-        <origin xyz="0 0 -7" rpy="0.0 0.0 0.0"/>
+        <origin xyz="0 2 -7" rpy="0.0 0.0 0.0"/>
         <geometry>
             <mesh filename="${visual_mesh_file}" scale="1 1 1" />
@@ -13,5 +13,5 @@
         <!-- Se deben cambiar los parametros reales-->
     <collision>
-      <origin xyz="0 0 -7" rpy="0.0 0.0 0.0"/>
+      <origin xyz="0 2 -7" rpy="0.0 0.0 0.0"/>
       <geometry>
         <mesh filename="${visual_mesh_file}" scale="1 1 1" />
@@ -19,5 +19,5 @@
     </collision>
     <inertial>
-      <origin xyz="0 0 -7" rpy="0.0 0.0 0.0"/>
+      <origin xyz="0 2 -7" rpy="0.0 0.0 0.0"/>
       <mass value="1"/>
       <inertia

Commit message: BIn position .dae

File: sim_challenges/urdf/bin1.xacro (robot description, xacro)
@@ -7,5 +7,5 @@
 <link name="bin1_base">
     <visual>
-        <origin xyz="0 2 -7" rpy="0.0 0.0 0.0"/>
+        <origin xyz="0 1.5 -7" rpy="0.0 0.0 0.0"/>
         <geometry>
             <mesh filename="${visual_mesh_file}" scale="1 1 1" />
@@ -14,5 +14,5 @@
         <!-- Se deben cambiar los parametros reales-->
     <collision>
-      <origin xyz="0 2 -7" rpy="0.0 0.0 0.0"/>
+      <origin xyz="0 1.5 -7" rpy="0.0 0.0 0.0"/>
       <geometry>
         <mesh filename="${visual_mesh_file}" scale="1 1 1" />
@@ -20,5 +20,5 @@
     </collision>
     <inertial>
-      <origin xyz="0 2 -7" rpy="0.0 0.0 0.0"/>
+      <origin xyz="0 1.5 -7" rpy="0.0 0.0 0.0"/>
       <mass value="1"/>
       <inertia
