Commit message: working

File: sim_challenges/urdf/torpedos1.xacro (robot description, xacro)
@@ -2,22 +2,22 @@
 <robot name="torpedos_1" xmlns:xacro="http://www.ros.org/wiki/xacro">
 <!-- Introducir meshes -->
-<xacro:property name="visual_mesh_file" value="file://$(find sim_challenges)/models/meshes/Mytorpedo1.dae" />
+<xacro:property name="visual_mesh_file" value="file://$(find sim_challenges)/models/meshes/finaltorpedos.dae" />
 <!-- <origin xyz="0.085 (0 -0.085) 0 0" rpy="0.0 0.0 1.57075"/> -->
 <link name="torpedos1_base">
     <visual>
-        <origin xyz="25.180420 1.835166 -4.0" rpy="0.0 0.0 1.57"/>
+        <origin xyz="0 0 -4.0" rpy="0.0 0.0 1.57"/>
         <geometry>
-            <mesh filename="${visual_mesh_file}" scale="1 1 1" />
+            <mesh filename="${visual_mesh_file}" scale="0.1 0.1 0.1" />
         </geometry>
     </visual>
         <!-- Se deben cambiar los parametros reales-->
     <collision>
-      <origin xyz="25.180420 1.835166 -4.0" rpy="0.0 0.0 1.57"/>
+      <origin xyz="0.0 0.0 1.57" rpy="0.0 0.0 1.57"/>
       <geometry>
-        <mesh filename="${visual_mesh_file}" scale="1 1 1" />
+        <mesh filename="${visual_mesh_file}" scale="0.1 0.1 0.1" />
       </geometry>
     </collision>
     <inertial>
-      <origin xyz="25.180420 1.835166 -4.0" rpy="0.0 0.0 1.57"/>
+      <origin xyz="0.0 0.0 1.57" rpy="0.0 0.0 1.57"/>
       <mass value="1"/>
       <inertia
