Commit message: Commented collisions on boat and lidar

File: sensors/velodyne_simulator/velodyne_description/urdf/VLP-16.urdf.xacro (robot description, xacro)
@@ -26,10 +26,10 @@
         </geometry>
       </visual>
-      <collision>
+      <!-- <collision>
         <origin rpy="0 0 0" xyz="0 0 0.03585"/>
         <geometry>
           <cylinder radius="0.0516" length="0.0717"/>
         </geometry>
-      </collision>
+      </collision> -->
     </link>
     <joint name="${name}_base_scan_joint" type="fixed" >

File: vtec_s3_description/urdf/base.xacro (robot description, xacro)
@@ -50,11 +50,11 @@
           </geometry>
         </visual>
-        <collision>
+        <!-- <collision>
           <origin xyz="0.05 0 0.19" rpy="0 0 0"/>
           <geometry>
             <box size="${x_size} ${y_size} ${z_size}"/>
-            <!-- <mesh filename="${collision_mesh_file}" scale="0.001 0.001 0.001" /> --> <!-- To improve performance, we replaced it by a box -->
+            <mesh filename="${collision_mesh_file}" scale="0.001 0.001 0.001" />  To improve performance, we replaced it by a box
           </geometry>
-        </collision>
+        </collision> -->
       </link>
     <gazebo reference="${namespace}/base_link">
