Commit message: new map

File: sim_challenges/urdf/pathmarkers/pathmarker1.xacro (robot description, xacro)
@@ -6,5 +6,5 @@
 <link name="path_marker_base">
     <visual>
-        <origin xyz="0 0 -4" rpy="0.0 0.0 0.0"/>
+        <origin xyz="0 0 -5.5" rpy="0.0 0.0 0.0"/>
         <geometry>
             <mesh filename="${visual_mesh_file}" scale="1 1 1" />
@@ -13,5 +13,5 @@
         <!-- Se deben cambiar los parametros reales-->
     <collision>
-      <origin xyz="0 0 -4" rpy="0.0 0.0 0.0"/>
+      <origin xyz="0 0 -5.5" rpy="0.0 0.0 0.0"/>
       <geometry>
         <mesh filename="${visual_mesh_file}" scale="1 1 1" />
@@ -19,5 +19,5 @@
     </collision>
     <inertial>
-      <origin xyz="0 0 -4" rpy="0.0 0.0 0.0"/>
+      <origin xyz="0 0 -5.5" rpy="0.0 0.0 0.0"/>
       <mass value="1"/>
       <inertia

File: sim_challenges/urdf/pathmarkers/pathmarker3.xacro (robot description, xacro)
@@ -6,5 +6,5 @@
 <link name="path_marker_base3">
     <visual>
-        <origin xyz="0 0 -4" rpy="0.0 0.0 0.0"/>
+        <origin xyz="0 0 -5.5" rpy="0.0 0.0 0.0"/>
         <geometry>
             <mesh filename="${visual_mesh_file}" scale="1 1 1" />
@@ -13,5 +13,5 @@
         <!-- Se deben cambiar los parametros reales-->
     <collision>
-      <origin xyz="0 0 -4" rpy="0.0 0.0 0.0"/>
+      <origin xyz="0 0 -5.5" rpy="0.0 0.0 0.0"/>
       <geometry>
         <mesh filename="${visual_mesh_file}" scale="1 1 1" />
@@ -19,5 +19,5 @@
     </collision>
     <inertial>
-      <origin xyz="0 0 -4" rpy="0.0 0.0 0.0"/>
+      <origin xyz="0 0 -5.5" rpy="0.0 0.0 0.0"/>
       <mass value="1"/>
       <inertia
