Commit message: fixed files

File: vehicle_descriptions/robots/vtec_s3.xacro (robot description, xacro)
@@ -4,7 +4,7 @@
   <xacro:arg name="namespace" default="vtec_s3"/>
   <xacro:arg name="inertial_reference_frame" default="world_ned"/>
-  <xacro:include filename="$(find vehicles_descriptions)/urdf/USVs/vtec_s3_base.xacro"/>
+  <xacro:include filename="$(find vehicle_descriptions)/urdf/USVs/vtec_s3_base.xacro"/>
   <xacro:include filename="$(find uuv_sensor_ros_plugins)/urdf/sensor_snippets.xacro"/>
-  <!-- <xacro:include filename="$(find vehicles_descriptions)/urdf/USVs/vtec_s3_sensors.xacro"/> -->
+  <!-- <xacro:include filename="$(find vehicle_descriptions)/urdf/USVs/vtec_s3_sensors.xacro"/> -->
   <xacro:include filename="$(find velodyne_description)/urdf/VLP-16.urdf.xacro"/>
   <xacro:vtec_s3_base namespace="$(arg namespace)"/>

File: vehicle_descriptions/robots/vtec_u3.xacro (robot description, xacro)
@@ -4,9 +4,9 @@
   <xacro:arg name="namespace" default="vtec_u3"/>
   <xacro:arg name="inertial_reference_frame" default="world_ned"/>
-  <xacro:include filename="$(find vehicles_descriptions)/urdf/UUVs/vtec_u3_base.xacro"/>
+  <xacro:include filename="$(find vehicle_descriptions)/urdf/UUVs/vtec_u3_base.xacro"/>
   <xacro:include filename="$(find uuv_sensor_ros_plugins)/urdf/sensor_snippets.xacro"/>
-  <xacro:include filename="$(find vehicles_descriptions)/urdf/UUVs/vtec_u3_sensors.xacro"/>
-  <xacro:include filename="$(find vehicles_descriptions)/urdf/UUVs/vtec_u3_arm.xacro"/>
-  <xacro:include filename="$(find vehicles_descriptions)/urdf/UUVs/vtec_u3_shooter.xacro"/>
+  <xacro:include filename="$(find vehicle_descriptions)/urdf/UUVs/vtec_u3_sensors.xacro"/>
+  <xacro:include filename="$(find vehicle_descriptions)/urdf/UUVs/vtec_u3_arm.xacro"/>
+  <xacro:include filename="$(find vehicle_descriptions)/urdf/UUVs/vtec_u3_shooter.xacro"/>
   <xacro:vtec_u3_base namespace="$(arg namespace)"/>
   <xacro:vtec_u3_sensors namespace="$(arg namespace)"/>

File: vehicle_descriptions/urdf/USVs/vtec_s3_base.xacro (robot description, xacro)
@@ -11,5 +11,5 @@
     the mesh pose will have to be corrected below in the <visual> block.
   -->
-  <xacro:property name="visual_mesh_file" value="file://$(find vehicles_descriptions)/meshes/vtec_s3.dae"/>
+  <xacro:property name="visual_mesh_file" value="file://$(find vehicle_descriptions)/meshes/vtec_s3.dae"/>
   <!--
     Collision geometry mesh, usually in STL format (it is recommended to keep
@@ -17,5 +17,5 @@
     regarding the computation of collision forces)
   -->
-  <xacro:property name="collision_mesh_file" value="file://$(find vehicles_descriptions)/meshes/vtec_s3.stl"/>
+  <xacro:property name="collision_mesh_file" value="file://$(find vehicle_descriptions)/meshes/vtec_s3.stl"/>
   <xacro:macro name="vtec_s3_base" params="namespace">
       <link name="${namespace}_base_link">

File: vehicle_descriptions/urdf/UUVs/vtec_u3_arm.xacro (robot description, xacro)
@@ -57,5 +57,5 @@
         <origin xyz="0 0 0" rpi="0 0 0"/>
         <geometry>
-          <mesh filename="package://vehicles_descriptions/meshes/arm/arm_rail.stl" />
+          <mesh filename="package://vehicle_descriptions/meshes/arm/arm_rail.stl" />
         </geometry>
       </visual>
@@ -64,5 +64,5 @@
         <origin xyz="0 0 0" rpy="0 0 0" />
         <geometry>
-          <mesh filename="package://vehicles_descriptions/meshes/arm/arm_rail.stl" />
+          <mesh filename="package://vehicle_descriptions/meshes/arm/arm_rail.stl" />
         </geometry>
       </collision> -->
@@ -84,11 +84,11 @@
         <origin xyz="0 0 0" rpy="0 0 0" />
         <geometry>
-          <mesh filename="package://vehicles_descriptions/meshes/arm/extendible_arm.stl" />
-        </geometry>
-      </visual>
-      <!-- <collision>
-        <origin xyz="0 0 0" rpy="0 0 0" />
-        <geometry>
-          <mesh filename="package://vehicles_descriptions/meshes/arm/extendible_arm.stl" />
+          <mesh filename="package://vehicle_descriptions/meshes/arm/extendible_arm.stl" />
+        </geometry>
+      </visual>
+      <!-- <collision>
+        <origin xyz="0 0 0" rpy="0 0 0" />
+        <geometry>
+          <mesh filename="package://vehicle_descriptions/meshes/arm/extendible_arm.stl" />
         </geometry>
       </collision> -->
@@ -110,11 +110,11 @@
         <origin xyz="0 0 0" rpy="0 0 0" />
         <geometry>
-          <mesh filename="package://vehicles_descriptions/meshes/arm/left_beam.stl" />
-        </geometry>
-      </visual>
-      <!-- <collision>
-        <origin xyz="0 0 0" rpy="0 0 0" />
-        <geometry>
-          <mesh filename="package://vehicles_descriptions/meshes/arm/left_beam.stl" />
+          <mesh filename="package://vehicle_descriptions/meshes/arm/left_beam.stl" />
+        </geometry>
+      </visual>
+      <!-- <collision>
+        <origin xyz="0 0 0" rpy="0 0 0" />
+        <geometry>
+          <mesh filename="package://vehicle_descriptions/meshes/arm/left_beam.stl" />
         </geometry>
       </collision> -->
@@ -137,11 +137,11 @@
         <origin xyz="0 0 0" rpy="0 0 0" />
         <geometry>
-          <mesh filename="package://vehicles_descriptions/meshes/arm/left_tip.stl" />
-        </geometry>
-      </visual>
-      <!-- <collision>
-        <origin xyz="0 0 0" rpy="0 0 0" />
-        <geometry>
-          <mesh filename="package://vehicles_descriptions/meshes/arm/left_tip.stl" />
+          <mesh filename="package://vehicle_descriptions/meshes/arm/left_tip.stl" />
+        </geometry>
+      </visual>
+      <!-- <collision>
+        <origin xyz="0 0 0" rpy="0 0 0" />
+        <geometry>
+          <mesh filename="package://vehicle_descriptions/meshes/arm/left_tip.stl" />
         </geometry>
       </collision> -->
@@ -164,11 +164,11 @@
         <origin xyz="0 0 0" rpy="0 0 0" />
         <geometry>
-          <mesh filename="package://vehicles_descriptions/meshes/arm/right_beam.stl" />
-        </geometry>
-      </visual>
-      <!-- <collision>
-        <origin xyz="0 0 0" rpy="0 0 0" />
-        <geometry>
-          <mesh filename="package://vehicles_descriptions/meshes/arm/right_beam.stl" />
+          <mesh filename="package://vehicle_descriptions/meshes/arm/right_beam.stl" />
+        </geometry>
+      </visual>
+      <!-- <collision>
+        <origin xyz="0 0 0" rpy="0 0 0" />
+        <geometry>
+          <mesh filename="package://vehicle_descriptions/meshes/arm/right_beam.stl" />
         </geometry>
       </collision> -->
@@ -191,11 +191,11 @@
         <origin xyz="0 0 0" rpy="0 0 0" />
         <geometry>
-          <mesh filename="package://vehicles_descriptions/meshes/arm/right_tip.stl" />
-        </geometry>
-      </visual>
-      <!-- <collision>
-        <origin xyz="0 0 0" rpy="0 0 0" />
-        <geometry>
-          <mesh filename="package://vehicles_descriptions/meshes/arm/right_tip.stl" />
+          <mesh filename="package://vehicle_descriptions/meshes/arm/right_tip.stl" />
+        </geometry>
+      </visual>
+      <!-- <collision>
+        <origin xyz="0 0 0" rpy="0 0 0" />
+        <geometry>
+          <mesh filename="package://vehicle_descriptions/meshes/arm/right_tip.stl" />
         </geometry>
       </collision> -->

File: vehicle_descriptions/urdf/UUVs/vtec_u3_base.xacro (robot description, xacro)
@@ -12,5 +12,5 @@
     the mesh pose will have to be corrected below in the <visual> block.
   -->
-  <xacro:property name="visual_mesh_file" value="file://$(find vehicles_descriptions)/meshes/vtec_u3.dae"/>
+  <xacro:property name="visual_mesh_file" value="file://$(find vehicle_descriptions)/meshes/vtec_u3.dae"/>
   <!--
     Collision geometry mesh, usually in STL format (it is recommended to keep
@@ -18,5 +18,5 @@
     regarding the computation of collision forces)
   -->
-  <xacro:property name="collision_mesh_file" value="file://$(find vehicles_descriptions)/meshes/vtec_u3.stl"/>
+  <xacro:property name="collision_mesh_file" value="file://$(find vehicle_descriptions)/meshes/vtec_u3.stl"/>
   <xacro:macro name="vtec_u3_base" params="namespace">
       <link name="${namespace}_base_link">

File: vehicle_descriptions/urdf/UUVs/vtec_u3_shooter.xacro (robot description, xacro)
@@ -2,6 +2,6 @@
 <robot xmlns:xacro="http://www.ros.org/wiki/xacro">
   <xacro:macro name="vtec_u3_shooter" params="parent">
-    <xacro:property name="visual_mesh_file" value="file://$(find vehicles_descriptions)/meshes/shooter/shooter_base.dae" />
-    <!-- <xacro:property name="collision_mesh_file" value="file://$(find vehicles_descriptions)/meshes/shooter/shooter_base.dae"/> -->
+    <xacro:property name="visual_mesh_file" value="file://$(find vehicle_descriptions)/meshes/shooter/shooter_base.dae" />
+    <!-- <xacro:property name="collision_mesh_file" value="file://$(find vehicle_descriptions)/meshes/shooter/shooter_base.dae"/> -->
     <gazebo reference="shooter_base_link">
         <material>Gazebo/White</material>
