Commit message: Renamed package

File: vehicle_descriptions/robots/vtec_u3.xacro (robot description, xacro)
@@ -6,9 +6,9 @@
   <xacro:include filename="$(find vehicles_descriptions)/urdf/UUVs/vtec_u3_base.xacro"/>
   <xacro:include filename="$(find uuv_sensor_ros_plugins)/urdf/sensor_snippets.xacro"/>
-  <!-- <xacro:include filename="$(find vehicles_descriptions)/urdf/UUVs/vtec_u3_sensors.xacro"/>  -->
+  <xacro:include filename="$(find vehicles_descriptions)/urdf/UUVs/vtec_u3_sensors.xacro"/>
   <xacro:include filename="$(find vehicles_descriptions)/urdf/UUVs/vtec_u3_arm.xacro"/>
   <xacro:include filename="$(find vehicles_descriptions)/urdf/UUVs/vtec_u3_shooter.xacro"/>
   <xacro:vtec_u3_base namespace="$(arg namespace)"/>
-  <!-- <xacro:vtec_u3_sensors namespace="$(arg namespace)"/> -->
+  <xacro:vtec_u3_sensors namespace="$(arg namespace)"/>
   <xacro:vtec_u3_arm parent="$(arg namespace)"/>
   <xacro:vtec_u3_shooter parent="$(arg namespace)"/>

File: vehicle_descriptions/urdf/UUVs/vtec_u3_sensors.xacro (robot description, xacro)
@@ -36,5 +36,5 @@
     <!-- Realsense R200 -->
     <xacro:realsense_camera namespace="${namespace}" parent_link="${namespace}_base_link" suffix="down">
-      <origin xyz="0.0 0.01961 0.18" rpy="0 -1.57 0"/>
+      <origin xyz="0.0 0.01961 0.18" rpy="0 1.57 0"/>
     </xacro:realsense_camera>
     <!-- Realsense R200 -->

Commit message: Add files via upload

File: vehicle_descriptions/robots/vtec_u3.xacro (robot description, xacro)
@@ -5,12 +5,12 @@
   <xacro:arg name="inertial_reference_frame" default="world_ned"/>
   <xacro:include filename="$(find vehicle_descriptions)/urdf/UUVs/vtec_u3_base.xacro"/>
-  <!-- <xacro:include filename="$(find vehicle_descriptions)/urdf/UUVs/vtec_u3_sensors.xacro"/>
+  <xacro:include filename="$(find vehicle_descriptions)/urdf/UUVs/vtec_u3_sensors.xacro"/>
   <xacro:include filename="$(find vehicle_descriptions)/urdf/UUVs/vtec_u3_arm.xacro"/>
-  <xacro:include filename="$(find vehicle_descriptions)/urdf/UUVs/vtec_u3_shooter.xacro"/>  -->
+  <xacro:include filename="$(find vehicle_descriptions)/urdf/UUVs/vtec_u3_shooter.xacro"/>
   <virtual_joint name="world_joint" type="planar" parent_frame="world_ned" child_link="vtec_u3_base_link"/>
   <xacro:vtec_u3_base namespace="$(arg namespace)"/>
-  <!-- <xacro:vtec_u3_sensors namespace="$(arg namespace)"/>
+  <xacro:vtec_u3_sensors namespace="$(arg namespace)"/>
   <xacro:vtec_u3_arm parent="$(arg namespace)"/>
-  <xacro:vtec_u3_shooter parent="$(arg namespace)"/> -->
+  <xacro:vtec_u3_shooter parent="$(arg namespace)"/>
   <!-- Joint state publisher plugin -->
   <!-- <xacro:default_joint_state_publisher namespace="$(arg namespace)" update_rate="10"/> -->

File: vehicle_descriptions/urdf/UUVs/vtec_u3_sensors.xacro (robot description, xacro)
@@ -2,4 +2,6 @@
 <robot xmlns:xacro="http://www.ros.org/wiki/xacro">
   <xacro:include filename="$(find uuv_sensor_ros_plugins)/urdf/sensor_snippets.xacro"/>
+  <include filename="$(find realsense_gazebo_plugin)/models/realsense_camera/model.sdf"/>
+  <xacro:include filename="$(find realsense_gazebo_plugin)/urdf/realsense-RS200.macro.xacro"/>
   <!--
     Some examples of sensors that can be added to the vehicle frame.
@@ -32,11 +34,11 @@
     </xacro:default_imu>
     <!-- Realsense R200 1-->
-    <xacro:realsense_camera namespace="${namespace}" parent_link="${namespace}_base_link" suffix="front">
+    <xacro:realsense-rs200 prefix="front" parent="${namespace}_base_link">
       <origin xyz="0.19281 0.01961 0.06659" rpy="0 0 0"/>
-    </xacro:realsense_camera>
+    </xacro:realsense-rs200>
     <!-- Realsense R200 -->
-    <xacro:realsense_camera namespace="${namespace}" parent_link="${namespace}_base_link" suffix="down">
-      <origin xyz="0.0 0.01961 0.18" rpy="0 1.57 0"/>
-    </xacro:realsense_camera>
+    <xacro:realsense-rs200 prefix="down" parent="${namespace}_base_link">
+      <origin xyz="0.0 0.01961 0.3" rpy="0 -1.57 0"/>
+    </xacro:realsense-rs200>
     <!-- Realsense R200 -->
     <!-- Import macro for realsense-RS200 camera-->
