Commit message: Removed unnecessary package

File: uv_worlds/urdf/bin1.xacro (robot description, xacro)
@@ -1,8 +1,9 @@
 <?xml version="1.0"?>
-<robot name="octagon_1" xmlns:xacro="http://www.ros.org/wiki/xacro">
+<robot name="bin_1" xmlns:xacro="http://www.ros.org/wiki/xacro">
+<!--Change .dae to binopen.dae, bintapadod.dae, bintapadoi.dae depending on the situation-->
 <!-- Introducir meshes -->
-<xacro:property name="visual_mesh_file" value="file://$(find sim_challenges)/models/meshes/Myoctagon2.dae" />
+<xacro:property name="visual_mesh_file" value="file://$(find uv_worlds)/models/props//bintapadoi.dae" />
 <!-- <origin xyz="0.085 (0 -0.085) 0 0" rpy="0.0 0.0 1.57075"/> -->
-<link name="octagon_base">
+<link name="bin1_base">
     <visual>
         <origin xyz="0 2 -7" rpy="0.0 0.0 0.0"/>
@@ -27,5 +28,5 @@
     </inertial>
 </link>
-<gazebo reference="octagon_base">
+<gazebo reference="bin1_base">
   <selfCollide>0</selfCollide>
   <turnGravityOff>1</turnGravityOff>

File: uv_worlds/urdf/bin2.xacro (robot description, xacro)
@@ -1,8 +1,8 @@
 <?xml version="1.0"?>
-<robot name="buoy_1" xmlns:xacro="http://www.ros.org/wiki/xacro">
+<robot name="bin_2" xmlns:xacro="http://www.ros.org/wiki/xacro">
 <!-- Introducir meshes -->
-<xacro:property name="visual_mesh_file" value="file://$(find sim_challenges)/models/meshes/buoy1.dae" />
+<xacro:property name="visual_mesh_file" value="file://$(find uv_worlds)/models/props//bin02.dae" />
 <!-- <origin xyz="0.085 (0 -0.085) 0 0" rpy="0.0 0.0 1.57075"/> -->
-<link name="buoy1_base">
+<link name="bin2_base">
     <visual>
         <origin xyz="0 2 -7" rpy="0.0 0.0 0.0"/>
@@ -27,5 +27,5 @@
     </inertial>
 </link>
-<gazebo reference="buoy1_base">
+<gazebo reference="bin2_base">
   <selfCollide>0</selfCollide>
   <turnGravityOff>1</turnGravityOff>

File: uv_worlds/urdf/buoy.xacro (robot description, xacro)
@@ -1,10 +1,10 @@
 <?xml version="1.0"?>
-<robot name="path_marker6" xmlns:xacro="http://www.ros.org/wiki/xacro">
+<robot name="buoy_1" xmlns:xacro="http://www.ros.org/wiki/xacro">
 <!-- Introducir meshes -->
-<xacro:property name="visual_mesh_file" value="file://$(find sim_challenges)/models/meshes/pathmarkers/pathmarker6.dae" />
-<!-- <origin xyz="0.085 (0 -0.085) 0 0" rpy="0.0 0.0 0.0075"/> -->
-<link name="path_marker_base6">
+<xacro:property name="visual_mesh_file" value="file://$(find uv_worlds)/models/props//buoy1.dae" />
+<!-- <origin xyz="0.085 (0 -0.085) 0 0" rpy="0.0 0.0 1.57075"/> -->
+<link name="buoy1_base">
     <visual>
-        <origin xyz="0 0 -4" rpy="0.0 0.0 0.0"/>
+        <origin xyz="0 2 -7" rpy="0.0 0.0 0.0"/>
         <geometry>
             <mesh filename="${visual_mesh_file}" scale="1 1 1" />
@@ -13,5 +13,5 @@
         <!-- Se deben cambiar los parametros reales-->
     <collision>
-      <origin xyz="0 0 -4" rpy="0.0 0.0 0.0"/>
+      <origin xyz="0 2 -7" rpy="0.0 0.0 0.0"/>
       <geometry>
         <mesh filename="${visual_mesh_file}" scale="1 1 1" />
@@ -19,5 +19,5 @@
     </collision>
     <inertial>
-      <origin xyz="0 0 -4" rpy="0.0 0.0 0.0"/>
+      <origin xyz="0 2 -7" rpy="0.0 0.0 0.0"/>
       <mass value="1"/>
       <inertia
@@ -27,5 +27,5 @@
     </inertial>
 </link>
-<gazebo reference="path_marker_base6">
+<gazebo reference="buoy1_base">
   <selfCollide>0</selfCollide>
   <turnGravityOff>1</turnGravityOff>

File: uv_worlds/urdf/buoy2.xacro (robot description, xacro)
@@ -1,10 +1,10 @@
 <?xml version="1.0"?>
-<robot name="gate_1" xmlns:xacro="http://www.ros.org/wiki/xacro">
+<robot name="buoy_2" xmlns:xacro="http://www.ros.org/wiki/xacro">
 <!-- Introducir meshes -->
-<xacro:property name="visual_mesh_file" value="file://$(find sim_challenges)/models/meshes/mygate1.dae" />
+<xacro:property name="visual_mesh_file" value="file://$(find uv_worlds)/models/props//buoy2.dae" />
 <!-- <origin xyz="0.085 (0 -0.085) 0 0" rpy="0.0 0.0 1.57075"/> -->
-<link name="gate_base">
+<link name="buoy2_base">
     <visual>
-        <origin xyz="0 0 -7" rpy="0.0 0.0 0"/>
+        <origin xyz="0 2 -7" rpy="0.0 0.0 0.0"/>
         <geometry>
             <mesh filename="${visual_mesh_file}" scale="1 1 1" />
@@ -13,5 +13,5 @@
         <!-- Se deben cambiar los parametros reales-->
     <collision>
-      <origin xyz="0 0 -7" rpy="0.0 0.0 0.0"/>
+      <origin xyz="0 2 -7" rpy="0.0 0.0 0.0"/>
       <geometry>
         <mesh filename="${visual_mesh_file}" scale="1 1 1" />
@@ -19,5 +19,5 @@
     </collision>
     <inertial>
-      <origin xyz="0 0 -7" rpy="0.0 0.0 0.0"/>
+      <origin xyz="0 2 -7" rpy="0.0 0.0 0.0"/>
       <mass value="1"/>
       <inertia
@@ -27,5 +27,5 @@
     </inertial>
 </link>
-<gazebo reference="gate_base">
+<gazebo reference="buoy2_base">
   <selfCollide>0</selfCollide>
   <turnGravityOff>1</turnGravityOff>

File: uv_worlds/urdf/gate.xacro (robot description, xacro)
@@ -1,10 +1,10 @@
 <?xml version="1.0"?>
-<robot name="path_marker2" xmlns:xacro="http://www.ros.org/wiki/xacro">
+<robot name="gate_1" xmlns:xacro="http://www.ros.org/wiki/xacro">
 <!-- Introducir meshes -->
-<xacro:property name="visual_mesh_file" value="file://$(find sim_challenges)/models/meshes/pathmarkers/pathmarker2.dae" />
-<!-- <origin xyz="0.085 (0 -0.085) 0 0" rpy="0.0 0.0 0.0075"/> -->
-<link name="path_marker_base2">
+<xacro:property name="visual_mesh_file" value="file://$(find uv_worlds)/models/props//mygate1.dae" />
+<!-- <origin xyz="0.085 (0 -0.085) 0 0" rpy="0.0 0.0 1.57075"/> -->
+<link name="gate_base">
     <visual>
-        <origin xyz="0 0 -4" rpy="0.0 0.0 0.0"/>
+        <origin xyz="0 0 -7" rpy="0.0 0.0 0"/>
         <geometry>
             <mesh filename="${visual_mesh_file}" scale="1 1 1" />
@@ -13,5 +13,5 @@
         <!-- Se deben cambiar los parametros reales-->
     <collision>
-      <origin xyz="0 0 -4" rpy="0.0 0.0 0.0"/>
+      <origin xyz="0 0 -7" rpy="0.0 0.0 0.0"/>
       <geometry>
         <mesh filename="${visual_mesh_file}" scale="1 1 1" />
@@ -19,5 +19,5 @@
     </collision>
     <inertial>
-      <origin xyz="0 0 -4" rpy="0.0 0.0 0.0"/>
+      <origin xyz="0 0 -7" rpy="0.0 0.0 0.0"/>
       <mass value="1"/>
       <inertia
@@ -27,5 +27,5 @@
     </inertial>
 </link>
-<gazebo reference="path_marker_base2">
+<gazebo reference="gate_base">
   <selfCollide>0</selfCollide>
   <turnGravityOff>1</turnGravityOff>

File: uv_worlds/urdf/octagon.xacro (robot description, xacro)
@@ -1,10 +1,10 @@
 <?xml version="1.0"?>
-<robot name="path_marker9" xmlns:xacro="http://www.ros.org/wiki/xacro">
+<robot name="octagon_1" xmlns:xacro="http://www.ros.org/wiki/xacro">
 <!-- Introducir meshes -->
-<xacro:property name="visual_mesh_file" value="file://$(find sim_challenges)/models/meshes/pathmarkers/pathmarker9.dae" />
-<!-- <origin xyz="0.085 (0 -0.085) 0 0" rpy="0.0 0.0 0.0075"/> -->
-<link name="path_marker_base9">
+<xacro:property name="visual_mesh_file" value="file://$(find uv_worlds)/models/props//Myoctagon2.dae" />
+<!-- <origin xyz="0.085 (0 -0.085) 0 0" rpy="0.0 0.0 1.57075"/> -->
+<link name="octagon_base">
     <visual>
-        <origin xyz="0 0 -4" rpy="0.0 0.0 0.0"/>
+        <origin xyz="0 2 -7" rpy="0.0 0.0 0.0"/>
         <geometry>
             <mesh filename="${visual_mesh_file}" scale="1 1 1" />
@@ -13,5 +13,5 @@
         <!-- Se deben cambiar los parametros reales-->
     <collision>
-      <origin xyz="0 0 -4" rpy="0.0 0.0 0.0"/>
+      <origin xyz="0 2 -7" rpy="0.0 0.0 0.0"/>
       <geometry>
         <mesh filename="${visual_mesh_file}" scale="1 1 1" />
@@ -19,5 +19,5 @@
     </collision>
     <inertial>
-      <origin xyz="0 0 -4" rpy="0.0 0.0 0.0"/>
+      <origin xyz="0 2 -7" rpy="0.0 0.0 0.0"/>
       <mass value="1"/>
       <inertia
@@ -27,5 +27,5 @@
     </inertial>
 </link>
-<gazebo reference="path_marker_base9">
+<gazebo reference="octagon_base">
   <selfCollide>0</selfCollide>
   <turnGravityOff>1</turnGravityOff>

File: uv_worlds/urdf/pathmarkers/pathmarker1.xacro (robot description, xacro)
@@ -1,10 +1,10 @@
 <?xml version="1.0"?>
-<robot name="bin_2" xmlns:xacro="http://www.ros.org/wiki/xacro">
+<robot name="path_marker" xmlns:xacro="http://www.ros.org/wiki/xacro">
 <!-- Introducir meshes -->
-<xacro:property name="visual_mesh_file" value="file://$(find sim_challenges)/models/meshes/bin02.dae" />
-<!-- <origin xyz="0.085 (0 -0.085) 0 0" rpy="0.0 0.0 1.57075"/> -->
-<link name="bin2_base">
+<xacro:property name="visual_mesh_file" value="file://$(find uv_worlds)/models/props/pathmarkers/pathmarker1.dae" />
+<!-- <origin xyz="0.085 (0 -0.085) 0 0" rpy="0.0 0.0 0.0075"/> -->
+<link name="path_marker_base">
     <visual>
-        <origin xyz="0 2 -7" rpy="0.0 0.0 0.0"/>
+        <origin xyz="0 0 -8.5" rpy="0.0 0.0 0.0"/>
         <geometry>
             <mesh filename="${visual_mesh_file}" scale="1 1 1" />
@@ -13,5 +13,5 @@
         <!-- Se deben cambiar los parametros reales-->
     <collision>
-      <origin xyz="0 2 -7" rpy="0.0 0.0 0.0"/>
+      <origin xyz="0 0 -8.5" rpy="0.0 0.0 0.0"/>
       <geometry>
         <mesh filename="${visual_mesh_file}" scale="1 1 1" />
@@ -19,5 +19,5 @@
     </collision>
     <inertial>
-      <origin xyz="0 2 -7" rpy="0.0 0.0 0.0"/>
+      <origin xyz="0 0 -8.5" rpy="0.0 0.0 0.0"/>
       <mass value="1"/>
       <inertia
@@ -27,5 +27,5 @@
     </inertial>
 </link>
-<gazebo reference="bin2_base">
+<gazebo reference="path_marker_base">
   <selfCollide>0</selfCollide>
   <turnGravityOff>1</turnGravityOff>

File: uv_worlds/urdf/pathmarkers/pathmarker10.xacro (robot description, xacro)
@@ -1,10 +1,10 @@
 <?xml version="1.0"?>
-<robot name="path_marker" xmlns:xacro="http://www.ros.org/wiki/xacro">
+<robot name="path_marker10" xmlns:xacro="http://www.ros.org/wiki/xacro">
 <!-- Introducir meshes -->
-<xacro:property name="visual_mesh_file" value="file://$(find sim_challenges)/models/meshes/pathmarkers/pathmarker1.dae" />
+<xacro:property name="visual_mesh_file" value="file://$(find uv_worlds)/models/props/pathmarkers/pathmarker10.dae" />
 <!-- <origin xyz="0.085 (0 -0.085) 0 0" rpy="0.0 0.0 0.0075"/> -->
-<link name="path_marker_base">
+<link name="path_marker_base10">
     <visual>
-        <origin xyz="0 0 -8.5" rpy="0.0 0.0 0.0"/>
+        <origin xyz="0 0 -4" rpy="0.0 0.0 0.0"/>
         <geometry>
             <mesh filename="${visual_mesh_file}" scale="1 1 1" />
@@ -13,5 +13,5 @@
         <!-- Se deben cambiar los parametros reales-->
     <collision>
-      <origin xyz="0 0 -8.5" rpy="0.0 0.0 0.0"/>
+      <origin xyz="0 0 -4" rpy="0.0 0.0 0.0"/>
       <geometry>
         <mesh filename="${visual_mesh_file}" scale="1 1 1" />
@@ -19,5 +19,5 @@
     </collision>
     <inertial>
-      <origin xyz="0 0 -8.5" rpy="0.0 0.0 0.0"/>
+      <origin xyz="0 0 -4" rpy="0.0 0.0 0.0"/>
       <mass value="1"/>
       <inertia
@@ -27,5 +27,5 @@
     </inertial>
 </link>
-<gazebo reference="path_marker_base">
+<gazebo reference="path_marker_base10">
   <selfCollide>0</selfCollide>
   <turnGravityOff>1</turnGravityOff>

File: uv_worlds/urdf/pathmarkers/pathmarker2.xacro (robot description, xacro)
@@ -1,10 +1,10 @@
 <?xml version="1.0"?>
-<robot name="torpedos_1" xmlns:xacro="http://www.ros.org/wiki/xacro">
+<robot name="path_marker2" xmlns:xacro="http://www.ros.org/wiki/xacro">
 <!-- Introducir meshes -->
-<xacro:property name="visual_mesh_file" value="file://$(find sim_challenges)/models/meshes/finaltorpedos.dae" />
-<!-- <origin xyz="0.085 (0 -0.085) 0 0" rpy="0.0 0.0 1.57075"/> -->
-<link name="torpedos1_base">
+<xacro:property name="visual_mesh_file" value="file://$(find uv_worlds)/models/props/pathmarkers/pathmarker2.dae" />
+<!-- <origin xyz="0.085 (0 -0.085) 0 0" rpy="0.0 0.0 0.0075"/> -->
+<link name="path_marker_base2">
     <visual>
-        <origin xyz="0 2 -7" rpy="0.0 0.0 0.0"/>
+        <origin xyz="0 0 -4" rpy="0.0 0.0 0.0"/>
         <geometry>
             <mesh filename="${visual_mesh_file}" scale="1 1 1" />
@@ -13,5 +13,5 @@
         <!-- Se deben cambiar los parametros reales-->
     <collision>
-      <origin xyz="0 2 -7" rpy="0.0 0.0 0.0"/>
+      <origin xyz="0 0 -4" rpy="0.0 0.0 0.0"/>
       <geometry>
         <mesh filename="${visual_mesh_file}" scale="1 1 1" />
@@ -19,5 +19,5 @@
     </collision>
     <inertial>
-      <origin xyz="0 2 -7" rpy="0.0 0.0 0.0"/>
+      <origin xyz="0 0 -4" rpy="0.0 0.0 0.0"/>
       <mass value="1"/>
       <inertia
@@ -27,5 +27,5 @@
     </inertial>
 </link>
-<gazebo reference="torpedos1_base">
+<gazebo reference="path_marker_base2">
   <selfCollide>0</selfCollide>
   <turnGravityOff>1</turnGravityOff>

File: uv_worlds/urdf/pathmarkers/pathmarker3.xacro (robot description, xacro)
@@ -1,10 +1,10 @@
 <?xml version="1.0"?>
-<robot name="path_marker5" xmlns:xacro="http://www.ros.org/wiki/xacro">
+<robot name="path_marker3" xmlns:xacro="http://www.ros.org/wiki/xacro">
 <!-- Introducir meshes -->
-<xacro:property name="visual_mesh_file" value="file://$(find sim_challenges)/models/meshes/pathmarkers/pathmarker5.dae" />
+<xacro:property name="visual_mesh_file" value="file://$(find uv_worlds)/models/props/pathmarkers/pathmarker3.dae" />
 <!-- <origin xyz="0.085 (0 -0.085) 0 0" rpy="0.0 0.0 0.0075"/> -->
-<link name="path_marker_base5">
+<link name="path_marker_base3">
     <visual>
-        <origin xyz="0 0 -4" rpy="0.0 0.0 0.0"/>
+        <origin xyz="0 2 -8.5" rpy="0.0 0.0 0.0"/>
         <geometry>
             <mesh filename="${visual_mesh_file}" scale="1 1 1" />
@@ -13,5 +13,5 @@
         <!-- Se deben cambiar los parametros reales-->
     <collision>
-      <origin xyz="0 0 -4" rpy="0.0 0.0 0.0"/>
+      <origin xyz="0 2 -8.5" rpy="0.0 0.0 0.0"/>
       <geometry>
         <mesh filename="${visual_mesh_file}" scale="1 1 1" />
@@ -19,5 +19,5 @@
     </collision>
     <inertial>
-      <origin xyz="0 0 -4" rpy="0.0 0.0 0.0"/>
+      <origin xyz="0 2 -8.5" rpy="0.0 0.0 0.0"/>
       <mass value="1"/>
       <inertia
@@ -27,5 +27,5 @@
     </inertial>
 </link>
-<gazebo reference="path_marker_base5">
+<gazebo reference="path_marker_base3">
   <selfCollide>0</selfCollide>
   <turnGravityOff>1</turnGravityOff>

File: uv_worlds/urdf/pathmarkers/pathmarker4.xacro (robot description, xacro)
@@ -1,8 +1,8 @@
 <?xml version="1.0"?>
-<robot name="path_marker7" xmlns:xacro="http://www.ros.org/wiki/xacro">
+<robot name="path_marker4" xmlns:xacro="http://www.ros.org/wiki/xacro">
 <!-- Introducir meshes -->
-<xacro:property name="visual_mesh_file" value="file://$(find sim_challenges)/models/meshes/pathmarkers/pathmarker7.dae" />
+<xacro:property name="visual_mesh_file" value="file://$(find uv_worlds)/models/props/pathmarkers/pathmarker4.dae" />
 <!-- <origin xyz="0.085 (0 -0.085) 0 0" rpy="0.0 0.0 0.0075"/> -->
-<link name="path_marker_base7">
+<link name="path_marker_base4">
     <visual>
         <origin xyz="0 0 -4" rpy="0.0 0.0 0.0"/>
@@ -27,5 +27,5 @@
     </inertial>
 </link>
-<gazebo reference="path_marker_base7">
+<gazebo reference="path_marker_base4">
   <selfCollide>0</selfCollide>
   <turnGravityOff>1</turnGravityOff>

File: uv_worlds/urdf/pathmarkers/pathmarker5.xacro (robot description, xacro)
@@ -1,10 +1,10 @@
 <?xml version="1.0"?>
-<robot name="buoy_2" xmlns:xacro="http://www.ros.org/wiki/xacro">
+<robot name="path_marker5" xmlns:xacro="http://www.ros.org/wiki/xacro">
 <!-- Introducir meshes -->
-<xacro:property name="visual_mesh_file" value="file://$(find sim_challenges)/models/meshes/buoy2.dae" />
-<!-- <origin xyz="0.085 (0 -0.085) 0 0" rpy="0.0 0.0 1.57075"/> -->
-<link name="buoy2_base">
+<xacro:property name="visual_mesh_file" value="file://$(find uv_worlds)/models/props/pathmarkers/pathmarker5.dae" />
+<!-- <origin xyz="0.085 (0 -0.085) 0 0" rpy="0.0 0.0 0.0075"/> -->
+<link name="path_marker_base5">
     <visual>
-        <origin xyz="0 2 -7" rpy="0.0 0.0 0.0"/>
+        <origin xyz="0 0 -4" rpy="0.0 0.0 0.0"/>
         <geometry>
             <mesh filename="${visual_mesh_file}" scale="1 1 1" />
@@ -13,5 +13,5 @@
         <!-- Se deben cambiar los parametros reales-->
     <collision>
-      <origin xyz="0 2 -7" rpy="0.0 0.0 0.0"/>
+      <origin xyz="0 0 -4" rpy="0.0 0.0 0.0"/>
       <geometry>
         <mesh filename="${visual_mesh_file}" scale="1 1 1" />
@@ -19,5 +19,5 @@
     </collision>
     <inertial>
-      <origin xyz="0 2 -7" rpy="0.0 0.0 0.0"/>
+      <origin xyz="0 0 -4" rpy="0.0 0.0 0.0"/>
       <mass value="1"/>
       <inertia
@@ -27,5 +27,5 @@
     </inertial>
 </link>
-<gazebo reference="buoy2_base">
+<gazebo reference="path_marker_base5">
   <selfCollide>0</selfCollide>
   <turnGravityOff>1</turnGravityOff>

File: uv_worlds/urdf/pathmarkers/pathmarker6.xacro (robot description, xacro)
@@ -1,8 +1,8 @@
 <?xml version="1.0"?>
-<robot name="path_marker10" xmlns:xacro="http://www.ros.org/wiki/xacro">
+<robot name="path_marker6" xmlns:xacro="http://www.ros.org/wiki/xacro">
 <!-- Introducir meshes -->
-<xacro:property name="visual_mesh_file" value="file://$(find sim_challenges)/models/meshes/pathmarkers/pathmarker10.dae" />
+<xacro:property name="visual_mesh_file" value="file://$(find uv_worlds)/models/props/pathmarkers/pathmarker6.dae" />
 <!-- <origin xyz="0.085 (0 -0.085) 0 0" rpy="0.0 0.0 0.0075"/> -->
-<link name="path_marker_base10">
+<link name="path_marker_base6">
     <visual>
         <origin xyz="0 0 -4" rpy="0.0 0.0 0.0"/>
@@ -27,5 +27,5 @@
     </inertial>
 </link>
-<gazebo reference="path_marker_base10">
+<gazebo reference="path_marker_base6">
   <selfCollide>0</selfCollide>
   <turnGravityOff>1</turnGravityOff>

File: uv_worlds/urdf/pathmarkers/pathmarker7.xacro (robot description, xacro)
@@ -1,8 +1,8 @@
 <?xml version="1.0"?>
-<robot name="path_marker4" xmlns:xacro="http://www.ros.org/wiki/xacro">
+<robot name="path_marker7" xmlns:xacro="http://www.ros.org/wiki/xacro">
 <!-- Introducir meshes -->
-<xacro:property name="visual_mesh_file" value="file://$(find sim_challenges)/models/meshes/pathmarkers/pathmarker4.dae" />
+<xacro:property name="visual_mesh_file" value="file://$(find uv_worlds)/models/props/pathmarkers/pathmarker7.dae" />
 <!-- <origin xyz="0.085 (0 -0.085) 0 0" rpy="0.0 0.0 0.0075"/> -->
-<link name="path_marker_base4">
+<link name="path_marker_base7">
     <visual>
         <origin xyz="0 0 -4" rpy="0.0 0.0 0.0"/>
@@ -27,5 +27,5 @@
     </inertial>
 </link>
-<gazebo reference="path_marker_base4">
+<gazebo reference="path_marker_base7">
   <selfCollide>0</selfCollide>
   <turnGravityOff>1</turnGravityOff>

File: uv_worlds/urdf/pathmarkers/pathmarker8.xacro (robot description, xacro)
@@ -1,11 +1,10 @@
 <?xml version="1.0"?>
-<robot name="bin_1" xmlns:xacro="http://www.ros.org/wiki/xacro">
-<!--Change .dae to binopen.dae, bintapadod.dae, bintapadoi.dae depending on the situation-->
+<robot name="path_marker8" xmlns:xacro="http://www.ros.org/wiki/xacro">
 <!-- Introducir meshes -->
-<xacro:property name="visual_mesh_file" value="file://$(find sim_challenges)/models/meshes/bintapadoi.dae" />
-<!-- <origin xyz="0.085 (0 -0.085) 0 0" rpy="0.0 0.0 1.57075"/> -->
-<link name="bin1_base">
+<xacro:property name="visual_mesh_file" value="file://$(find uv_worlds)/models/props/pathmarkers/pathmarker8.dae" />
+<!-- <origin xyz="0.085 (0 -0.085) 0 0" rpy="0.0 0.0 0.0075"/> -->
+<link name="path_marker_base8">
     <visual>
-        <origin xyz="0 2 -7" rpy="0.0 0.0 0.0"/>
+        <origin xyz="0 0 -4" rpy="0.0 0.0 0.0"/>
         <geometry>
             <mesh filename="${visual_mesh_file}" scale="1 1 1" />
@@ -14,5 +13,5 @@
         <!-- Se deben cambiar los parametros reales-->
     <collision>
-      <origin xyz="0 2 -7" rpy="0.0 0.0 0.0"/>
+      <origin xyz="0 0 -4" rpy="0.0 0.0 0.0"/>
       <geometry>
         <mesh filename="${visual_mesh_file}" scale="1 1 1" />
@@ -20,5 +19,5 @@
     </collision>
     <inertial>
-      <origin xyz="0 2 -7" rpy="0.0 0.0 0.0"/>
+      <origin xyz="0 0 -4" rpy="0.0 0.0 0.0"/>
       <mass value="1"/>
       <inertia
@@ -28,5 +27,5 @@
     </inertial>
 </link>
-<gazebo reference="bin1_base">
+<gazebo reference="path_marker_base8">
   <selfCollide>0</selfCollide>
   <turnGravityOff>1</turnGravityOff>

File: uv_worlds/urdf/pathmarkers/pathmarker9.xacro (robot description, xacro)
@@ -1,10 +1,10 @@
 <?xml version="1.0"?>
-<robot name="torpedos_2" xmlns:xacro="http://www.ros.org/wiki/xacro">
+<robot name="path_marker9" xmlns:xacro="http://www.ros.org/wiki/xacro">
 <!-- Introducir meshes -->
-<xacro:property name="visual_mesh_file" value="file://$(find sim_challenges)/models/meshes/Mytorpedos2.dae" />
-<!-- <origin xyz="0.085 (0 -0.085) 0 0" rpy="0.0 0.0 1.57075"/> -->
-<link name="torpedos2_base">
+<xacro:property name="visual_mesh_file" value="file://$(find uv_worlds)/models/props/pathmarkers/pathmarker9.dae" />
+<!-- <origin xyz="0.085 (0 -0.085) 0 0" rpy="0.0 0.0 0.0075"/> -->
+<link name="path_marker_base9">
     <visual>
-        <origin xyz="0 2 -7" rpy="0.0 0.0 0.0"/>
+        <origin xyz="0 0 -4" rpy="0.0 0.0 0.0"/>
         <geometry>
             <mesh filename="${visual_mesh_file}" scale="1 1 1" />
@@ -13,5 +13,5 @@
         <!-- Se deben cambiar los parametros reales-->
     <collision>
-      <origin xyz="0 2 -7" rpy="0.0 0.0 0.0"/>
+      <origin xyz="0 0 -4" rpy="0.0 0.0 0.0"/>
       <geometry>
         <mesh filename="${visual_mesh_file}" scale="1 1 1" />
@@ -19,5 +19,5 @@
     </collision>
     <inertial>
-      <origin xyz="0 2 -7" rpy="0.0 0.0 0.0"/>
+      <origin xyz="0 0 -4" rpy="0.0 0.0 0.0"/>
       <mass value="1"/>
       <inertia
@@ -27,5 +27,5 @@
     </inertial>
 </link>
-<gazebo reference="torpedos2_base">
+<gazebo reference="path_marker_base9">
   <selfCollide>0</selfCollide>
   <turnGravityOff>1</turnGravityOff>

File: uv_worlds/urdf/torpedos1.xacro (robot description, xacro)
@@ -1,10 +1,10 @@
 <?xml version="1.0"?>
-<robot name="path_marker3" xmlns:xacro="http://www.ros.org/wiki/xacro">
+<robot name="torpedos_1" xmlns:xacro="http://www.ros.org/wiki/xacro">
 <!-- Introducir meshes -->
-<xacro:property name="visual_mesh_file" value="file://$(find sim_challenges)/models/meshes/pathmarkers/pathmarker3.dae" />
-<!-- <origin xyz="0.085 (0 -0.085) 0 0" rpy="0.0 0.0 0.0075"/> -->
-<link name="path_marker_base3">
+<xacro:property name="visual_mesh_file" value="file://$(find uv_worlds)/models/props//finaltorpedos.dae" />
+<!-- <origin xyz="0.085 (0 -0.085) 0 0" rpy="0.0 0.0 1.57075"/> -->
+<link name="torpedos1_base">
     <visual>
-        <origin xyz="0 2 -8.5" rpy="0.0 0.0 0.0"/>
+        <origin xyz="0 2 -7" rpy="0.0 0.0 0.0"/>
         <geometry>
             <mesh filename="${visual_mesh_file}" scale="1 1 1" />
@@ -13,5 +13,5 @@
         <!-- Se deben cambiar los parametros reales-->
     <collision>
-      <origin xyz="0 2 -8.5" rpy="0.0 0.0 0.0"/>
+      <origin xyz="0 2 -7" rpy="0.0 0.0 0.0"/>
       <geometry>
         <mesh filename="${visual_mesh_file}" scale="1 1 1" />
@@ -19,5 +19,5 @@
     </collision>
     <inertial>
-      <origin xyz="0 2 -8.5" rpy="0.0 0.0 0.0"/>
+      <origin xyz="0 2 -7" rpy="0.0 0.0 0.0"/>
       <mass value="1"/>
       <inertia
@@ -27,5 +27,5 @@
     </inertial>
 </link>
-<gazebo reference="path_marker_base3">
+<gazebo reference="torpedos1_base">
   <selfCollide>0</selfCollide>
   <turnGravityOff>1</turnGravityOff>
