Commit message: Removed unnecessary package

File: uv_worlds/urdf/torpedos2.xacro (robot description, xacro)
@@ -1,10 +1,10 @@
 <?xml version="1.0"?>
-<robot name="path_marker8" xmlns:xacro="http://www.ros.org/wiki/xacro">
+<robot name="torpedos_2" xmlns:xacro="http://www.ros.org/wiki/xacro">
 <!-- Introducir meshes -->
-<xacro:property name="visual_mesh_file" value="file://$(find sim_challenges)/models/meshes/pathmarkers/pathmarker8.dae" />
-<!-- <origin xyz="0.085 (0 -0.085) 0 0" rpy="0.0 0.0 0.0075"/> -->
-<link name="path_marker_base8">
+<xacro:property name="visual_mesh_file" value="file://$(find uv_worlds)/models/props//Mytorpedos2.dae" />
+<!-- <origin xyz="0.085 (0 -0.085) 0 0" rpy="0.0 0.0 1.57075"/> -->
+<link name="torpedos2_base">
     <visual>
-        <origin xyz="0 0 -4" rpy="0.0 0.0 0.0"/>
+        <origin xyz="0 2 -7" rpy="0.0 0.0 0.0"/>
         <geometry>
             <mesh filename="${visual_mesh_file}" scale="1 1 1" />
@@ -13,5 +13,5 @@
         <!-- Se deben cambiar los parametros reales-->
     <collision>
-      <origin xyz="0 0 -4" rpy="0.0 0.0 0.0"/>
+      <origin xyz="0 2 -7" rpy="0.0 0.0 0.0"/>
       <geometry>
         <mesh filename="${visual_mesh_file}" scale="1 1 1" />
@@ -19,5 +19,5 @@
     </collision>
     <inertial>
-      <origin xyz="0 0 -4" rpy="0.0 0.0 0.0"/>
+      <origin xyz="0 2 -7" rpy="0.0 0.0 0.0"/>
       <mass value="1"/>
       <inertia
@@ -27,5 +27,5 @@
     </inertial>
 </link>
-<gazebo reference="path_marker_base8">
+<gazebo reference="torpedos2_base">
   <selfCollide>0</selfCollide>
   <turnGravityOff>1</turnGravityOff>
