Commit message: update robot files, ignore new models for now

File: sensors/uuv_sensor_plugins/uuv_sensor_ros_plugins/urdf/dvl_snippets.xacro (robot description, xacro)
@@ -168,5 +168,5 @@
         <robot_namespace>${namespace}</robot_namespace> <!-- (string, required): ros namespace in which the messages are published -->
 	<!-- Changed from dvl_link to base_link to get ENU coordinate frame -->
-        <link_name>${namespace}/base_link</link_name> <!-- (string, required): name of the body which holds the IMU sensor -->
+        <link_name>${namespace}_base_link</link_name> <!-- (string, required): name of the body which holds the IMU sensor -->
         <sensor_topic>${topic}</sensor_topic> <!-- (string): name of the sensor output topic and prefix of service names -->
         <update_rate>${update_rate}</update_rate> <!-- Update period [s] -->

File: uv_worlds/urdf/bottle.xacro (robot description, xacro)
@@ -1,10 +1,10 @@
 <?xml version="1.0"?>
-<robot name="gate_1" xmlns:xacro="http://www.ros.org/wiki/xacro">
+<robot name="bottle" xmlns:xacro="http://www.ros.org/wiki/xacro">
 <!-- Introducir meshes -->
-<xacro:property name="visual_mesh_file" value="file://$(find uv_worlds)/models/gate1/mygate1.dae" />
+<xacro:property name="visual_mesh_file" value="file://$(find uv_worlds)/models/props/bottle/water_bottle.dae" />
 <!-- <origin xyz="0.085 (0 -0.085) 0 0" rpy="0.0 0.0 1.57075"/> -->
-<link name="gate_base">
+<link name="bottle_base">
     <visual>
-        <origin xyz="0 0 -7" rpy="0.0 0.0 0"/>
+        <origin xyz="9.85 27.9 -8.45" rpy="0.0 0.0 0.0"/>
         <geometry>
             <mesh filename="${visual_mesh_file}" scale="1 1 1" />
@@ -13,5 +13,5 @@
         <!-- Se deben cambiar los parametros reales-->
     <collision>
-      <origin xyz="0 0 -7" rpy="0.0 0.0 0.0"/>
+      <origin xyz="9.85 27.9 -8.45" rpy="0.0 0.0 0.0"/>
       <geometry>
         <mesh filename="${visual_mesh_file}" scale="1 1 1" />
@@ -19,5 +19,5 @@
     </collision>
     <inertial>
-      <origin xyz="0 0 -7" rpy="0.0 0.0 0.0"/>
+      <origin xyz="9.85 27.9 -8.45" rpy="0.0 0.0 0.0"/>
       <mass value="1"/>
       <inertia
@@ -27,5 +27,5 @@
     </inertial>
 </link>
-<gazebo reference="gate_base">
+<gazebo reference="bottle_base">
   <selfCollide>0</selfCollide>
   <turnGravityOff>1</turnGravityOff>

File: uv_worlds/urdf/mapa1.xacro (robot description, xacro)
@@ -1,8 +1,8 @@
 <?xml version="1.0"?>
-<robot name="gate_1" xmlns:xacro="http://www.ros.org/wiki/xacro">
+<robot name="mapa1_1" xmlns:xacro="http://www.ros.org/wiki/xacro">
 <!-- Introducir meshes -->
-<xacro:property name="visual_mesh_file" value="file://$(find uv_worlds)/models/gate1/mygate1.dae" />
+<xacro:property name="visual_mesh_file" value="file://$(find uv_worlds)/newworlds/mapa_1_1.dae"/>
 <!-- <origin xyz="0.085 (0 -0.085) 0 0" rpy="0.0 0.0 1.57075"/> -->
-<link name="gate_base">
+<link name="mapa1_base">
     <visual>
         <origin xyz="0 0 -7" rpy="0.0 0.0 0"/>
@@ -27,5 +27,5 @@
     </inertial>
 </link>
-<gazebo reference="gate_base">
+<gazebo reference="mapa1_base">
   <selfCollide>0</selfCollide>
   <turnGravityOff>1</turnGravityOff>

File: vehicle_descriptions/robots/vtec_u3.xacro (robot description, xacro)
@@ -8,4 +8,5 @@
   <xacro:include filename="$(find vehicle_descriptions)/urdf/UUVs/vtec_u3_arm.xacro"/>
   <xacro:include filename="$(find vehicle_descriptions)/urdf/UUVs/vtec_u3_shooter.xacro"/>
+  <virtual_joint name="world_joint" type="planar" parent_frame="world_ned" child_link="vtec_u3_base_link"/>
   <xacro:vtec_u3_base namespace="$(arg namespace)"/>
   <xacro:vtec_u3_sensors namespace="$(arg namespace)"/>
