Commit message: Add files via upload

File: sensors/uuv_sensor_plugins/uuv_sensor_ros_plugins/urdf/camera_snippets.xacro (robot description, xacro)
@@ -28,5 +28,5 @@
       parent_link="${parent_link}"
       topic="camera"
-      mass="0.001"
+      mass="0.1"
       update_rate="30"
       hfov="1.5125"
@@ -166,4 +166,24 @@
       <limit upper="0" lower="0" effort="0" velocity="0" />
     </joint>
+    <link name="${namespace}/camera${suffix}_link_optical">
+      <xacro:box_inertial x="0.0001" y="0.0001" z="0.0001" mass="0.001">
+        <origin xyz="0 0 0" rpy="0 0 0"/>
+      </xacro:box_inertial>
+      <collision>
+        <!-- todo: gazebo needs a collision volume or it will ignore the pose of
+           the joint that leads to this link (and assume it to be the identity) -->
+        <geometry>
+          <cylinder length="0.000001" radius="0.000001"/>
+        </geometry>
+        <origin xyz="0 0 0" rpy="0 ${0.5*pi} 0"/>
+      </collision>
+    </link>
+    <joint name="${namespace}/camera${suffix}_optical_joint" type="revolute">
+      <origin xyz="0 0 0" rpy="${-pi/2} 0 ${-pi/2}"/>
+      <parent link="${namespace}/camera${suffix}_link"/>
+      <child link="${namespace}/camera${suffix}_link_optical"/>
+      <limit upper="0" lower="0" effort="0" velocity="0" />
+      <axis xyz="1 0 0"/>
+    </joint>
     <gazebo reference="${namespace}/camera${suffix}_link">
       <sensor type="depth" name="camera${suffix}">

File: sensors/uuv_sensor_plugins/uuv_sensor_ros_plugins/urdf/dvl_snippets.xacro (robot description, xacro)
@@ -29,7 +29,7 @@
       update_rate="7"
       topic="dvl"
-      noise_sigma="0.0"
-      noise_amplitude="0.0"
-      scale="0.5">
+      noise_sigma="0"
+      noise_amplitude="0"
+      scale="1">
       <xacro:insert_block name="origin" />
     </xacro:dvl_plugin_macro>
@@ -52,6 +52,4 @@
   </xacro:macro>
   <!-- DEPRECATED MACRO: See default_dvl_sensor_enu -->
-<!--  noise_sigma="1.0"
-      noise_amplitude="1.0" -->
   <xacro:macro name="default_dvl" params="namespace parent_link *origin">
     <xacro:dvl_plugin_macro
@@ -62,11 +60,11 @@
       update_rate="7"
       topic="dvl"
-      noise_sigma="0.0"
-      noise_amplitude="0.0"
-      scale="0.5">
+      noise_sigma="0"
+      noise_amplitude="0"
+      scale="1">
       <xacro:insert_block name="origin" />
     </xacro:dvl_plugin_macro>
   </xacro:macro>
-  <xacro:macro name="dvl_single_sonar" params="namespace suffix index pitch yaw">
+  <xacro:macro name="dvl_single_sonar" params="namespace suffix index pitch yaw update_rate">
     <link name="${namespace}/dvl${suffix}_sonar${index}_link">
       <inertial>
@@ -87,5 +85,5 @@
       <sensor type="ray" name="dvl${suffix}_sonar${index}">
         <pose>0 0 0 0 0 0</pose>
-        <update_rate>1</update_rate>
+        <update_rate>${update_rate}</update_rate>
         <visualize>false</visualize>
         <ray>
@@ -113,5 +111,5 @@
           <gaussianNoise>0.005</gaussianNoise>
           <alwaysOn>true</alwaysOn>
-          <updateRate>1</updateRate>
+          <updateRate>${update_rate}</updateRate>
           <topicName>${topic}_sonar${index}</topicName>
           <frameName>${namespace}/dvl${suffix}_sonar${index}_link</frameName>
@@ -138,7 +136,4 @@
       <xacro:no_collision/>
     </link>
-    <gazebo reference="${namespace}/dvl${suffix}_link">
-      <turnGravityOff>1</turnGravityOff>
-    </gazebo>
     <joint name="${namespace}/dvl${suffix}_joint" type="revolute">
       <xacro:insert_block name="origin" />
@@ -150,23 +145,22 @@
     <xacro:dvl_single_sonar
       namespace="${namespace}" suffix=""
-      index="0" pitch="-0.52" yaw="0.0">
+      index="0" pitch="-0.52" yaw="0.0" update_rate="${update_rate}">
     </xacro:dvl_single_sonar>
     <xacro:dvl_single_sonar
       namespace="${namespace}" suffix=""
-      index="1" pitch="0" yaw="0.52">
+      index="1" pitch="0" yaw="0.52" update_rate="${update_rate}">
     </xacro:dvl_single_sonar>
     <xacro:dvl_single_sonar
       namespace="${namespace}" suffix=""
-      index="2" pitch="0.52" yaw="0.0">
+      index="2" pitch="0.52" yaw="0.0" update_rate="${update_rate}">
     </xacro:dvl_single_sonar>
     <xacro:dvl_single_sonar
       namespace="${namespace}" suffix=""
-      index="3" pitch="0.0" yaw="-0.52">
+      index="3" pitch="0.0" yaw="-0.52" update_rate="${update_rate}">
     </xacro:dvl_single_sonar>
     <gazebo>
       <plugin filename="libuuv_gazebo_ros_dvl_plugin.so" name="libuuv_gazebo_dvl${suffix}_plugin">
         <robot_namespace>${namespace}</robot_namespace> <!-- (string, required): ros namespace in which the messages are published -->
-	<!-- Changed from dvl_link to base_link to get ENU coordinate frame -->
-        <link_name>${namespace}_base_link</link_name> <!-- (string, required): name of the body which holds the IMU sensor -->
+        <link_name>${namespace}/dvl${suffix}_link</link_name> <!-- (string, required): name of the body which holds the IMU sensor -->
         <sensor_topic>${topic}</sensor_topic> <!-- (string): name of the sensor output topic and prefix of service names -->
         <update_rate>${update_rate}</update_rate> <!-- Update period [s] -->

File: sensors/uuv_sensor_plugins/uuv_sensor_ros_plugins/urdf/imu_snippets.xacro (robot description, xacro)
@@ -130,7 +130,4 @@
       </inertial>
     </link>
-    <gazebo reference="${namespace}/imu${imu_suffix}_link">
-      <turnGravityOff>1</turnGravityOff>
-    </gazebo>
     <!-- IMU joint -->
     <joint name="${namespace}/imu${imu_suffix}_joint" type="revolute">

File: sensors/uuv_sensor_plugins/uuv_sensor_ros_plugins/urdf/magnetometer_snippets.xacro (robot description, xacro)
@@ -54,5 +54,5 @@
       <visual>
         <geometry>
-          <box size="0.05 0.05 0.05" />
+          <box size="0.1 0.1 0.1" />
         </geometry>
       </visual>
@@ -75,6 +75,5 @@
         <intensity>${mag_intensity}</intensity> <!-- magnitude of magnetic field [muT] -->
         <reference_heading>${pi}</reference_heading> <!-- reference heading [rad] -->
-	<!-- Kristoffer changed magnetic declination from being 0.0 -->
-        <declination>${-pi}</declination> <!-- reference declination [rad] -->
+        <declination>0.0</declination> <!-- reference declination [rad] -->
         <inclination>${pi*60/180}</inclination> <!-- refernce inclination [rad] -->
         <noise_xy>${noise_xy}</noise_xy> <!-- Discrete-time std. dev. of output noise in xy-axis [muT] -->

File: sensors/uuv_sensor_plugins/uuv_sensor_ros_plugins/urdf/pressure_snippets.xacro (robot description, xacro)
@@ -69,12 +69,9 @@
       <visual>
         <geometry>
-          <mesh filename="file://$(find uuv_sensor_ros_plugins)/meshes/pressure.dae" scale="0.1 0.1 0.1"/>
+          <mesh filename="file://$(find uuv_sensor_ros_plugins)/meshes/pressure.dae" scale="1 1 1"/>
         </geometry>
       </visual>
       <xacro:no_collision/>
     </link>
-    <gazebo reference="${namespace}/pressure${suffix}_link">>
-      <turnGravityOff>1</turnGravityOff>
-    </gazebo>
     <joint name="${namespace}/pressure${suffix}_joint" type="revolute">
       <xacro:insert_block name="origin" />

File: sensors/uuv_sensor_plugins/uuv_sensor_ros_plugins/urdf/sensor_snippets.xacro (robot description, xacro)
@@ -17,5 +17,4 @@
   <xacro:include filename="$(find uuv_sensor_ros_plugins)/urdf/pressure_snippets.xacro" />
   <xacro:include filename="$(find uuv_sensor_ros_plugins)/urdf/camera_snippets.xacro" />
-  <xacro:include filename="$(find uuv_sensor_ros_plugins)/urdf/realsense_camera.xacro" />
   <xacro:include filename="$(find uuv_sensor_ros_plugins)/urdf/dvl_snippets.xacro" />
   <xacro:include filename="$(find uuv_sensor_ros_plugins)/urdf/rpt_snippets.xacro" />
